File: hardware/keyboard/RGBMatrix2.sch (KiCad schematic (older format))
At the start: 29 parts

Commit message: use proper footprint, link symbols and footprints
Parts:
- D69, D70, D71, D72, D73, D74, D75, D76, D77, D78, D79, D80, D81, D82, D83, D84, D85, D86, D87, D88, D89, D90, D91, D92, D93, D94, D95, D96, D97: footprint (none) -> KiCad:XZMDKCBDDG45S9
Changed lines of the file:
@@
 F 0 "D69" H 1750 2897 50  0000 C CNN
 F 1 "LED_RABG" H 1750 2806 50  0000 C CNN
-F 2 "" H 1750 2350 50  0001 C CNN
+F 2 "KiCad:XZMDKCBDDG45S9" H 1750 2350 50  0001 C CNN
 F 3 "~" H 1750 2350 50  0001 C CNN
 	1    1750 2400
@@
 F 0 "D71" H 2350 2897 50  0000 C CNN
 F 1 "LED_RABG" H 2350 2806 50  0000 C CNN
-F 2 "" H 2350 2350 50  0001 C CNN
+F 2 "KiCad:XZMDKCBDDG45S9" H 2350 2350 50  0001 C CNN
 F 3 "~" H 2350 2350 50  0001 C CNN
 	1    2350 2400
@@
 F 0 "D73" H 2950 2897 50  0000 C CNN
 F 1 "LED_RABG" H 2950 2806 50  0000 C CNN
-F 2 "" H 2950 2350 50  0001 C CNN
+F 2 "KiCad:XZMDKCBDDG45S9" H 2950 2350 50  0001 C CNN
 F 3 "~" H 2950 2350 50  0001 C CNN
 	1    2950 2400
@@
 F 0 "D75" H 3550 2897 50  0000 C CNN
 F 1 "LED_RABG" H 3550 2806 50  0000 C CNN
-F 2 "" H 3550 2350 50  0001 C CNN
+F 2 "KiCad:XZMDKCBDDG45S9" H 3550 2350 50  0001 C CNN
 F 3 "~" H 3550 2350 50  0001 C CNN
 	1    3550 2400
@@
 F 0 "D77" H 4100 2897 50  0000 C CNN
 F 1 "LED_RABG" H 4100 2806 50  0000 C CNN
-F 2 "" H 4100 2350 50  0001 C CNN
+F 2 "KiCad:XZMDKCBDDG45S9" H 4100 2350 50  0001 C CNN
 F 3 "~" H 4100 2350 50  0001 C CNN
 	1    4100 2400
@@
 F 0 "D79" H 4700 2897 50  0000 C CNN
 F 1 "LED_RABG" H 4700 2806 50  0000 C CNN
-F 2 "" H 4700 2350 50  0001 C CNN
+F 2 "KiCad:XZMDKCBDDG45S9" H 4700 2350 50  0001 C CNN
 F 3 "~" H 4700 2350 50  0001 C CNN
 	1    4700 2400
@@
 F 0 "D81" H 5300 2897 50  0000 C CNN
 F 1 "LED_RABG" H 5300 2806 50  0000 C CNN
-F 2 "" H 5300 2350 50  0001 C CNN
+F 2 "KiCad:XZMDKCBDDG45S9" H 5300 2350 50  0001 C CNN
 F 3 "~" H 5300 2350 50  0001 C CNN
 	1    5300 2400
@@
 F 0 "D82" H 5900 2897 50  0000 C CNN
 F 1 "LED_RABG" H 5900 2806 50  0000 C CNN
-F 2 "" H 5900 2350 50  0001 C CNN
+F 2 "KiCad:XZMDKCBDDG45S9" H 5900 2350 50  0001 C CNN
 F 3 "~" H 5900 2350 50  0001 C CNN
 	1    5900 2400
@@
 F 0 "D84" H 6500 2897 50  0000 C CNN
 F 1 "LED_RABG" H 6500 2806 50  0000 C CNN
-F 2 "" H 6500 2350 50  0001 C CNN
+F 2 "KiCad:XZMDKCBDDG45S9" H 6500 2350 50  0001 C CNN
 F 3 "~" H 6500 2350 50  0001 C CNN
 	1    6500 2400
@@
 F 0 "D86" H 7100 2897 50  0000 C CNN
 F 1 "LED_RABG" H 7100 2806 50  0000 C CNN
-F 2 "" H 7100 2350 50  0001 C CNN
+F 2 "KiCad:XZMDKCBDDG45S9" H 7100 2350 50  0001 C CNN
 F 3 "~" H 7100 2350 50  0001 C CNN
 	1    7100 2400
@@
 F 0 "D88" H 7700 2897 50  0000 C CNN
 F 1 "LED_RABG" H 7700 2806 50  0000 C CNN
-F 2 "" H 7700 2350 50  0001 C CNN
+F 2 "KiCad:XZMDKCBDDG45S9" H 7700 2350 50  0001 C CNN
 F 3 "~" H 7700 2350 50  0001 C CNN
 	1    7700 2400
@@
 F 0 "D90" H 8300 2897 50  0000 C CNN
 F 1 "LED_RABG" H 8300 2806 50  0000 C CNN
-F 2 "" H 8300 2350 50  0001 C CNN
+F 2 "KiCad:XZMDKCBDDG45S9" H 8300 2350 50  0001 C CNN
 F 3 "~" H 8300 2350 50  0001 C CNN
 	1    8300 2400
@@
 F 0 "D92" H 8900 2897 50  0000 C CNN
 F 1 "LED_RABG" H 8900 2806 50  0000 C CNN
-F 2 "" H 8900 2350 50  0001 C CNN
+F 2 "KiCad:XZMDKCBDDG45S9" H 8900 2350 50  0001 C CNN
 F 3 "~" H 8900 2350 50  0001 C CNN
 	1    8900 2400
@@
 F 0 "D94" H 9500 2897 50  0000 C CNN
 F 1 "LED_RABG" H 9500 2806 50  0000 C CNN
-F 2 "" H 9500 2350 50  0001 C CNN
+F 2 "KiCad:XZMDKCBDDG45S9" H 9500 2350 50  0001 C CNN
 F 3 "~" H 9500 2350 50  0001 C CNN
 	1    9500 2400
@@
 F 0 "D96" H 10100 2897 50  0000 C CNN
 F 1 "LED_RABG" H 10100 2806 50  0000 C CNN
-F 2 "" H 10100 2350 50  0001 C CNN
+F 2 "KiCad:XZMDKCBDDG45S9" H 10100 2350 50  0001 C CNN
 F 3 "~" H 10100 2350 50  0001 C CNN
 	1    10100 2400
@@
 F 0 "D97" H 10100 3947 50  0000 C CNN
 F 1 "LED_RABG" H 10100 3856 50  0000 C CNN
-F 2 "" H 10100 3400 50  0001 C CNN
+F 2 "KiCad:XZMDKCBDDG45S9" H 10100 3400 50  0001 C CNN
 F 3 "~" H 10100 3400 50  0001 C CNN
 	1    10100 3450
@@
 F 0 "D95" H 9500 3947 50  0000 C CNN
 F 1 "LED_RABG" H 9500 3856 50  0000 C CNN
-F 2 "" H 9500 3400 50  0001 C CNN
+F 2 "KiCad:XZMDKCBDDG45S9" H 9500 3400 50  0001 C CNN
 F 3 "~" H 9500 3400 50  0001 C CNN
 	1    9500 3450
@@
 F 0 "D93" H 8900 3947 50  0000 C CNN
 F 1 "LED_RABG" H 8900 3856 50  0000 C CNN
-F 2 "" H 8900 3400 50  0001 C CNN
+F 2 "KiCad:XZMDKCBDDG45S9" H 8900 3400 50  0001 C CNN
 F 3 "~" H 8900 3400 50  0001 C CNN
 	1    8900 3450
@@
 F 0 "D91" H 8300 3947 50  0000 C CNN
 F 1 "LED_RABG" H 8300 3856 50  0000 C CNN
-F 2 "" H 8300 3400 50  0001 C CNN
+F 2 "KiCad:XZMDKCBDDG45S9" H 8300 3400 50  0001 C CNN
 F 3 "~" H 8300 3400 50  0001 C CNN
 	1    8300 3450
@@
 F 0 "D89" H 7700 3947 50  0000 C CNN
 F 1 "LED_RABG" H 7700 3856 50  0000 C CNN
-F 2 "" H 7700 3400 50  0001 C CNN
+F 2 "KiCad:XZMDKCBDDG45S9" H 7700 3400 50  0001 C CNN
 F 3 "~" H 7700 3400 50  0001 C CNN
 	1    7700 3450
@@
 F 0 "D87" H 7100 3947 50  0000 C CNN
 F 1 "LED_RABG" H 7100 3856 50  0000 C CNN
-F 2 "" H 7100 3400 50  0001 C CNN
+F 2 "KiCad:XZMDKCBDDG45S9" H 7100 3400 50  0001 C CNN
 F 3 "~" H 7100 3400 50  0001 C CNN
 	1    7100 3450
@@
 F 0 "D85" H 6500 3947 50  0000 C CNN
 F 1 "LED_RABG" H 6500 3856 50  0000 C CNN
-F 2 "" H 6500 3400 50  0001 C CNN
+F 2 "KiCad:XZMDKCBDDG45S9" H 6500 3400 50  0001 C CNN
 F 3 "~" H 6500 3400 50  0001 C CNN
 	1    6500 3450
@@
 F 0 "D83" H 5900 3947 50  0000 C CNN
 F 1 "LED_RABG" H 5900 3856 50  0000 C CNN
-F 2 "" H 5900 3400 50  0001 C CNN
+F 2 "KiCad:XZMDKCBDDG45S9" H 5900 3400 50  0001 C CNN
 F 3 "~" H 5900 3400 50  0001 C CNN
 	1    5900 3450
@@
 F 0 "D80" H 4700 3947 50  0000 C CNN
 F 1 "LED_RABG" H 4700 3856 50  0000 C CNN
-F 2 "" H 4700 3400 50  0001 C CNN
+F 2 "KiCad:XZMDKCBDDG45S9" H 4700 3400 50  0001 C CNN
 F 3 "~" H 4700 3400 50  0001 C CNN
 	1    4700 3450
@@
 F 0 "D78" H 4100 3947 50  0000 C CNN
 F 1 "LED_RABG" H 4100 3856 50  0000 C CNN
-F 2 "" H 4100 3400 50  0001 C CNN
+F 2 "KiCad:XZMDKCBDDG45S9" H 4100 3400 50  0001 C CNN
 F 3 "~" H 4100 3400 50  0001 C CNN
 	1    4100 3450
@@
 F 0 "D76" H 3550 3947 50  0000 C CNN
 F 1 "LED_RABG" H 3550 3856 50  0000 C CNN
-F 2 "" H 3550 3400 50  0001 C CNN
+F 2 "KiCad:XZMDKCBDDG45S9" H 3550 3400 50  0001 C CNN
 F 3 "~" H 3550 3400 50  0001 C CNN
 	1    3550 3450
@@
 F 0 "D74" H 2950 3947 50  0000 C CNN
 F 1 "LED_RABG" H 2950 3856 50  0000 C CNN
-F 2 "" H 2950 3400 50  0001 C CNN
+F 2 "KiCad:XZMDKCBDDG45S9" H 2950 3400 50  0001 C CNN
 F 3 "~" H 2950 3400 50  0001 C CNN
 	1    2950 3450
@@
 F 0 "D72" H 2350 3947 50  0000 C CNN
 F 1 "LED_RABG" H 2350 3856 50  0000 C CNN
-F 2 "" H 2350 3400 50  0001 C CNN
+F 2 "KiCad:XZMDKCBDDG45S9" H 2350 3400 50  0001 C CNN
 F 3 "~" H 2350 3400 50  0001 C CNN
 	1    2350 3450
@@
 F 0 "D70" H 1750 3947 50  0000 C CNN
 F 1 "LED_RABG" H 1750 3856 50  0000 C CNN
-F 2 "" H 1750 3400 50  0001 C CNN
+F 2 "KiCad:XZMDKCBDDG45S9" H 1750 3400 50  0001 C CNN
 F 3 "~" H 1750 3400 50  0001 C CNN
 	1    1750 3450
