File: hardware/PCB/keyboard.kicad_pcb (KiCad board)
At the start: 2 copper layers, 282.7 x 117.3 mm, 263 parts, among them J1 USB_B_Micro, SW1 SW_DIP_x01, U1 STM32F303CCTx, U2 IS31FL3733-QF, U3 IS31FL3733-QF, U4 LD3985M33R, Y1 YSX530GA

Commit message: PCB is done??
Parts:
- removed TP3, TP4: TestPoint, TestPoint:TestPoint_Pad_D1.0mm
- J1: moved to F.Cu
- R26, R27, U1: moved to B.Cu
- SW1: footprint Button_Switch_SMD:SW_SPST_EVQPE1 -> Button_Switch_SMD:SW_SPST_B3U-1000P
- moved TP1 243.2 mm to (352.7, 92.2)
- moved TP2 234.7 mm to (339.6, 92.1)
- moved TP5 231.8 mm to (352.7, 95.4)
- moved R25 180.0 mm to (332.6, 93.9), turned to 90 degrees
- moved SW1 178.7 mm to (310.4, 100.1), turned to 180 degrees
- moved R32 177.3 mm to (328.3, 93.6), turned to 180 degrees
- moved C24 177.1 mm to (349.6, 93.8), turned to 90 degrees
- moved C25 176.5 mm to (348.6, 93.9), turned to 90 degrees
- moved R30 173.3 mm to (326.8, 92.6), turned to 90 degrees
- moved R31 172.9 mm to (325.8, 91.7), turned to 270 degrees
- moved R33 171.2 mm to (328.3, 94.6)
- moved C26 171.2 mm to (347.6, 93.9), turned to 90 degrees
- moved C27 170.6 mm to (346.6, 93.9), turned to 90 degrees
- moved C22 161.3 mm to (304.5, 90.2)
- moved Y1 159.3 mm to (303.1, 92.6)
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Connections:
- R25 pad 1: /SMT32/USB_D- -> /SMT32/USB_D+
- U1 pad 10: /SMT32/ROW1 -> /SMT32/COL4
- U1 pad 11: /SMT32/ROW2 -> /SMT32/COL5
- U1 pad 12: /SMT32/ROW3 -> /SMT32/COL6
- U1 pad 13: /SMT32/ROW4 -> /SMT32/COL7
- U1 pad 14: /SMT32/ROW5 -> /SMT32/COL8
- U1 pad 15: Net-(U1-Pad15) -> /SMT32/COL9
- U1 pad 16: Net-(U1-Pad16) -> /SMT32/COL10
- U1 pad 17: Net-(U1-Pad17) -> /SMT32/COL11
- U1 pad 18: /SMT32/COL14 -> /SMT32/COL12
- U1 pad 20: /SMT32/COL12 -> /SMT32/COL14
- U1 pad 21: /SMT32/COL4 -> /SMT32/COL2
- U1 pad 22: /SMT32/COL3 -> /SMT32/COL1
- U1 pad 25: /SMT32/COL2 -> Net-(U1-Pad25)
- U1 pad 26: /SMT32/COL1 -> Net-(U1-Pad26)
- U1 pad 27: /RGB/LED_EN_PIN -> Net-(U1-Pad27)
- U1 pad 34: Net-(U1-Pad34) -> /RGB/LED_EN_PIN
- U1 pad 37: Net-(U1-Pad37) -> /SMT32/ROW1
- U1 pad 38: Net-(U1-Pad38) -> /SMT32/ROW2
- U1 pad 39: /SMT32/COL11 -> /SMT32/ROW3
- U1 pad 40: /SMT32/COL10 -> /SMT32/ROW4
- U1 pad 41: /SMT32/COL9 -> /SMT32/ROW5
- U1 pad 42: /SMT32/COL8 -> Net-(U1-Pad42)
- U1 pad 43: /SMT32/COL7 -> Net-(U1-Pad43)
- U1 pad 45: /SMT32/COL6 -> Net-(U1-Pad45)
- U1 pad 46: /SMT32/COL5 -> /SMT32/COL3
Routing:
- net +3V3: track 0.00 -> 451.7 mm, vias 0 -> 8
- net GND: track 30.2 -> 466.2 mm, vias 0 -> 9
- net /SMT32/ROW5: track 0.00 -> 407.5 mm, vias 0 -> 2
- net /SMT32/ROW4: track 0.00 -> 376.7 mm, vias 0 -> 3
- net /SMT32/ROW3: track 0.00 -> 343.1 mm, vias 0 -> 2
- net /SMT32/ROW2: track 0.00 -> 336.9 mm, vias 0 -> 2
- net /RGB/RGBmatrix/ROW3: track 0.00 -> 324.6 mm, vias 0 -> 2
- net /SMT32/COL14: track 1.02 -> 324.5 mm, vias 1 -> 5
- net /SMT32/ROW1: track 0.00 -> 317.2 mm, vias 0 -> 2
- net /RGB/RGBmatrix/ROW1: track 0.00 -> 311.4 mm, vias 0 -> 2
- net /RGB/RGBmatrix/ROW2: track 0.00 -> 308.5 mm, vias 0 -> 28
- net /RGB/RGBmatrix2/ROW3: track 0.00 -> 306.1 mm, vias 0 -> 2
- net /SMT32/COL13: track 0.00 -> 304.3 mm, vias 0 -> 6
- net /RGB/RGBmatrix/ROW6: track 0.00 -> 303.7 mm, vias 0 -> 2
- net /RGB/RGBmatrix/COL2: track 0.00 -> 303.0 mm, vias 0 -> 4
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- added copper zone on B.Cu, net GND
- added copper zone on F.Cu, net GND
