File: hardware/PCB/keyboard.kicad_pcb (KiCad board)
At the start: 2 copper layers, 282.7 x 117.3 mm, 261 parts, among them J1 USB_B_Micro, SW1 SW_DIP_x01, U1 STM32F303CCTx, U2 IS31FL3733-QF, U3 IS31FL3733-QF, U4 LD3985M33R, Y1 YSX530GA

Commit message: Making progress, so many distance warning!!!
Parts:
- removed the C10 at (186.9, 193.0)
- removed the C18 at (341.5, 93.1)
- removed the C19 at (344.9, 90.3)
- removed the C20 at (344.9, 92.2)
- removed the D96 at (344.9, 94.3)
- removed TP1, TP2, TP5: TestPoint, TestPoint:TestPoint_Pad_D1.0mm
- removed the U4 at (342.0, 91.2)
- added C21: 22uf, Capacitor_SMD:C_0402_1005Metric, F.Cu at (128.1, 72.6)
- added C26: 100nF, Capacitor_SMD:C_0402_1005Metric, F.Cu at (128.8, 96.8)
- added C9: 22μF/10V, Capacitor_Tantalum_SMD:CP_EIA-3216-18_Kemet-A, F.Cu at (262.4, 188.6)
- added SW2: SW_DIP_x01, Button_Switch_SMD:SW_SPST_B3U-1000P, F.Cu at (129.7, 79.8)
- added U3: AZ1117CH-3.3, Package_TO_SOT_SMD:SOT-223-3_TabPin2, F.Cu at (110.0, 93.5)
- C1: renamed from C3; moved to F.Cu
- C10: renamed from C11; value 0.47μF -> 470nF; moved to F.Cu
- C11: renamed from C12; value 0.1μF -> 100nF; moved to F.Cu
- C12: renamed from C13; value 0.47μF -> 470nF; moved to F.Cu
- C13: renamed from C14; value 0.1μF -> 100nF; moved to F.Cu
- C14: renamed from C15; value 0.47μF -> 470nF; moved to F.Cu
- C15: renamed from C16; value 0.1μF -> 100nF; moved to F.Cu
- C16: renamed from C2; value 0.47μF -> 470nF; moved to F.Cu
- C17: value 1μF -> 10uf; moved to F.Cu
- C18: renamed from C24; value 0.1μF -> 100nF; moved to F.Cu
- C19: renamed from C25; value 0.1μF -> 100nF; moved to F.Cu
- C2: renamed from C1; value 0.47μF -> 470nF; moved to F.Cu
- C20: renamed from C26; value 0.1μF -> 100nF; moved to F.Cu
- C22: renamed from C27; value 0.1μF -> 100nF; moved to F.Cu
- C23: renamed from C21; moved to F.Cu
- C24: renamed from C22; moved to F.Cu
- C25: renamed from C23; value 1μF -> 100nF; moved to F.Cu
- C3: renamed from C4; value 0.47μF -> 470nF; moved to F.Cu
- C4: renamed from C5; value 0.1μF -> 100nF; moved to F.Cu
- C5: renamed from C6; value 0.47μF -> 470nF; moved to F.Cu
- C6: renamed from C7; value 0.1μF -> 100nF; moved to F.Cu
- C7: renamed from C8; value 0.47μF -> 470nF; moved to F.Cu
- C8: renamed from C9; value 0.1μF -> 100nF; moved to F.Cu
- CherryMX1, CherryMX10, CherryMX11, CherryMX12, CherryMX13, CherryMX14, CherryMX15, CherryMX16, CherryMX17, CherryMX18, CherryMX19, CherryMX2, CherryMX20, CherryMX21, CherryMX22, CherryMX23, CherryMX24, CherryMX25, CherryMX26, CherryMX27, CherryMX28, CherryMX29, CherryMX3, CherryMX30, CherryMX31, CherryMX32, CherryMX33, CherryMX34, CherryMX35, CherryMX36, CherryMX37, CherryMX38, CherryMX39, CherryMX4, CherryMX40, CherryMX41, CherryMX42, CherryMX43, CherryMX44, CherryMX45, CherryMX46, CherryMX47, CherryMX48, CherryMX49, CherryMX5, CherryMX50, CherryMX51, CherryMX52, CherryMX53, CherryMX54, CherryMX55, CherryMX56, CherryMX57, CherryMX58, CherryMX59, CherryMX6, CherryMX60, CherryMX61, CherryMX62, CherryMX63, CherryMX64, CherryMX65, CherryMX66, CherryMX67, CherryMX68, CherryMX7, CherryMX8, CherryMX9: moved to B.Cu
- D1, D10, D11, D12, D13, D14, D15, D16, D17, D18, D19, D2, D20, D21, D22, D23, D24, D25, D26, D27, D28, D29, D3, D30, D31, D32, D33, D34, D35, D36, D37, D38, D39, D4, D40, D41, D42, D43, D44, D45, D46, D47, D48, D49, D5, D50, D51, D52, D53, D54, D55, D56, D57, D58, D59, D6, D60, D61, D62, D63, D64, D65, D66, D67, D68, D69, D7, D70, D71, D72, D73, D74, D75, D76, D77, D78, D79, D8, D80, D81, D82, D83, D84, D85, D86, D87, D88, D89, D9, D90, D91, D92, D93, D94, D95, SW1: moved to F.Cu
- D100: renamed from D102; moved to F.Cu
- D101: renamed from D103; moved to F.Cu
- D102: renamed from D104; moved to F.Cu
- D103: renamed from D105; moved to F.Cu
- D104: renamed from D106; moved to F.Cu
- D105: renamed from D107; moved to F.Cu
- D106: renamed from D108; moved to F.Cu
- D107: renamed from D109; moved to F.Cu
- D108: renamed from D110; moved to F.Cu
- D109: renamed from D111; moved to F.Cu
- D110: renamed from D112; moved to F.Cu
- D111: renamed from D113; moved to F.Cu
- D112: renamed from D114; moved to F.Cu
- D113: renamed from D115; moved to F.Cu
- D114: renamed from D116; moved to F.Cu
- D115: renamed from D117; moved to F.Cu
- D116: renamed from D118; moved to F.Cu
- D117: renamed from D119; moved to F.Cu
- D118: renamed from D120; moved to F.Cu
- D119: renamed from D121; moved to F.Cu
- D120: renamed from D122; moved to F.Cu
- D121: renamed from D123; moved to F.Cu
- D122: renamed from D124; moved to F.Cu
- D123: renamed from D125; moved to F.Cu
- D124: renamed from D126; moved to F.Cu
- D125: renamed from D127; moved to F.Cu
- D126: renamed from D128; moved to F.Cu
- D127: renamed from D129; moved to F.Cu
- D128: renamed from D130; moved to F.Cu
- D129: renamed from D131; moved to F.Cu
- D130: renamed from D132; moved to F.Cu
- D131: renamed from D133; moved to F.Cu
- D132: renamed from D134; moved to F.Cu
- D133: renamed from D135; moved to F.Cu
- D134: renamed from D136; moved to F.Cu
- D135: renamed from D137; moved to F.Cu
- D136: renamed from D138; moved to F.Cu
- D96: renamed from D98; moved to F.Cu
- D97: renamed from D99; moved to F.Cu
- D98: renamed from D100; moved to F.Cu
- D99: renamed from D101; moved to F.Cu
- R1: renamed from R23; moved to F.Cu
- R10: renamed from R24; moved to F.Cu
- R11: renamed from R25; moved to F.Cu
- R12: renamed from R28; moved to F.Cu
- R13: renamed from R29; moved to F.Cu
- R14: renamed from R26; moved to F.Cu
- R15: renamed from R27; moved to F.Cu
- R16: renamed from R30; moved to F.Cu
- R17: renamed from R31; moved to F.Cu
- R18: renamed from R32; moved to F.Cu
- R19: renamed from R33; moved to F.Cu
- R2: renamed from R16; moved to F.Cu
- R3: renamed from R17; moved to F.Cu
- R4: renamed from R18; moved to F.Cu
- R5: renamed from R19; moved to F.Cu
- R6: renamed from R20; moved to F.Cu
- R7: renamed from R21; moved to F.Cu
- R8: renamed from R15; moved to F.Cu
- R9: renamed from R22; moved to F.Cu
- U1: renamed from U2; moved to F.Cu
- U2: renamed from U3; moved to F.Cu
- U4: renamed from U1; moved to F.Cu
- Y1: value YSX530GA -> X50328MSB2GI; moved to F.Cu
- moved C3 265.5 mm to (87.0, 159.5), turned to 0 degrees
- moved C4 265.5 mm to (87.0, 158.5), turned to 0 degrees
- moved C5 265.5 mm to (87.0, 157.5), turned to 0 degrees
- moved C6 265.5 mm to (87.0, 156.5), turned to 0 degrees
- moved C7 265.5 mm to (87.0, 155.4), turned to 0 degrees
- moved C8 265.5 mm to (87.0, 154.4), turned to 0 degrees
- moved C1 263.8 mm to (87.6, 149.8), turned to 90 degrees
- moved D1 263.0 mm to (356.4, 109.4)
- moved D2 263.0 mm to (356.4, 128.4)
- moved D3 263.0 mm to (356.4, 147.5)
- moved D4 263.0 mm to (356.4, 166.5)
- moved D5 263.0 mm to (356.4, 185.6)
- moved R5 261.6 mm to (94.1, 142.4), turned to 180 degrees
- moved R3 260.8 mm to (94.6, 148.6)
- moved C2 258.8 mm to (93.6, 144.9), turned to 180 degrees
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Connections:
- R14 pad 1: Net-(R26-Pad1) -> Net-(R14-Pad1)
- R15 pad 2: Net-(R27-Pad2) -> Net-(R15-Pad2)
- U4 pad 32: Net-(R27-Pad2) -> Net-(R14-Pad1)
- U4 pad 33: Net-(R26-Pad1) -> Net-(R15-Pad2)
Routing:
- net +3V3: track 451.7 -> 253.7 mm
- net GND: track 466.2 -> 299.5 mm, vias 9 -> 8
- net /RGB/RGBmatrix2/ROW4: track 156.8 -> 277.3 mm
- net /RGB/RGBmatrix2/ROW6: track 173.4 -> 284.9 mm, vias 4 -> 2
- net /RGB/RGBmatrix2/ROW5: track 189.9 -> 275.8 mm, vias 18 -> 26
- net /SMT32/I2C2_SDA: track 278.7 -> 194.0 mm, vias 8 -> 5
- net /SMT32/I2C2_SCL: track 285.1 -> 201.0 mm, vias 7 -> 4
- net /SMT32/COL1: track 124.1 -> 105.9 mm, vias 7 -> 5
- net /SMT32/COL3: track 106.6 -> 91.3 mm, vias 6 -> 5
- net /SMT32/COL5: track 145.5 -> 158.9 mm
- net /SMT32/COL2: track 119.5 -> 108.0 mm, vias 6 -> 5
- net Net-(C25-Pad2): track 9.27 -> 17.0 mm
- net /RGB/SYNC: track 184.5 -> 177.1 mm, vias 2 -> 1
- net /RGB/RGBmatrix/ROW6: track 303.7 -> 296.7 mm
- net Net-(C23-Pad2): track 16.1 -> 9.21 mm
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
Commit message: Rotate the RGB controller. gonna have a lot of work to do
Parts:
- moved C21 26.7 mm to (114.2, 95.4), turned to 90 degrees
- moved SW2 19.4 mm to (123.7, 98.2), turned to 0 degrees
- moved C17 12.3 mm to (109.0, 88.3)
- moved R1 10.3 mm to (91.2, 150.8)
- moved R5 10.2 mm to (89.1, 133.5)
- moved R3 8.68 mm to (87.0, 144.3)
- moved R4 8.68 mm to (88.0, 144.3)
- moved C2 7.27 mm to (87.6, 140.8)
- moved R2 6.38 mm to (97.4, 149.4)
- moved R7 3.64 mm to (223.4, 191.7)
- moved R6 3.60 mm to (222.4, 191.7)
- moved U2 2.61 mm to (230.6, 185.0), turned to 135 degrees
- moved R8 1.88 mm to (226.0, 191.3)
- moved C26 1.82 mm to (127.5, 95.5), turned to 90 degrees
- moved U1 0.91 mm to (98.3, 140.7), turned to 45 degrees
Routing:
- net /RGB/LED_EN_PIN: track 275.9 -> 0.00 mm, vias 2 -> 0
- net /RGB/RGBmatrix/COL1: track 302.3 -> 46.1 mm
- net /RGB/RGBmatrix/COL2: track 303.0 -> 65.2 mm
- net /RGB/RGBmatrix/COL3: track 265.6 -> 46.1 mm
- net /RGB/RGBmatrix/COL4: track 247.2 -> 46.1 mm
- net /SMT32/I2C2_SCL: track 201.0 -> 0.00 mm, vias 4 -> 0
- net /SMT32/I2C2_SDA: track 194.0 -> 0.32 mm, vias 5 -> 0
- net +3V3: track 253.7 -> 60.7 mm, vias 8 -> 0
- net GND: track 299.5 -> 107.4 mm, vias 8 -> 3
- net /RGB/RGBmatrix/COL5: track 229.6 -> 46.1 mm
- net /RGB/SYNC: track 177.1 -> 0.00 mm, vias 1 -> 0
- net /RGB/RGBmatrix/COL6: track 211.3 -> 46.1 mm
- net /RGB/RGBmatrix/COL7: track 192.7 -> 46.1 mm
- net /RGB/RGBmatrix2/COL1: track 162.3 -> 24.4 mm, vias 3 -> 2
- net /RGB/RGBmatrix/COL8: track 174.4 -> 46.1 mm
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
Commit message: getting closer to it actually works
Parts:
- removed C21: 22uf, Capacitor_SMD:C_0402_1005Metric
- removed C9: 22μF/10V, Capacitor_Tantalum_SMD:CP_EIA-3216-18_Kemet-A
- moved C1 61.6 mm to (114.8, 94.5)
- moved C11 33.7 mm to (227.8, 180.9), turned to 135 degrees
- moved C10 33.2 mm to (227.1, 181.6), turned to 135 degrees
- moved C15 32.6 mm to (224.7, 181.6), turned to 45 degrees
- moved C14 29.9 mm to (226.1, 182.9), turned to 45 degrees
- moved C16 29.8 mm to (225.4, 182.2), turned to 225 degrees
- moved C7 25.1 mm to (103.8, 136.8), turned to 45 degrees
- moved C3 25.1 mm to (96.7, 136.4), turned to 135 degrees
- moved C4 25.0 mm to (97.4, 135.7), turned to 135 degrees
- moved C12 25.0 mm to (234.8, 180.6), turned to 135 degrees
- moved C13 24.5 mm to (234.1, 181.3), turned to 135 degrees
- moved C8 24.4 mm to (103.1, 136.1), turned to 45 degrees
- moved R18 18.3 mm to (119.5, 98.0)
- moved R19 18.3 mm to (119.5, 99.0)
- moved C5 17.8 mm to (101.3, 146.7), turned to 225 degrees
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Routing:
- net +3V3: track 60.7 -> 370.1 mm, vias 0 -> 8
- net /RGB/LED_EN_PIN: track 0.00 -> 292.6 mm, vias 0 -> 4
- net /SMT32/I2C2_SCL: track 0.00 -> 285.0 mm, vias 0 -> 5
- net /SMT32/I2C2_SDA: track 0.32 -> 279.7 mm, vias 0 -> 5
- net /RGB/SYNC: track 0.00 -> 202.7 mm
- net GND: track 107.4 -> 167.4 mm, vias 3 -> 5
- net Net-(R16-Pad1): track 0.00 -> 18.5 mm, vias 0 -> 2
- net Net-(R17-Pad2): track 1.32 -> 19.1 mm, vias 0 -> 2
- net /SMT32/COL1: track 116.0 -> 123.9 mm, vias 5 -> 6
- net /RGB/RGBmatrix2/COL8: track 27.1 -> 23.6 mm, vias 3 -> 2
- net Net-(R12-Pad2): track 10.1 -> 13.0 mm
- net /SMT32/ROW5: track 398.8 -> 401.2 mm
- net /SMT32/USB_D+: track 17.3 -> 15.3 mm
- net /SMT32/USB_D-: track 15.3 -> 13.3 mm
- net Net-(R8-Pad1): track 0.00 -> 1.48 mm
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- removed copper zone on B.Cu, net GND
- removed copper zone on F.Cu, net GND

Commit message: Use the correct Footprint
I think I can't do more things before the parts arrive and figure out what LED im going to use
Parts:
- removed the R1 at (91.2, 150.8)
- removed the R10 at (229.3, 190.6)
- added R14: 100k, Resistor_SMD:R_0402_1005Metric, F.Cu at (123.2, 94.8)
- U3: value AZ1117CH-3.3 -> AZ1117-3.3
- moved R4 12.9 mm to (101.0, 135.9), turned to 45 degrees
- moved C10 1.15 mm to (234.5, 181.7), turned to 315 degrees
- moved C11 1.15 mm to (235.2, 181.0), turned to 315 degrees
- renumbered C2 to C1, C12 to C10, C13 to C11, C14 to C12, C15 to C13, C16 to C14, C18 to C15, C17 to C16, C19 to C17, C20 to C18, C1 to C19, C3 to C2, C22 to C20, C26 to C21, C23 to C22, C24 to C23, C25 to C24, C4 to C3, C5 to C4, C6 to C5, C7 to C6, C8 to C7, C10 to C8, C11 to C9, R2 to R1, R12 to R10, R13 to R11, R14 to R12, R15 to R13, R16 to R15, R17 to R16, R18 to R17, R19 to R18, R3 to R2, R4 to R3, R5 to R4, R6 to R5, R7 to R6, R8 to R7, R9 to R8, R11 to R9
Routing:
- net +3V3: track 370.1 -> 391.6 mm, vias 8 -> 12
- net /RGB/RGBmatrix2/COL14: track 39.0 -> 25.9 mm
- net /RGB/RGBmatrix2/COL12: track 37.3 -> 24.4 mm
- net GND: track 167.4 -> 178.1 mm, vias 5 -> 6
- net /RGB/RGBmatrix/COL14: track 30.3 -> 23.7 mm, vias 3 -> 2
- net /RGB/LED_EN_PIN: track 292.6 -> 297.1 mm, vias 4 -> 5
- net Net-(R4-Pad1): track 0.00 -> 1.73 mm
- net /SMT32/ROW5: track 401.2 -> 400.4 mm
- added copper zone on B.Cu, net GND
- added copper zone on F.Cu, net GND

Commit message: alot of changes
modify the QFN-48 so PCB 3d view in future would look better (so I don't design a part that doesn't fit)
I made a useless QFN-40 3d model
modify schematics so it looks better
Parts:
- U1, U2: footprint Package_DFN_QFN:QFN-48-1EP_6x6mm_P0.4mm_EP4.2x4.2mm_ThermalVias -> KiCad:QFN-48-1EP_6x6mm_P0.4mm_EP4.2x4.2mm_ThermalVias
- U4: value STM32F303CCTx -> STM32F303CCT6
- moved R5 0.22 mm to (225.2, 186.8)
- moved R6 0.22 mm to (226.2, 186.8)
- turned R12 to 0 degrees
Connections:
- R12 pad 1: Net-(R12-Pad1) -> /SMT32/USB_D-
- R12 pad 2: /SMT32/USB_D- -> Net-(R12-Pad2)
- U4 pad 32: Net-(R12-Pad1) -> Net-(R12-Pad2)
Routing:
- net +3V3: track 391.6 -> 403.4 mm, vias 12 -> 8
- net GND: track 178.1 -> 181.4 mm
- net /SMT32/I2C2_SCL: track 285.0 -> 282.5 mm
- net Net-(R12-Pad2): track 0.00 -> 2.13 mm
- net Net-(R12-Pad1): track 2.13 -> 0.00 mm
- net /RGB/SYNC: track 202.7 -> 203.7 mm
- net /SMT32/I2C2_SDA: track 279.7 -> 279.2 mm
- net /RGB/RGBmatrix/COL9: vias 4 -> 3
- net /RGB/RGBmatrix/COL8: vias 4 -> 3
- net /RGB/RGBmatrix/COL7: vias 4 -> 3
- net /RGB/RGBmatrix/COL6: vias 4 -> 3
- net /RGB/RGBmatrix/COL5: vias 4 -> 3
- net /RGB/RGBmatrix/COL4: vias 4 -> 3
- net /RGB/RGBmatrix/COL3: vias 4 -> 3
- net /RGB/RGBmatrix/COL2: vias 4 -> 3
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
Commit message: Clear the errors
Parts:
- moved C5 2.55 mm to (103.4, 145.4)
- moved C4 2.55 mm to (102.7, 144.6)
Routing:
- net /RGB/RGBmatrix2/ROW5: track 260.9 -> 200.2 mm, vias 24 -> 18
- net /RGB/RGBmatrix/ROW3: track 270.8 -> 288.7 mm
- net +3V3: track 403.4 -> 416.0 mm, vias 8 -> 6
- net /SMT32/ROW3: track 343.1 -> 353.1 mm
- net /RGB/RGBmatrix/ROW6: track 264.5 -> 269.2 mm
- net /RGB/RGBmatrix2/ROW6: track 268.3 -> 271.0 mm
- net /SMT32/ROW5: track 400.6 -> 398.0 mm
- net /SMT32/COL9: track 230.5 -> 228.5 mm
- net /RGB/SYNC: track 203.7 -> 204.6 mm
- net /RGB/RGBmatrix2/ROW3: track 265.2 -> 264.4 mm
- net GND: track 181.4 -> 181.9 mm

Commit message: Connecting RGBs
Parts:
- moved C5 4.30 mm to (106.3, 142.2), turned to 0 degrees
- moved C4 3.89 mm to (106.3, 143.2), turned to 0 degrees
- moved C6 1.16 mm to (104.5, 137.8)
- moved C7 1.16 mm to (103.8, 137.1)
- moved R4 0.73 mm to (101.6, 136.3), turned to 315 degrees
Connections:
- U1 pad 10: /RGB/RGBmatrix/ROW2 -> /RGB/RGBmatrix/ROW5
- U1 pad 11: /RGB/RGBmatrix/ROW1 -> /RGB/RGBmatrix/ROW6
- U1 pad 13: Net-(U1-Pad13) -> /RGB/RGBmatrix/ROW7
- U1 pad 14: Net-(U1-Pad14) -> /RGB/RGBmatrix/ROW8
- U1 pad 15: Net-(U1-Pad15) -> /RGB/RGBmatrix/ROW9
- U1 pad 2: /RGB/RGBmatrix/ROW9 -> Net-(U1-Pad2)
- U1 pad 3: /RGB/RGBmatrix/ROW8 -> Net-(U1-Pad3)
- U1 pad 4: /RGB/RGBmatrix/ROW7 -> Net-(U1-Pad4)
- U1 pad 6: /RGB/RGBmatrix/ROW6 -> /RGB/RGBmatrix/ROW1
- U1 pad 7: /RGB/RGBmatrix/ROW5 -> /RGB/RGBmatrix/ROW2
- U1 pad 8: /RGB/RGBmatrix/ROW4 -> /RGB/RGBmatrix/ROW3
- U1 pad 9: /RGB/RGBmatrix/ROW3 -> /RGB/RGBmatrix/ROW4
Routing:
- net /RGB/RGBmatrix/ROW9: track 253.5 -> 805.6 mm, vias 0 -> 2
- net /RGB/RGBmatrix/COL1: track 46.1 -> 309.2 mm, vias 3 -> 5
- net /RGB/RGBmatrix/COL2: track 65.2 -> 307.1 mm, vias 3 -> 6
- net /RGB/RGBmatrix/COL3: track 46.1 -> 268.8 mm, vias 3 -> 6
- net /RGB/RGBmatrix/COL4: track 46.1 -> 249.7 mm, vias 3 -> 6
- net /RGB/RGBmatrix/COL5: track 46.1 -> 230.0 mm, vias 3 -> 6
- net /RGB/RGBmatrix/COL6: track 46.1 -> 211.3 mm, vias 3 -> 6
- net /RGB/RGBmatrix/COL7: track 46.1 -> 191.1 mm, vias 3 -> 6
- net /RGB/RGBmatrix/COL8: track 46.1 -> 171.2 mm, vias 3 -> 6
- net /RGB/RGBmatrix/COL9: track 46.1 -> 151.8 mm, vias 3 -> 6
- net /RGB/RGBmatrix/COL10: track 46.1 -> 133.5 mm, vias 3 -> 6
- net GND: track 181.9 -> 106.7 mm, vias 6 -> 7
- net /RGB/RGBmatrix/COL11: track 46.1 -> 114.4 mm, vias 3 -> 6
- net /RGB/RGBmatrix/ROW3: track 288.7 -> 350.2 mm, vias 0 -> 2
- net /RGB/RGBmatrix/ROW2: track 262.8 -> 315.4 mm, vias 26 -> 28
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