File: hardware/PCB/keyboard.kicad_pcb (KiCad board)
At the start: 2 copper layers, 282.7 x 117.3 mm, 254 parts, among them J1 USB_B_Micro, SW1 SW_DIP_x01, SW2 SW_DIP_x01, U1 IS31FL3733-QF, U2 IS31FL3733-QF, U3 AZ1117-3.3, U4 STM32F303CCT6, Y1 X50328MSB2GI

Commit message: I guess it is done, maybe just make it?
Parts:
- moved C10 0.79 mm to (235.0, 181.2)
- moved C11 0.77 mm to (235.7, 180.4)
- renumbered CherryMX1 to Key1, CherryMX10 to Key10, CherryMX11 to Key11, CherryMX12 to Key12, CherryMX13 to Key13, CherryMX14 to Key14, CherryMX15 to Key15, CherryMX16 to Key16, CherryMX17 to Key17, CherryMX18 to Key18, CherryMX19 to Key19, CherryMX2 to Key2, CherryMX20 to Key20, CherryMX21 to Key21, CherryMX22 to Key22, CherryMX23 to Key23, CherryMX24 to Key24, CherryMX25 to Key25, CherryMX26 to Key26, CherryMX27 to Key27, CherryMX28 to Key28, CherryMX29 to Key29, CherryMX3 to Key3, CherryMX30 to Key30, CherryMX31 to Key31, CherryMX32 to Key32, CherryMX33 to Key33, CherryMX34 to Key34, CherryMX35 to Key35, CherryMX36 to Key36, CherryMX37 to Key37, CherryMX38 to Key38, CherryMX39 to Key39, CherryMX4 to Key4, CherryMX40 to Key40, CherryMX41 to Key41, CherryMX42 to Key42, CherryMX43 to Key43, CherryMX44 to Key44, CherryMX45 to Key45, CherryMX46 to Key46, CherryMX47 to Key47, CherryMX48 to Key48, CherryMX49 to Key49, CherryMX5 to Key5, CherryMX50 to Key50, CherryMX51 to Key51, CherryMX52 to Key52, CherryMX53 to Key53, CherryMX54 to Key54, CherryMX55 to Key55, CherryMX56 to Key56, CherryMX57 to Key57, CherryMX58 to Key58, CherryMX59 to Key59, CherryMX6 to Key6, CherryMX60 to Key60, CherryMX61 to Key61, CherryMX62 to Key62, CherryMX63 to Key63, CherryMX64 to Key64, CherryMX65 to Key65, CherryMX66 to Key66, CherryMX67 to Key67, CherryMX68 to Key68, CherryMX7 to Key7, CherryMX8 to Key8, CherryMX9 to Key9
Routing:
- net /RGB/RGBmatrix2/COL1: track 24.4 -> 164.5 mm, vias 2 -> 3
- net /RGB/RGBmatrix2/COL14: track 25.8 -> 164.9 mm
- net /RGB/RGBmatrix2/COL13: track 25.4 -> 146.5 mm, vias 2 -> 3
- net /RGB/RGBmatrix2/COL2: track 24.4 -> 143.1 mm, vias 2 -> 3
- net /RGB/RGBmatrix2/COL3: track 24.4 -> 125.5 mm, vias 2 -> 3
- net /RGB/RGBmatrix2/COL12: track 25.7 -> 126.4 mm
- net /RGB/RGBmatrix2/ROW5: track 200.2 -> 296.4 mm, vias 18 -> 27
- net /RGB/RGBmatrix2/COL4: track 25.5 -> 107.5 mm
- net /RGB/RGBmatrix2/COL11: track 25.9 -> 107.4 mm
- net /RGB/RGBmatrix2/COL10: track 26.1 -> 88.6 mm
- net /RGB/RGBmatrix2/COL5: track 26.5 -> 73.9 mm
- net /RGB/RGBmatrix2/ROW3: track 264.4 -> 309.8 mm, vias 1 -> 2
- net /RGB/RGBmatrix2/ROW4: track 265.3 -> 303.7 mm, vias 0 -> 4
- net /RGB/RGBmatrix2/ROW2: track 262.1 -> 298.7 mm, vias 26 -> 27
- net /RGB/RGBmatrix2/ROW6: track 271.0 -> 301.0 mm, vias 0 -> 4
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
Commit message: making progress
Parts:
- C19: value 22μF/10V -> 22uf; footprint Capacitor_Tantalum_SMD:CP_EIA-3216-18_Kemet-A -> Capacitor_SMD:C_0402_1005Metric
- D1, D10, D11, D12, D13, D14, D15, D16, D17, D18, D19, D2, D20, D21, D22, D23, D24, D25, D26, D27, D28, D29, D3, D30, D31, D32, D33, D34, D35, D36, D37, D38, D39, D4, D40, D41, D42, D43, D44, D45, D46, D47, D48, D49, D5, D50, D51, D52, D53, D54, D55, D56, D57, D58, D59, D6, D60, D61, D62, D63, D64, D65, D66, D67, D68, D7, D8, D9: value 1N4148W -> 1N4148WS
- D100, D101, D102, D103, D104, D105, D106, D107, D108, D109, D110, D111, D112, D113, D114, D115, D116, D117, D118, D119, D120, D121, D122, D123, D124, D125, D126, D127, D128, D129, D130, D131, D132, D133, D134, D135, D136, D69, D70, D71, D72, D73, D74, D75, D76, D77, D78, D79, D80, D81, D82, D83, D84, D85, D86, D87, D88, D89, D90, D91, D92, D93, D94, D95, D96, D97, D98, D99: value LED_RABG -> XZMDKCBDDG45S-9
- J1: value USB_B_Micro -> 473460001; footprint Connector_USB:USB_Micro-B_Molex-105017-0001 -> Connector_USB:USB_Micro-B_Molex_47346-0001
- Key1, Key10, Key11, Key12, Key13, Key14, Key15, Key16, Key17, Key18, Key19, Key2, Key20, Key21, Key22, Key23, Key24, Key25, Key26, Key27, Key28, Key29, Key3, Key30, Key31, Key32, Key33, Key34, Key35, Key36, Key37, Key38, Key39, Key4, Key40, Key41, Key42, Key43, Key44, Key45, Key46, Key47, Key48, Key49, Key5, Key50, Key51, Key52, Key53, Key54, Key55, Key56, Key57, Key58, Key59, Key6, Key60, Key61, Key62, Key63, Key64, Key65, Key66, Key67, Key68, Key7, Key8, Key9: value SW_SPST -> CPG151101S03
- SW1, SW2: value SW_DIP_x01 -> B3U-1000P
- U1, U2: value IS31FL3733-QF -> IS31FL3733-QFLS4-TR
- U3: value AZ1117-3.3 -> AZ1117CH-3.3TRG1
- Y1: value X50328MSB2GI -> 8Mhz20pF
- moved C19 0.88 mm to (114.8, 95.4)
- moved J1 0.08 mm to (115.0, 86.4)
Routing:
- net /RGB/RGBmatrix/ROW1: track 316.0 -> 358.3 mm
- net GND: track 105.7 -> 91.1 mm, vias 7 -> 8
- net +5V: track 12.0 -> 13.4 mm

Commit message: Wiring now have no errors and uses less vias
Parts:
- moved C6 4.06 mm to (101.6, 135.0), turned to 135 degrees
- moved C7 3.21 mm to (100.9, 135.7), turned to 135 degrees
- moved C9 1.86 mm to (226.1, 180.2), turned to 225 degrees
- moved C5 1.53 mm to (107.2, 143.4), turned to 270 degrees
- moved R4 1.44 mm to (100.2, 136.4), turned to 135 degrees
- moved C8 0.74 mm to (226.8, 180.9), turned to 225 degrees
- moved C4 0.24 mm to (106.2, 143.4), turned to 270 degrees
Connections:
- U1 pad 10: /RGB/RGBmatrix/ROW5 -> /RGB/RGBmatrix/ROW2
- U1 pad 11: /RGB/RGBmatrix/ROW6 -> /RGB/RGBmatrix/ROW3
- U1 pad 6: /RGB/RGBmatrix/ROW1 -> /RGB/RGBmatrix/ROW4
- U1 pad 7: /RGB/RGBmatrix/ROW2 -> /RGB/RGBmatrix/ROW5
- U1 pad 8: /RGB/RGBmatrix/ROW3 -> /RGB/RGBmatrix/ROW6
- U1 pad 9: /RGB/RGBmatrix/ROW4 -> /RGB/RGBmatrix/ROW1
Routing:
- net /RGB/RGBmatrix/ROW9: track 806.3 -> 276.0 mm, vias 2 -> 0
- net GND: track 91.1 -> 26.9 mm, vias 8 -> 15
- net /RGB/RGBmatrix/ROW1: track 358.3 -> 317.2 mm, vias 2 -> 0
- net /RGB/LED_EN_PIN: track 303.5 -> 291.1 mm
- net /SMT32/I2C2_SCL: track 283.5 -> 276.7 mm
- net /SMT32/I2C2_SDA: track 280.4 -> 273.9 mm
- net /RGB/RGBmatrix/ROW6: track 312.4 -> 307.6 mm
- net /RGB/RGBmatrix/ROW4: track 297.8 -> 294.2 mm
- net /RGB/RGBmatrix/ROW5: track 296.6 -> 293.0 mm
- net /RGB/RGBmatrix/COL10: track 133.5 -> 130.2 mm, vias 6 -> 4
- net /RGB/RGBmatrix2/COL7: track 29.1 -> 26.1 mm
- net +3V3: track 402.5 -> 405.5 mm, vias 4 -> 7
- net /RGB/RGBmatrix/COL11: track 114.4 -> 111.5 mm, vias 6 -> 4
- net /RGB/RGBmatrix/COL9: track 151.8 -> 148.9 mm, vias 6 -> 4
- net /RGB/RGBmatrix2/COL13: track 146.5 -> 143.7 mm
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
Commit message: minor changes to the LED controller PCB layout, make it much better
Parts:
- moved C8 3.43 mm to (224.1, 183.0), turned to 135 degrees
- moved C12 2.81 mm to (226.9, 180.2), turned to 135 degrees
- moved C9 2.47 mm to (224.8, 182.3), turned to 135 degrees
- moved C4 2.25 mm to (108.3, 144.2)
- moved C5 2.25 mm to (109.4, 144.2)
- moved R7 1.64 mm to (225.7, 184.8), turned to 225 degrees
- moved C10 1.53 mm to (235.0, 179.6), turned to 135 degrees
- moved C14 1.51 mm to (226.2, 180.9), turned to 315 degrees
- moved C11 1.46 mm to (234.3, 180.3), turned to 135 degrees
- moved R6 1.01 mm to (225.3, 187.3), turned to 315 degrees
- moved R5 0.84 mm to (226.0, 186.6), turned to 315 degrees
- moved C13 0.74 mm to (225.5, 181.6), turned to 135 degrees
Connections:
- U2 pad 10: Net-(U2-Pad10) -> /RGB/RGBmatrix2/ROW5
- U2 pad 11: Net-(U2-Pad11) -> /RGB/RGBmatrix2/ROW6
- U2 pad 13: Net-(U2-Pad13) -> /RGB/RGBmatrix2/ROW3
- U2 pad 14: Net-(U2-Pad14) -> /RGB/RGBmatrix2/ROW2
- U2 pad 15: Net-(U2-Pad15) -> /RGB/RGBmatrix2/ROW1
- U2 pad 2: /RGB/RGBmatrix2/ROW6 -> Net-(U2-Pad2)
- U2 pad 3: /RGB/RGBmatrix2/ROW5 -> Net-(U2-Pad3)
- U2 pad 4: /RGB/RGBmatrix2/ROW4 -> Net-(U2-Pad4)
- U2 pad 6: /RGB/RGBmatrix2/ROW3 -> Net-(U2-Pad6)
- U2 pad 7: /RGB/RGBmatrix2/ROW2 -> Net-(U2-Pad7)
- U2 pad 8: /RGB/RGBmatrix2/ROW1 -> Net-(U2-Pad8)
- U2 pad 9: Net-(U2-Pad9) -> /RGB/RGBmatrix2/ROW4
Routing:
- net /RGB/RGBmatrix2/COL8: track 37.1 -> 61.7 mm, vias 5 -> 3
- net /RGB/RGBmatrix2/ROW5: track 295.2 -> 275.4 mm, vias 27 -> 26
- net /RGB/RGBmatrix2/ROW4: track 304.2 -> 285.1 mm, vias 4 -> 2
- net /SMT32/ROW1: track 317.2 -> 335.5 mm
- net /RGB/RGBmatrix2/ROW3: track 310.8 -> 297.4 mm
- net /RGB/RGBmatrix2/ROW6: track 300.4 -> 287.3 mm, vias 4 -> 2
- net /RGB/RGBmatrix2/COL6: track 51.7 -> 64.3 mm
- net /RGB/RGBmatrix2/COL4: track 107.8 -> 96.4 mm
- net /SMT32/ROW4: track 376.7 -> 386.8 mm, vias 3 -> 2
- net /RGB/RGBmatrix2/COL1: track 161.7 -> 152.0 mm
- net /SMT32/ROW3: track 354.5 -> 364.2 mm
- net /RGB/RGBmatrix2/COL3: track 124.7 -> 115.1 mm
- net /RGB/RGBmatrix2/COL2: track 143.1 -> 133.6 mm
- net /RGB/RGBmatrix2/COL13: track 143.7 -> 134.4 mm
- net /RGB/RGBmatrix2/COL14: track 162.1 -> 152.8 mm
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
Commit message: Make it nicer, rev0.1 alpha
Parts:
- moved C4 0.89 mm to (107.4, 144.3)
- moved C5 0.89 mm to (108.5, 144.3)
Routing:
- net /SMT32/ROW2: track 337.9 -> 344.7 mm
- net /SMT32/ROW5: track 398.1 -> 392.2 mm
- net +3V3: track 401.9 -> 401.0 mm
- net Net-(D51-Pad2): track 1.98 -> 2.81 mm
Other:
- board text added: "JLCJLCJLCJLC"
- board text added: "NHW68 Rev:0.1 MIT License Copyright (c) 2019 Yifei Ding https://github.com/dingyifei/NHW68/"
