File: hardware/PCB/RGB.sch (KiCad schematic (older format))
At the start: 28 parts, among them U2 IS31FL3733-QF, U3 IS31FL3733-QF

Commit message: I think I figured it out
Connections:
- wire segments 72 -> 71
Other:
- moved on the sheet: C15
Changed lines of the file:
@@
 $Descr A4 11693 8268
 encoding utf-8
-Sheet 3 5
+Sheet 3 6
 Title ""
 Date ""
@@
 L Device:C_Small C15
 U 1 1 5E45EC90
-P 7850 1150
-F 0 "C15" H 7942 1196 50  0000 L CNN
-F 1 "0.47μF" H 7942 1105 50  0000 L CNN
-F 2 "Capacitor_SMD:C_0603_1608Metric_Pad1.05x0.95mm_HandSolder" H 7850 1150 50  0001 C CNN
-F 3 "~" H 7850 1150 50  0001 C CNN
-F 4 "Capacitor_SMD:C_0603_1608Metric_Pad1.05x0.95mm_HandSolder" H 7850 1150 50  0001 C CNN "Footprint"
-F 5 "0.47μF" H 7850 1150 50  0001 C CNN "Value"
-	1    7850 1150
+P 7550 1150
+F 0 "C15" H 7642 1196 50  0000 L CNN
+F 1 "0.47μF" H 7642 1105 50  0000 L CNN
+F 2 "Capacitor_SMD:C_0603_1608Metric_Pad1.05x0.95mm_HandSolder" H 7550 1150 50  0001 C CNN
+F 3 "~" H 7550 1150 50  0001 C CNN
+F 4 "Capacitor_SMD:C_0603_1608Metric_Pad1.05x0.95mm_HandSolder" H 7550 1150 50  0001 C CNN "Footprint"
+F 5 "0.47μF" H 7550 1150 50  0001 C CNN "Value"
+	1    7550 1150
 	0    -1   -1   0
 $EndComp
@@
 L power:GND #PWR0106
 U 1 1 5E45EC96
-P 7950 1150
-F 0 "#PWR0106" H 7950 900 50  0001 C CNN
-F 1 "GND" H 7955 977 50  0000 C CNN
-F 2 "" H 7950 1150 50  0001 C CNN
-F 3 "" H 7950 1150 50  0001 C CNN
-	1    7950 1150
+P 7650 1150
+F 0 "#PWR0106" H 7650 900 50  0001 C CNN
+F 1 "GND" H 7655 977 50  0000 C CNN
+F 2 "" H 7650 1150 50  0001 C CNN
+F 3 "" H 7650 1150 50  0001 C CNN
+	1    7650 1150
 	0    -1   -1   0
 $EndComp
@@
 	2400 950  2400 1100
 Connection ~ 3700 950
-Wire Wire Line
-	7450 950  7450 1150
-Wire Wire Line
-	7750 1150 7450 1150
-Connection ~ 7450 1150
 Connection ~ 3700 1900
 Wire Wire Line
@@
 Wire Wire Line
 	7450 1900 7450 2000
+Connection ~ 8050 2100
+Wire Wire Line
+	7950 2100 8050 2100
+Wire Wire Line
+	8150 3100 7800 3100
+Wire Wire Line
+	7450 950  7450 1150
+Connection ~ 7450 1150
 Wire Wire Line
 	7450 1150 7450 1900
-Connection ~ 8050 2100
-Wire Wire Line
-	7950 2100 8050 2100
-Wire Wire Line
-	8150 3100 7800 3100
 $EndSCHEMATC

Commit message: Make it better by get rid of the protonC
1. Remove protonC. use STM32F303CCT6 instead
2.Use parts based on avalibility
3.Extend the case so it now fits more parts( should be big enough
4. A reasonable USB connector
5. Probably a working DC-DC solution to providde 3.3V
6. Move 3733's 5V to only 3.3V (maybe it won't work?)
Parts:
- C1, C11, C13, C15, C2, C4, C6, C8: footprint Capacitor_SMD:C_0603_1608Metric_Pad1.05x0.95mm_HandSolder -> Capacitor_SMD:C_1206_3216Metric
- C10, C3: footprint Capacitor_Tantalum_SMD:CP_EIA-3528-12_Kemet-T_Pad1.50x2.35mm_HandSolder -> Capacitor_Tantalum_SMD:CP_EIA-3216-18_Kemet-A
- C12, C14, C16, C5, C7, C9: footprint Capacitor_SMD:C_0603_1608Metric_Pad1.05x0.95mm_HandSolder -> Capacitor_SMD:C_0603_1608Metric
- R15, R16, R17, R18, R19, R20, R21, R22, R23, R24: footprint Resistor_SMD:R_0603_1608Metric_Pad1.05x0.95mm_HandSolder -> Resistor_SMD:R_0603_1608Metric
Connections:
- net labels added: +3.3V
- net labels removed: VBUS, VCC
- no-connect marks 13 -> 15

Commit message: PSU placed
Parts:
- C1, C11, C13, C15, C2, C4, C6, C8: footprint Capacitor_SMD:C_1206_3216Metric -> Capacitor_SMD:C_0402_1005Metric
- C12, C14, C16, C5, C7, C9: footprint Capacitor_SMD:C_0603_1608Metric -> Capacitor_SMD:C_0402_1005Metric
- R15, R16, R17, R18, R19, R20, R21, R22, R23, R24: footprint Resistor_SMD:R_0603_1608Metric -> Resistor_SMD:R_0402_1005Metric
Changed lines of the file:
@@
 F 0 "R15" V 8093 3100 50  0000 C CNN
 F 1 "20k" V 8184 3100 50  0000 C CNN
-F 2 "Resistor_SMD:R_0603_1608Metric" V 8230 3100 50  0001 C CNN
+F 2 "Resistor_SMD:R_0402_1005Metric" V 8230 3100 50  0001 C CNN
 F 3 "~" H 8300 3100 50  0001 C CNN
 F 4 "20k" H 8300 3100 50  0001 C CNN "Value"
@@
 F 0 "R22" V 8193 2800 50  0000 C CNN
 F 1 "100k" V 8284 2800 50  0000 C CNN
-F 2 "Resistor_SMD:R_0603_1608Metric" V 8330 2800 50  0001 C CNN
+F 2 "Resistor_SMD:R_0402_1005Metric" V 8330 2800 50  0001 C CNN
 F 3 "~" H 8400 2800 50  0001 C CNN
 F 4 "100k" H 8400 2800 50  0001 C CNN "Value"
@@
 F 0 "C2" H 8142 2046 50  0000 L CNN
 F 1 "0.47μF" H 8142 1955 50  0000 L CNN
-F 2 "Capacitor_SMD:C_1206_3216Metric" H 8050 2000 50  0001 C CNN
+F 2 "Capacitor_SMD:C_0402_1005Metric" H 8050 2000 50  0001 C CNN
 F 3 "~" H 8050 2000 50  0001 C CNN
 F 4 "Capacitor_SMD:C_0603_1608Metric_Pad1.05x0.95mm_HandSolder" H 8050 2000 50  0001 C CNN "Footprint"
@@
 F 0 "R20" H 8020 2396 50  0000 L CNN
 F 1 "1k" H 8020 2305 50  0000 L CNN
-F 2 "Resistor_SMD:R_0603_1608Metric" V 7880 2350 50  0001 C CNN
+F 2 "Resistor_SMD:R_0402_1005Metric" V 7880 2350 50  0001 C CNN
 F 3 "~" H 7950 2350 50  0001 C CNN
 F 4 "1k" H 7950 2350 50  0001 C CNN "Value"
@@
 F 0 "R21" H 8220 2296 50  0000 L CNN
 F 1 "1k" H 8220 2205 50  0000 L CNN
-F 2 "Resistor_SMD:R_0603_1608Metric" V 8080 2250 50  0001 C CNN
+F 2 "Resistor_SMD:R_0402_1005Metric" V 8080 2250 50  0001 C CNN
 F 3 "~" H 8150 2250 50  0001 C CNN
 F 4 "1k" H 8150 2250 50  0001 C CNN "Value"
@@
 F 0 "C1" H 3342 2046 50  0000 L CNN
 F 1 "0.47μF" H 3342 1955 50  0000 L CNN
-F 2 "Capacitor_SMD:C_1206_3216Metric" H 3250 2000 50  0001 C CNN
+F 2 "Capacitor_SMD:C_0402_1005Metric" H 3250 2000 50  0001 C CNN
 F 3 "~" H 3250 2000 50  0001 C CNN
 F 4 "Capacitor_SMD:C_0603_1608Metric_Pad1.05x0.95mm_HandSolder" H 3250 2000 50  0001 C CNN "Footprint"
@@
 F 0 "R19" V 3093 3100 50  0000 C CNN
 F 1 "20k" V 3184 3100 50  0000 C CNN
-F 2 "Resistor_SMD:R_0603_1608Metric" V 3230 3100 50  0001 C CNN
+F 2 "Resistor_SMD:R_0402_1005Metric" V 3230 3100 50  0001 C CNN
 F 3 "~" H 3300 3100 50  0001 C CNN
 F 4 "20k" H 3300 3100 50  0001 C CNN "Value"
@@
 F 0 "R18" H 3370 2396 50  0000 L CNN
 F 1 "1k" H 3370 2305 50  0000 L CNN
-F 2 "Resistor_SMD:R_0603_1608Metric" V 3230 2350 50  0001 C CNN
+F 2 "Resistor_SMD:R_0402_1005Metric" V 3230 2350 50  0001 C CNN
 F 3 "~" H 3300 2350 50  0001 C CNN
 F 4 "1k" H 3300 2350 50  0001 C CNN "Value"
@@
 F 0 "R17" H 3170 2296 50  0000 L CNN
 F 1 "1k" H 3170 2205 50  0000 L CNN
-F 2 "Resistor_SMD:R_0603_1608Metric" V 3030 2250 50  0001 C CNN
+F 2 "Resistor_SMD:R_0402_1005Metric" V 3030 2250 50  0001 C CNN
 F 3 "~" H 3100 2250 50  0001 C CNN
 F 4 "1k" H 3100 2250 50  0001 C CNN "Value"
@@
 F 0 "R16" V 2643 2800 50  0000 C CNN
 F 1 "100k" V 2734 2800 50  0000 C CNN
-F 2 "Resistor_SMD:R_0603_1608Metric" V 2780 2800 50  0001 C CNN
+F 2 "Resistor_SMD:R_0402_1005Metric" V 2780 2800 50  0001 C CNN
 F 3 "~" H 2850 2800 50  0001 C CNN
 F 4 "100k" H 2850 2800 50  0001 C CNN "Value"
@@
 F 0 "C14" H 7192 1946 50  0000 L CNN
 F 1 "0.1μF" H 7192 1855 50  0000 L CNN
-F 2 "Capacitor_SMD:C_0603_1608Metric" H 7100 1900 50  0001 C CNN
+F 2 "Capacitor_SMD:C_0402_1005Metric" H 7100 1900 50  0001 C CNN
 F 3 "~" H 7100 1900 50  0001 C CNN
 F 4 "Capacitor_SMD:C_0603_1608Metric_Pad1.05x0.95mm_HandSolder" H 7100 1900 50  0001 C CNN "Footprint"
@@
 F 0 "C13" H 7192 1196 50  0000 L CNN
 F 1 "0.47μF" H 7192 1105 50  0000 L CNN
-F 2 "Capacitor_SMD:C_1206_3216Metric" H 7100 1150 50  0001 C CNN
+F 2 "Capacitor_SMD:C_0402_1005Metric" H 7100 1150 50  0001 C CNN
 F 3 "~" H 7100 1150 50  0001 C CNN
 F 4 "Capacitor_SMD:C_0603_1608Metric_Pad1.05x0.95mm_HandSolder" H 7100 1150 50  0001 C CNN "Footprint"
@@
 F 0 "C12" H 6742 1946 50  0000 L CNN
 F 1 "0.1μF" H 6742 1855 50  0000 L CNN
-F 2 "Capacitor_SMD:C_0603_1608Metric" H 6650 1900 50  0001 C CNN
+F 2 "Capacitor_SMD:C_0402_1005Metric" H 6650 1900 50  0001 C CNN
 F 3 "~" H 6650 1900 50  0001 C CNN
 F 4 "Capacitor_SMD:C_0603_1608Metric_Pad1.05x0.95mm_HandSolder" H 6650 1900 50  0001 C CNN "Footprint"
@@
 F 0 "C11" H 6742 1196 50  0000 L CNN
 F 1 "0.47μF" H 6742 1105 50  0000 L CNN
-F 2 "Capacitor_SMD:C_1206_3216Metric" H 6650 1150 50  0001 C CNN
+F 2 "Capacitor_SMD:C_0402_1005Metric" H 6650 1150 50  0001 C CNN
 F 3 "~" H 6650 1150 50  0001 C CNN
 F 4 "Capacitor_SMD:C_0603_1608Metric_Pad1.05x0.95mm_HandSolder" H 6650 1150 50  0001 C CNN "Footprint"
@@
 F 0 "C16" H 7642 1946 50  0000 L CNN
 F 1 "0.1μF" H 7642 1855 50  0000 L CNN
-F 2 "Capacitor_SMD:C_0603_1608Metric" H 7550 1900 50  0001 C CNN
+F 2 "Capacitor_SMD:C_0402_1005Metric" H 7550 1900 50  0001 C CNN
 F 3 "~" H 7550 1900 50  0001 C CNN
 F 4 "Capacitor_SMD:C_0603_1608Metric_Pad1.05x0.95mm_HandSolder" H 7550 1900 50  0001 C CNN "Footprint"
@@
 F 0 "C15" H 7642 1196 50  0000 L CNN
 F 1 "0.47μF" H 7642 1105 50  0000 L CNN
-F 2 "Capacitor_SMD:C_1206_3216Metric" H 7550 1150 50  0001 C CNN
+F 2 "Capacitor_SMD:C_0402_1005Metric" H 7550 1150 50  0001 C CNN
 F 3 "~" H 7550 1150 50  0001 C CNN
 F 4 "Capacitor_SMD:C_0603_1608Metric_Pad1.05x0.95mm_HandSolder" H 7550 1150 50  0001 C CNN "Footprint"
@@
 F 0 "C7" H 4342 1946 50  0000 L CNN
 F 1 "0.1μF" H 4342 1855 50  0000 L CNN
-F 2 "Capacitor_SMD:C_0603_1608Metric" H 4250 1900 50  0001 C CNN
+F 2 "Capacitor_SMD:C_0402_1005Metric" H 4250 1900 50  0001 C CNN
 F 3 "~" H 4250 1900 50  0001 C CNN
 F 4 "Capacitor_SMD:C_0603_1608Metric_Pad1.05x0.95mm_HandSolder" H 4250 1900 50  0001 C CNN "Footprint"
@@
 F 0 "C6" H 4342 1196 50  0000 L CNN
 F 1 "0.47μF" H 4342 1105 50  0000 L CNN
-F 2 "Capacitor_SMD:C_1206_3216Metric" H 4250 1150 50  0001 C CNN
+F 2 "Capacitor_SMD:C_0402_1005Metric" H 4250 1150 50  0001 C CNN
 F 3 "~" H 4250 1150 50  0001 C CNN
 F 4 "Capacitor_SMD:C_0603_1608Metric_Pad1.05x0.95mm_HandSolder" H 4250 1150 50  0001 C CNN "Footprint"
@@
 F 0 "C5" H 3892 1946 50  0000 L CNN
 F 1 "0.1μF" H 3892 1855 50  0000 L CNN
-F 2 "Capacitor_SMD:C_0603_1608Metric" H 3800 1900 50  0001 C CNN
+F 2 "Capacitor_SMD:C_0402_1005Metric" H 3800 1900 50  0001 C CNN
 F 3 "~" H 3800 1900 50  0001 C CNN
 F 4 "Capacitor_SMD:C_0603_1608Metric_Pad1.05x0.95mm_HandSolder" H 3800 1900 50  0001 C CNN "Footprint"
@@
 F 0 "C4" H 3892 1196 50  0000 L CNN
 F 1 "0.47μF" H 3892 1105 50  0000 L CNN
-F 2 "Capacitor_SMD:C_1206_3216Metric" H 3800 1150 50  0001 C CNN
+F 2 "Capacitor_SMD:C_0402_1005Metric" H 3800 1150 50  0001 C CNN
 F 3 "~" H 3800 1150 50  0001 C CNN
 F 4 "Capacitor_SMD:C_0603_1608Metric_Pad1.05x0.95mm_HandSolder" H 3800 1150 50  0001 C CNN "Footprint"
@@
 F 0 "C9" H 4792 1946 50  0000 L CNN
 F 1 "0.1μF" H 4792 1855 50  0000 L CNN
-F 2 "Capacitor_SMD:C_0603_1608Metric" H 4700 1900 50  0001 C CNN
+F 2 "Capacitor_SMD:C_0402_1005Metric" H 4700 1900 50  0001 C CNN
 F 3 "~" H 4700 1900 50  0001 C CNN
 F 4 "Capacitor_SMD:C_0603_1608Metric_Pad1.05x0.95mm_HandSolder" H 4700 1900 50  0001 C CNN "Footprint"
@@
 F 0 "C8" H 4792 1196 50  0000 L CNN
 F 1 "0.47μF" H 4792 1105 50  0000 L CNN
-F 2 "Capacitor_SMD:C_1206_3216Metric" H 4700 1150 50  0001 C CNN
+F 2 "Capacitor_SMD:C_0402_1005Metric" H 4700 1150 50  0001 C CNN
 F 3 "~" H 4700 1150 50  0001 C CNN
 F 4 "Capacitor_SMD:C_0603_1608Metric_Pad1.05x0.95mm_HandSolder" H 4700 1150 50  0001 C CNN "Footprint"
@@
 F 0 "R23" V 1993 2850 50  0000 C CNN
 F 1 "100k" V 2084 2850 50  0000 C CNN
-F 2 "Resistor_SMD:R_0603_1608Metric" V 2130 2850 50  0001 C CNN
+F 2 "Resistor_SMD:R_0402_1005Metric" V 2130 2850 50  0001 C CNN
 F 3 "~" H 2200 2850 50  0001 C CNN
 F 4 "100k" H 2200 2850 50  0001 C CNN "Value"
@@
 F 0 "R24" V 8843 2850 50  0000 C CNN
 F 1 "100k" V 8934 2850 50  0000 C CNN
-F 2 "Resistor_SMD:R_0603_1608Metric" V 8980 2850 50  0001 C CNN
+F 2 "Resistor_SMD:R_0402_1005Metric" V 8980 2850 50  0001 C CNN
 F 3 "~" H 9050 2850 50  0001 C CNN
 F 4 "100k" H 9050 2850 50  0001 C CNN "Value"

Commit message: Making progress, so many distance warning!!!
Parts:
- C10: renamed from C11; value 0.47μF -> 470nF
- C11: renamed from C12; value 0.1μF -> 100nF
- C12: renamed from C13; value 0.47μF -> 470nF
- C13: renamed from C14; value 0.1μF -> 100nF
- C14: renamed from C15; value 0.47μF -> 470nF
- C15: renamed from C16; value 0.1μF -> 100nF
- C16: renamed from C2; value 0.47μF -> 470nF
- C2: renamed from C1; value 0.47μF -> 470nF
- C3: renamed from C4; value 0.47μF -> 470nF
- C4: renamed from C5; value 0.1μF -> 100nF
- C5: renamed from C6; value 0.47μF -> 470nF
- C6: renamed from C7; value 0.1μF -> 100nF
- C7: renamed from C8; value 0.47μF -> 470nF
- C8: renamed from C9; value 0.1μF -> 100nF
- renumbered C3 to C1, C10 to C9, R23 to R1, R24 to R10, R16 to R2, R17 to R3, R18 to R4, R19 to R5, R20 to R6, R21 to R7, R15 to R8, R22 to R9, U2 to U1, U3 to U2

Commit message: getting closer to it actually works
Parts:
- removed C1, C9: 22μF/10V, Capacitor_Tantalum_SMD:CP_EIA-3216-18_Kemet-A, symbol Device:CP1_Small
Other:
- moved on the sheet: C5, C6
Changed lines of the file:
@@
 Connection ~ 7000 950
 Connection ~ 6550 1150
-$Comp
-L Device:CP1_Small C9
-U 1 1 5E475E34
-P 5650 1150
-F 0 "C9" H 5741 1196 50  0000 L CNN
-F 1 "22μF/10V" H 5741 1105 50  0000 L CNN
-F 2 "Capacitor_Tantalum_SMD:CP_EIA-3216-18_Kemet-A" H 5650 1150 50  0001 C CNN
-F 3 "~" H 5650 1150 50  0001 C CNN
-F 4 "Capacitor_Tantalum_SMD:CP_EIA-3528-12_Kemet-T_Pad1.50x2.35mm_HandSolder" H 5650 1150 50  0001 C CNN "Footprint"
-F 5 "22μF/10V" H 5650 1150 50  0001 C CNN "Value"
-	1    5650 1150
-	1    0    0    -1
-$EndComp
-$Comp
-L power:GND #PWR016
-U 1 1 5E476AB6
-P 5650 1250
-F 0 "#PWR016" H 5650 1000 50  0001 C CNN
-F 1 "GND" H 5655 1077 50  0000 C CNN
-F 2 "" H 5650 1250 50  0001 C CNN
-F 3 "" H 5650 1250 50  0001 C CNN
-	1    5650 1250
-	1    0    0    -1
-$EndComp
 Connection ~ 6550 950
 $Comp
 L Device:C_Small C6
 U 1 1 5E48765C
-P 4250 1900
-F 0 "C6" H 4342 1946 50  0000 L CNN
-F 1 "100nF" H 4342 1855 50  0000 L CNN
-F 2 "Capacitor_SMD:C_0402_1005Metric" H 4250 1900 50  0001 C CNN
-F 3 "~" H 4250 1900 50  0001 C CNN
-F 4 "Capacitor_SMD:C_0603_1608Metric_Pad1.05x0.95mm_HandSolder" H 4250 1900 50  0001 C CNN "Footprint"
-F 5 "0.1μF" H 4250 1900 50  0001 C CNN "Value"
-	1    4250 1900
+P 4350 1900
+F 0 "C6" H 4442 1946 50  0000 L CNN
+F 1 "100nF" H 4442 1855 50  0000 L CNN
+F 2 "Capacitor_SMD:C_0402_1005Metric" H 4350 1900 50  0001 C CNN
+F 3 "~" H 4350 1900 50  0001 C CNN
+F 4 "Capacitor_SMD:C_0603_1608Metric_Pad1.05x0.95mm_HandSolder" H 4350 1900 50  0001 C CNN "Footprint"
+F 5 "0.1μF" H 4350 1900 50  0001 C CNN "Value"
+	1    4350 1900
 	0    -1   -1   0
 $EndComp
@@
 L power:GND #PWR012
 U 1 1 5E487662
-P 4350 1900
-F 0 "#PWR012" H 4350 1650 50  0001 C CNN
-F 1 "GND" H 4355 1727 50  0000 C CNN
-F 2 "" H 4350 1900 50  0001 C CNN
-F 3 "" H 4350 1900 50  0001 C CNN
-	1    4350 1900
+P 4450 1900
+F 0 "#PWR012" H 4450 1650 50  0001 C CNN
+F 1 "GND" H 4455 1727 50  0000 C CNN
+F 2 "" H 4450 1900 50  0001 C CNN
+F 3 "" H 4450 1900 50  0001 C CNN
+	1    4450 1900
 	0    -1   -1   0
 $EndComp
@@
 L Device:C_Small C5
 U 1 1 5E487668
-P 4250 1150
-F 0 "C5" H 4342 1196 50  0000 L CNN
-F 1 "470nF" H 4342 1105 50  0000 L CNN
-F 2 "Capacitor_SMD:C_0402_1005Metric" H 4250 1150 50  0001 C CNN
-F 3 "~" H 4250 1150 50  0001 C CNN
-F 4 "Capacitor_SMD:C_0603_1608Metric_Pad1.05x0.95mm_HandSolder" H 4250 1150 50  0001 C CNN "Footprint"
-F 5 "0.47μF" H 4250 1150 50  0001 C CNN "Value"
-	1    4250 1150
+P 4350 1150
+F 0 "C5" H 4442 1196 50  0000 L CNN
+F 1 "470nF" H 4442 1105 50  0000 L CNN
+F 2 "Capacitor_SMD:C_0402_1005Metric" H 4350 1150 50  0001 C CNN
+F 3 "~" H 4350 1150 50  0001 C CNN
+F 4 "Capacitor_SMD:C_0603_1608Metric_Pad1.05x0.95mm_HandSolder" H 4350 1150 50  0001 C CNN "Footprint"
+F 5 "0.47μF" H 4350 1150 50  0001 C CNN "Value"
+	1    4350 1150
 	0    -1   -1   0
 $EndComp
@@
 L power:GND #PWR011
 U 1 1 5E48766E
-P 4350 1150
-F 0 "#PWR011" H 4350 900 50  0001 C CNN
-F 1 "GND" H 4355 977 50  0000 C CNN
-F 2 "" H 4350 1150 50  0001 C CNN
-F 3 "" H 4350 1150 50  0001 C CNN
-	1    4350 1150
+P 4450 1150
+F 0 "#PWR011" H 4450 900 50  0001 C CNN
+F 1 "GND" H 4455 977 50  0000 C CNN
+F 2 "" H 4450 1150 50  0001 C CNN
+F 3 "" H 4450 1150 50  0001 C CNN
+	1    4450 1150
 	0    -1   -1   0
 $EndComp
@@
 $EndComp
 Wire Wire Line
-	4600 950  4150 950
-Wire Wire Line
-	4150 950  4150 1150
-Connection ~ 4150 1150
-Wire Wire Line
-	4150 950  3700 950
+	4600 950  4250 950
+Wire Wire Line
+	4250 950  4250 1150
+Connection ~ 4250 1150
 Wire Wire Line
 	3700 950  3700 1150
-Connection ~ 4150 950
 Connection ~ 3700 1150
 Wire Wire Line
@@
 Wire Wire Line
 	4600 2000 4350 2000
-Connection ~ 4350 2000
-Wire Wire Line
-	4350 2000 4250 2000
 Text HLabel 2100 2700 0    50   Input ~ 0
 LED_EN_PIN
@@
 Wire Wire Line
 	5650 850  5650 950
-Connection ~ 5650 950
-Wire Wire Line
-	5650 950  5650 1050
-$Comp
-L Device:CP1_Small C1
-U 1 1 5E6C50D8
-P 2400 1200
-F 0 "C1" H 2491 1246 50  0000 L CNN
-F 1 "22μF/10V" H 2491 1155 50  0000 L CNN
-F 2 "Capacitor_Tantalum_SMD:CP_EIA-3216-18_Kemet-A" H 2400 1200 50  0001 C CNN
-F 3 "~" H 2400 1200 50  0001 C CNN
-F 4 "Capacitor_Tantalum_SMD:CP_EIA-3528-12_Kemet-T_Pad1.50x2.35mm_HandSolder" H 2400 1200 50  0001 C CNN "Footprint"
-F 5 "22μF/10V" H 2400 1200 50  0001 C CNN "Value"
-	1    2400 1200
-	1    0    0    -1
-$EndComp
-$Comp
-L power:GND #PWR03
-U 1 1 5E6C50E2
-P 2400 1300
-F 0 "#PWR03" H 2400 1050 50  0001 C CNN
-F 1 "GND" H 2405 1127 50  0000 C CNN
-F 2 "" H 2400 1300 50  0001 C CNN
-F 3 "" H 2400 1300 50  0001 C CNN
-	1    2400 1300
-	1    0    0    -1
-$EndComp
 Wire Wire Line
 	2400 900  2400 950
-Connection ~ 2400 950
-Wire Wire Line
-	2400 950  2400 1100
 Connection ~ 3700 950
 Connection ~ 3700 1900
@@
 Wire Wire Line
 	3700 1150 3700 1900
-Connection ~ 4150 1900
-Wire Wire Line
-	4150 1900 4150 2000
-Wire Wire Line
-	4150 1150 4150 1900
+Connection ~ 4250 1900
+Wire Wire Line
+	4250 1900 4250 2000
+Wire Wire Line
+	4250 1150 4250 1900
 Connection ~ 4600 1900
 Wire Wire Line
@@
 NoConn ~ 6400 3600
 NoConn ~ 4850 3600
+Wire Wire Line
+	4150 2000 4050 2000
+Connection ~ 4050 2000
+Connection ~ 4250 950
+Wire Wire Line
+	3700 950  4250 950
 $EndSCHEMATC
