File: hardware/PCB/RGB.sch (KiCad schematic (older format))
At the start: 20 parts, among them U1 IS31FL3733-QFLS4-TR, U2 IS31FL3733-QFLS4-TR

Commit message: changed to 0603
Parts:
- C1, C10, C11, C12, C13, C14, C2, C3, C4, C5, C6, C7, C8, C9: footprint Capacitor_SMD:C_0402_1005Metric -> Capacitor_SMD:C_0603_1608Metric
- R1, R4, R7, R8: footprint Resistor_SMD:R_0402_1005Metric -> Resistor_SMD:R_0603_1608Metric
Changed lines of the file:
@@
 F 0 "R7" V 8093 3100 50  0000 C CNN
 F 1 "20k" V 8184 3100 50  0000 C CNN
-F 2 "Resistor_SMD:R_0402_1005Metric" V 8230 3100 50  0001 C CNN
+F 2 "Resistor_SMD:R_0603_1608Metric" V 8230 3100 50  0001 C CNN
 F 3 "~" H 8300 3100 50  0001 C CNN
 	1    8300 3100
@@
 F 0 "R8" V 8193 2800 50  0000 C CNN
 F 1 "100k" V 8284 2800 50  0000 C CNN
-F 2 "Resistor_SMD:R_0402_1005Metric" V 8330 2800 50  0001 C CNN
+F 2 "Resistor_SMD:R_0603_1608Metric" V 8330 2800 50  0001 C CNN
 F 3 "~" H 8400 2800 50  0001 C CNN
 	1    8400 2800
@@
 F 0 "C14" H 8242 2046 50  0000 L CNN
 F 1 "470nF" H 8242 1955 50  0000 L CNN
-F 2 "Capacitor_SMD:C_0402_1005Metric" H 8150 2000 50  0001 C CNN
+F 2 "Capacitor_SMD:C_0603_1608Metric" H 8150 2000 50  0001 C CNN
 F 3 "~" H 8150 2000 50  0001 C CNN
 	1    8150 2000
@@
 F 0 "C1" H 3192 2146 50  0000 L CNN
 F 1 "470nF" H 3192 2055 50  0000 L CNN
-F 2 "Capacitor_SMD:C_0402_1005Metric" H 3100 2100 50  0001 C CNN
+F 2 "Capacitor_SMD:C_0603_1608Metric" H 3100 2100 50  0001 C CNN
 F 3 "~" H 3100 2100 50  0001 C CNN
 	1    3100 2100
@@
 F 0 "R4" V 3093 3100 50  0000 C CNN
 F 1 "20k" V 3184 3100 50  0000 C CNN
-F 2 "Resistor_SMD:R_0402_1005Metric" V 3230 3100 50  0001 C CNN
+F 2 "Resistor_SMD:R_0603_1608Metric" V 3230 3100 50  0001 C CNN
 F 3 "~" H 3300 3100 50  0001 C CNN
 	1    3300 3100
@@
 F 0 "R1" V 2643 2800 50  0000 C CNN
 F 1 "100k" V 2734 2800 50  0000 C CNN
-F 2 "Resistor_SMD:R_0402_1005Metric" V 2780 2800 50  0001 C CNN
+F 2 "Resistor_SMD:R_0603_1608Metric" V 2780 2800 50  0001 C CNN
 F 3 "~" H 2850 2800 50  0001 C CNN
 	1    2850 2800
@@
 F 0 "C11" H 7192 1946 50  0000 L CNN
 F 1 "100nF" H 7192 1855 50  0000 L CNN
-F 2 "Capacitor_SMD:C_0402_1005Metric" H 7100 1900 50  0001 C CNN
+F 2 "Capacitor_SMD:C_0603_1608Metric" H 7100 1900 50  0001 C CNN
 F 3 "~" H 7100 1900 50  0001 C CNN
 	1    7100 1900
@@
 F 0 "C10" H 7192 1196 50  0000 L CNN
 F 1 "470nF" H 7192 1105 50  0000 L CNN
-F 2 "Capacitor_SMD:C_0402_1005Metric" H 7100 1150 50  0001 C CNN
+F 2 "Capacitor_SMD:C_0603_1608Metric" H 7100 1150 50  0001 C CNN
 F 3 "~" H 7100 1150 50  0001 C CNN
 	1    7100 1150
@@
 F 0 "C9" H 6742 1946 50  0000 L CNN
 F 1 "100nF" H 6742 1855 50  0000 L CNN
-F 2 "Capacitor_SMD:C_0402_1005Metric" H 6650 1900 50  0001 C CNN
+F 2 "Capacitor_SMD:C_0603_1608Metric" H 6650 1900 50  0001 C CNN
 F 3 "~" H 6650 1900 50  0001 C CNN
 	1    6650 1900
@@
 F 0 "C8" H 6742 1196 50  0000 L CNN
 F 1 "470nF" H 6742 1105 50  0000 L CNN
-F 2 "Capacitor_SMD:C_0402_1005Metric" H 6650 1150 50  0001 C CNN
+F 2 "Capacitor_SMD:C_0603_1608Metric" H 6650 1150 50  0001 C CNN
 F 3 "~" H 6650 1150 50  0001 C CNN
 	1    6650 1150
@@
 F 0 "C13" H 7642 1946 50  0000 L CNN
 F 1 "100nF" H 7642 1855 50  0000 L CNN
-F 2 "Capacitor_SMD:C_0402_1005Metric" H 7550 1900 50  0001 C CNN
+F 2 "Capacitor_SMD:C_0603_1608Metric" H 7550 1900 50  0001 C CNN
 F 3 "~" H 7550 1900 50  0001 C CNN
 	1    7550 1900
@@
 F 0 "C12" H 7642 1196 50  0000 L CNN
 F 1 "470nF" H 7642 1105 50  0000 L CNN
-F 2 "Capacitor_SMD:C_0402_1005Metric" H 7550 1150 50  0001 C CNN
+F 2 "Capacitor_SMD:C_0603_1608Metric" H 7550 1150 50  0001 C CNN
 F 3 "~" H 7550 1150 50  0001 C CNN
 	1    7550 1150
@@
 F 0 "C5" H 4442 1946 50  0000 L CNN
 F 1 "100nF" H 4442 1855 50  0000 L CNN
-F 2 "Capacitor_SMD:C_0402_1005Metric" H 4350 1900 50  0001 C CNN
+F 2 "Capacitor_SMD:C_0603_1608Metric" H 4350 1900 50  0001 C CNN
 F 3 "~" H 4350 1900 50  0001 C CNN
 	1    4350 1900
@@
 F 0 "C4" H 4442 1196 50  0000 L CNN
 F 1 "470nF" H 4442 1105 50  0000 L CNN
-F 2 "Capacitor_SMD:C_0402_1005Metric" H 4350 1150 50  0001 C CNN
+F 2 "Capacitor_SMD:C_0603_1608Metric" H 4350 1150 50  0001 C CNN
 F 3 "~" H 4350 1150 50  0001 C CNN
 	1    4350 1150
@@
 F 0 "C3" H 3892 1946 50  0000 L CNN
 F 1 "100nF" H 3892 1855 50  0000 L CNN
-F 2 "Capacitor_SMD:C_0402_1005Metric" H 3800 1900 50  0001 C CNN
+F 2 "Capacitor_SMD:C_0603_1608Metric" H 3800 1900 50  0001 C CNN
 F 3 "~" H 3800 1900 50  0001 C CNN
 	1    3800 1900
@@
 F 0 "C2" H 3892 1196 50  0000 L CNN
 F 1 "470nF" H 3892 1105 50  0000 L CNN
-F 2 "Capacitor_SMD:C_0402_1005Metric" H 3800 1150 50  0001 C CNN
+F 2 "Capacitor_SMD:C_0603_1608Metric" H 3800 1150 50  0001 C CNN
 F 3 "~" H 3800 1150 50  0001 C CNN
 	1    3800 1150
@@
 F 0 "C7" H 4792 1946 50  0000 L CNN
 F 1 "100nF" H 4792 1855 50  0000 L CNN
-F 2 "Capacitor_SMD:C_0402_1005Metric" H 4700 1900 50  0001 C CNN
+F 2 "Capacitor_SMD:C_0603_1608Metric" H 4700 1900 50  0001 C CNN
 F 3 "~" H 4700 1900 50  0001 C CNN
 	1    4700 1900
@@
 F 0 "C6" H 4792 1196 50  0000 L CNN
 F 1 "470nF" H 4792 1105 50  0000 L CNN
-F 2 "Capacitor_SMD:C_0402_1005Metric" H 4700 1150 50  0001 C CNN
+F 2 "Capacitor_SMD:C_0603_1608Metric" H 4700 1150 50  0001 C CNN
 F 3 "~" H 4700 1150 50  0001 C CNN
 	1    4700 1150

Commit message: Rev 0.5
1. Use a better 1205 LED (much chaper on LCSC)
2. Fix the crystal CL, Rext
3. did a better job on wiring (but might come with power issues?)
4. fix the key position (0.01mm shifted so its a big fix)
5. generate better bom files
6. add in LCSC and part number so easier to source
0.4 is gone
Parts:
- C1, C10, C12, C14, C2, C4, C6, C8: LCSC (none) -> C1623; Part Number (none) -> CL10B474KA8NNNC
- R1, R8: LCSC (none) -> C116674; Part Number (none) -> AC0603FR-07100KL
- R4, R7: value 20k -> 22k; LCSC (none) -> C100865; Part Number (none) -> CR0603FA2202G
Connections:
- net RGBmatrix/COL10: now also U1.27 (CS11); no longer U1.26 (CS10)
- net RGBmatrix/COL11: now also U1.28 (CS12); no longer U1.27 (CS11)
- net RGBmatrix/COL12: now also U1.30 (CS13); no longer U1.28 (CS12)
- net RGBmatrix/COL13: now also U1.19 (CS4); no longer U1.30 (CS13)
- net RGBmatrix/COL4: now also U1.21 (CS5); no longer U1.19 (CS4)
- net RGBmatrix/COL5: now also U1.22 (CS6); no longer U1.21 (CS5)
- net RGBmatrix/COL6: now also U1.23 (CS7); no longer U1.22 (CS6)
- net RGBmatrix/COL7: now also U1.24 (CS8); no longer U1.23 (CS7)
- net RGBmatrix/COL8: now also U1.25 (CS9); no longer U1.24 (CS8)
- net RGBmatrix/COL9: now also U1.26 (CS10); no longer U1.25 (CS9)
- net RGBmatrix/ROW1: now also U1.11 (SW9); no longer U1.9 (SW7)
- net RGBmatrix/ROW3: now also U1.9 (SW7); no longer U1.11 (SW9)
- net RGBmatrix/ROW4: now also U1.8 (SW6); no longer U1.6 (SW4)
- net RGBmatrix/ROW6: now also U1.6 (SW4); no longer U1.8 (SW6)
- net RGBmatrix/ROW7: now also U1.15 (SW12); no longer U1.13 (SW10)
- net RGBmatrix/ROW9: now also U1.13 (SW10); no longer U1.15 (SW12)
- net RGBmatrix2/COL1: now also U2.22 (CS6); no longer U2.16 (CS1)
- net RGBmatrix2/COL2: now also U2.21 (CS5); no longer U2.17 (CS2)
- net RGBmatrix2/COL3: now also U2.19 (CS4); no longer U2.18 (CS3)
- net RGBmatrix2/COL4: now also U2.18 (CS3); no longer U2.19 (CS4)
- net RGBmatrix2/COL5: now also U2.17 (CS2); no longer U2.21 (CS5)
- net RGBmatrix2/COL6: now also U2.16 (CS1); no longer U2.22 (CS6)
- net RGBmatrix2/ROW4: now also U2.11 (SW9); no longer U2.9 (SW7)
- net RGBmatrix2/ROW6: now also U2.9 (SW7); no longer U2.11 (SW9)
Other:
- moved on the sheet: C14, R4
Changed lines of the file:
@@
 Sheet 3 6
 Title "NHW68"
-Date "2020-02-04"
-Rev "0.3"
+Date "2020-02-08"
+Rev "0.5"
 Comp ""
 Comment1 ""
@@
 Comment4 ""
 $EndDescr
-Text HLabel 8300 2500 2    50   Input ~ 0
+Text HLabel 7800 2500 2    50   Input ~ 0
 SCL
-Text HLabel 8300 2400 2    50   Input ~ 0
+Text HLabel 7800 2400 2    50   Input ~ 0
 SDA
-Text HLabel 2950 2500 0    50   Input ~ 0
+Text HLabel 3450 2500 0    50   Input ~ 0
 SCL
-Text HLabel 2950 2400 0    50   Input ~ 0
+Text HLabel 3450 2400 0    50   Input ~ 0
 SDA
 $Comp
@@
 P 8300 3100
 F 0 "R7" V 8093 3100 50  0000 C CNN
-F 1 "20k" V 8184 3100 50  0000 C CNN
+F 1 "22k" V 8184 3100 50  0000 C CNN
 F 2 "Resistor_SMD:R_0603_1608Metric" V 8230 3100 50  0001 C CNN
 F 3 "~" H 8300 3100 50  0001 C CNN
+F 4 "C100865" H 8300 3100 50  0001 C CNN "LCSC"
+F 5 "CR0603FA2202G" H 8300 3100 50  0001 C CNN "Part Number"
 	1    8300 3100
 	0    -1   -1   0
@@
 	0    1    -1   0
 $EndComp
-Connection ~ 3150 3200
-Wire Wire Line
-	3150 3300 3150 3200
-Wire Wire Line
-	3450 3300 3150 3300
-Wire Wire Line
-	3450 3200 3150 3200
-Connection ~ 3150 3100
-Wire Wire Line
-	3150 3100 3150 3200
+Connection ~ 3000 3200
+Wire Wire Line
+	3000 3300 3000 3200
+Connection ~ 3000 3100
+Wire Wire Line
+	3000 3100 3000 3200
 $Comp
 L power:GND #PWR04
 U 1 1 5E425D93
-P 3150 3100
-F 0 "#PWR04" H 3150 2850 50  0001 C CNN
-F 1 "GND" V 3155 2972 50  0000 R CNN
-F 2 "" H 3150 3100 50  0001 C CNN
-F 3 "" H 3150 3100 50  0001 C CNN
-	1    3150 3100
+P 3000 3100
+F 0 "#PWR04" H 3000 2850 50  0001 C CNN
+F 1 "GND" V 3005 2972 50  0000 R CNN
+F 2 "" H 3000 3100 50  0001 C CNN
+F 3 "" H 3000 3100 50  0001 C CNN
+	1    3000 3100
 	0    1    -1   0
 $EndComp
@@
 L power:GND #PWR022
 U 1 1 5E42518F
-P 8150 1900
-F 0 "#PWR022" H 8150 1650 50  0001 C CNN
-F 1 "GND" H 8155 1727 50  0000 C CNN
-F 2 "" H 8150 1900 50  0001 C CNN
-F 3 "" H 8150 1900 50  0001 C CNN
-	1    8150 1900
+P 8150 2000
+F 0 "#PWR022" H 8150 1750 50  0001 C CNN
+F 1 "GND" H 8155 1827 50  0000 C CNN
+F 2 "" H 8150 2000 50  0001 C CNN
+F 3 "" H 8150 2000 50  0001 C CNN
+	1    8150 2000
 	-1   0    0    1
 $EndComp
@@
 F 2 "Resistor_SMD:R_0603_1608Metric" V 8330 2800 50  0001 C CNN
 F 3 "~" H 8400 2800 50  0001 C CNN
+F 4 "C116674" H 8400 2800 50  0001 C CNN "LCSC"
+F 5 "AC0603FR-07100KL" H 8400 2800 50  0001 C CNN "Part Number"
 	1    8400 2800
 	0    -1   1    0
@@
 L Device:C_Small C14
 U 1 1 5E406F19
-P 8150 2000
-F 0 "C14" H 8242 2046 50  0000 L CNN
-F 1 "470nF" H 8242 1955 50  0000 L CNN
-F 2 "Capacitor_SMD:C_0603_1608Metric" H 8150 2000 50  0001 C CNN
-F 3 "~" H 8150 2000 50  0001 C CNN
-	1    8150 2000
+P 8150 2100
+F 0 "C14" H 8242 2146 50  0000 L CNN
+F 1 "470nF" H 8242 2055 50  0000 L CNN
+F 2 "Capacitor_SMD:C_0603_1608Metric" H 8150 2100 50  0001 C CNN
+F 3 "~" H 8150 2100 50  0001 C CNN
+F 4 "C1623" H 8150 2100 50  0001 C CNN "LCSC"
+F 5 "CL10B474KA8NNNC" H 8150 2100 50  0001 C CNN "Part Number"
+	1    8150 2100
 	-1   0    0    -1
 $EndComp
@@
 F 2 "Capacitor_SMD:C_0603_1608Metric" H 3100 2100 50  0001 C CNN
 F 3 "~" H 3100 2100 50  0001 C CNN
+F 4 "C1623" H 3100 2100 50  0001 C CNN "LCSC"
+F 5 "CL10B474KA8NNNC" H 3100 2100 50  0001 C CNN "Part Number"
 	1    3100 2100
 	1    0    0    -1
@@
 L Device:R R4
 U 1 1 5E39AF39
-P 3300 3100
-F 0 "R4" V 3093 3100 50  0000 C CNN
-F 1 "20k" V 3184 3100 50  0000 C CNN
-F 2 "Resistor_SMD:R_0603_1608Metric" V 3230 3100 50  0001 C CNN
-F 3 "~" H 3300 3100 50  0001 C CNN
-	1    3300 3100
+P 3150 3100
+F 0 "R4" V 2943 3100 50  0000 C CNN
+F 1 "22k" V 3034 3100 50  0000 C CNN
+F 2 "Resistor_SMD:R_0603_1608Metric" V 3080 3100 50  0001 C CNN
+F 3 "~" H 3150 3100 50  0001 C CNN
+F 4 "C100865" H 3150 3100 50  0001 C CNN "LCSC"
+F 5 "CR0603FA2202G" H 3150 3100 50  0001 C CNN "Part Number"
+	1    3150 3100
 	0    1    1    0
 $EndComp
@@
 U 1 1 5E390363
 P 2850 2800
-F 0 "R1" V 2643 2800 50  0000 C CNN
+F 0 "R1" V 2650 2800 50  0000 C CNN
 F 1 "100k" V 2734 2800 50  0000 C CNN
 F 2 "Resistor_SMD:R_0603_1608Metric" V 2780 2800 50  0001 C CNN
 F 3 "~" H 2850 2800 50  0001 C CNN
+F 4 "C116674" H 2850 2800 50  0001 C CNN "LCSC"
+F 5 "AC0603FR-07100KL" H 2850 2800 50  0001 C CNN "Part Number"
 	1    2850 2800
 	0    1    1    0
@@
 F3 "COL2" I L 4850 2300 50
 F4 "COL3" I L 4850 2400 50
-F5 "COL4" I L 4850 2500 50
-F6 "COL5" I L 4850 2600 50
-F7 "COL6" I L 4850 2700 50
-F8 "COL7" I L 4850 2800 50
-F9 "COL8" I L 4850 2900 50
-F10 "COL9" I L 4850 3000 50
-F11 "COL10" I L 4850 3100 50
-F12 "COL11" I L 4850 3200 50
-F13 "COL12" I L 4850 3300 50
-F14 "COL13" I L 4850 3400 50
+F5 "COL4" I L 4850 2600 50
+F6 "COL5" I L 4850 2700 50
+F7 "COL6" I L 4850 2800 50
+F8 "COL7" I L 4850 2900 50
+F9 "COL8" I L 4850 3000 50
+F10 "COL9" I L 4850 3100 50
+F11 "COL10" I L 4850 3200 50
+F12 "COL11" I L 4850 3300 50
+F13 "COL12" I L 4850 3400 50
+F14 "COL13" I L 4850 2500 50
 F15 "COL14" I L 4850 3500 50
-F16 "ROW1" I L 4850 4500 50
+F16 "ROW1" I L 4850 4700 50
 F17 "ROW2" I L 4850 4600 50
-F18 "ROW3" I L 4850 4700 50
-F19 "ROW4" I L 4850 4200 50
+F18 "ROW3" I L 4850 4500 50
+F19 "ROW4" I L 4850 4400 50
 F20 "ROW5" I L 4850 4300 50
-F21 "ROW6" I L 4850 4400 50
-F22 "ROW7" I L 4850 4800 50
+F21 "ROW6" I L 4850 4200 50
+F22 "ROW7" I L 4850 5000 50
 F23 "ROW8" I L 4850 4900 50
-F24 "ROW9" I L 4850 5000 50
+F24 "ROW9" I L 4850 4800 50
 $EndSheet
 $Comp
@@
 F 2 "Capacitor_SMD:C_0603_1608Metric" H 7100 1150 50  0001 C CNN
 F 3 "~" H 7100 1150 50  0001 C CNN
+F 4 "C1623" H 7100 1150 50  0001 C CNN "LCSC"
+F 5 "CL10B474KA8NNNC" H 7100 1150 50  0001 C CNN "Part Number"
 	1    7100 1150
 	0    -1   -1   0
@@
 F 2 "Capacitor_SMD:C_0603_1608Metric" H 6650 1150 50  0001 C CNN
 F 3 "~" H 6650 1150 50  0001 C CNN
+F 4 "C1623" H 6650 1150 50  0001 C CNN "LCSC"
+F 5 "CL10B474KA8NNNC" H 6650 1150 50  0001 C CNN "Part Number"
 	1    6650 1150
 	0    -1   -1   0
@@
 F 2 "Capacitor_SMD:C_0603_1608Metric" H 7550 1150 50  0001 C CNN
 F 3 "~" H 7550 1150 50  0001 C CNN
+F 4 "C1623" H 7550 1150 50  0001 C CNN "LCSC"
+F 5 "CL10B474KA8NNNC" H 7550 1150 50  0001 C CNN "Part Number"
 	1    7550 1150
 	0    -1   -1   0
@@
 F 2 "Capacitor_SMD:C_0603_1608Metric" H 4350 1150 50  0001 C CNN
 F 3 "~" H 4350 1150 50  0001 C CNN
+F 4 "C1623" H 4350 1150 50  0001 C CNN "LCSC"
+F 5 "CL10B474KA8NNNC" H 4350 1150 50  0001 C CNN "Part Number"
 	1    4350 1150
 	0    -1   -1   0
@@
 F 2 "Capacitor_SMD:C_0603_1608Metric" H 3800 1150 50  0001 C CNN
 F 3 "~" H 3800 1150 50  0001 C CNN
+F 4 "C1623" H 3800 1150 50  0001 C CNN "LCSC"
+F 5 "CL10B474KA8NNNC" H 3800 1150 50  0001 C CNN "Part Number"
 	1    3800 1150
 	0    -1   -1   0
@@
 F 2 "Capacitor_SMD:C_0603_1608Metric" H 4700 1150 50  0001 C CNN
 F 3 "~" H 4700 1150 50  0001 C CNN
+F 4 "C1623" H 4700 1150 50  0001 C CNN "LCSC"
+F 5 "CL10B474KA8NNNC" H 4700 1150 50  0001 C CNN "Part Number"
 	1    4700 1150
 	0    -1   -1   0
@@
 Wire Wire Line
 	4600 2000 4350 2000
-Text HLabel 2450 2700 0    50   Input ~ 0
+Text HLabel 3450 2700 0    50   Input ~ 0
 LED_EN_PIN
-Text HLabel 9150 2700 2    50   Input ~ 0
+Text HLabel 7800 2700 2    50   Input ~ 0
 LED_EN_PIN
-Text Label 2750 3000 2    50   ~ 0
+Text Label 3450 3000 2    50   ~ 0
 SYNC
-Text Label 8100 3000 0    50   ~ 0
+Text Label 7800 3000 0    50   ~ 0
 SYNC
-Wire Wire Line
-	8100 3000 7800 3000
 $Comp
 L power:PWR_FLAG #FLG01
@@
 	7450 1900 7450 2000
 Wire Wire Line
-	8150 3100 7800 3100
-Wire Wire Line
 	7450 950  7450 1150
 Connection ~ 7450 1150
@@
 Wire Wire Line
 	3700 950  4250 950
-Wire Wire Line
-	7800 2700 9150 2700
 NoConn ~ 4850 4100
 NoConn ~ 4850 4000
@@
 F0 "RGBmatrix2" 50
 F1 "RGBMatrix2.sch" 50
-F2 "COL1" I R 6400 2200 50
-F3 "COL2" I R 6400 2300 50
-F4 "COL3" I R 6400 2400 50
-F5 "COL4" I R 6400 2500 50
-F6 "COL5" I R 6400 2600 50
-F7 "COL6" I R 6400 2700 50
+F2 "COL1" I R 6400 2700 50
+F3 "COL2" I R 6400 2600 50
+F4 "COL3" I R 6400 2500 50
+F5 "COL4" I R 6400 2400 50
+F6 "COL5" I R 6400 2300 50
+F7 "COL6" I R 6400 2200 50
 F8 "COL7" I R 6400 2800 50
 F9 "COL8" I R 6400 2900 50
@@
 F17 "ROW2" I R 6400 4900 50
 F18 "ROW3" I R 6400 4800 50
-F19 "ROW4" I R 6400 4500 50
+F19 "ROW4" I R 6400 4700 50
 F20 "ROW5" I R 6400 4600 50
-F21 "ROW6" I R 6400 4700 50
+F21 "ROW6" I R 6400 4500 50
 $EndSheet
 Wire Wire Line
-	2950 2500 3450 2500
-Wire Wire Line
 	7950 3200 7800 3200
-Wire Wire Line
-	3450 2400 2950 2400
-Wire Wire Line
-	7800 2500 8300 2500
 Wire Wire Line
 	3100 2200 3450 2200
@@
 $EndComp
 Connection ~ 3700 950
-Wire Wire Line
-	8300 2400 7800 2400
-Wire Wire Line
-	7800 2200 8150 2200
-Wire Wire Line
-	8150 2200 8150 2100
-Connection ~ 8150 2200
-Wire Wire Line
-	8150 2200 8300 2200
-Wire Wire Line
-	3450 2700 2450 2700
-Wire Wire Line
-	2750 3000 3450 3000
 Text Label 1700 3000 3    50   ~ 0
 SYNC
+Wire Wire Line
+	3300 3100 3450 3100
+Wire Wire Line
+	3000 3200 3450 3200
+Wire Wire Line
+	3000 3300 3450 3300
+Wire Wire Line
+	8150 3100 7800 3100
+Wire Wire Line
+	7800 2200 8150 2200
+Connection ~ 8150 2200
+Wire Wire Line
+	8150 2200 8300 2200
 $EndSCHEMATC

Commit message: 0.6 I hate these auto generated code from STM32Cube
1. ready for the firmware nightmare
2. adjust the M3 screw holes
3. add tooling holes for future PCBA
4. if nothing go wrong, this will be the V1 after testing
Parts:
- C11, C13, C3, C5, C7, C9: LCSC (none) -> C24452; Part Number (none) -> CL10B104JB8NNNC
- renumbered R4 to R2, R7 to R3, R8 to R4
Changed lines of the file:
@@
 Sheet 3 6
 Title "NHW68"
-Date "2020-02-08"
-Rev "0.5"
+Date "2020-02-10"
+Rev "0.6"
 Comp ""
 Comment1 ""
@@
 $EndComp
 $Comp
-L Device:R R7
+L Device:R R3
 U 1 1 5E43A1BE
 P 8300 3100
-F 0 "R7" V 8093 3100 50  0000 C CNN
+F 0 "R3" V 8093 3100 50  0000 C CNN
 F 1 "22k" V 8184 3100 50  0000 C CNN
 F 2 "Resistor_SMD:R_0603_1608Metric" V 8230 3100 50  0001 C CNN
@@
 $EndComp
 $Comp
-L power:GND #PWR05
+L power:GND #PWR04
 U 1 1 5E42BB66
 P 3100 2000
-F 0 "#PWR05" H 3100 1750 50  0001 C CNN
+F 0 "#PWR04" H 3100 1750 50  0001 C CNN
 F 1 "GND" H 3105 1827 50  0000 C CNN
 F 2 "" H 3100 2000 50  0001 C CNN
@@
 $EndComp
 $Comp
-L power:GND #PWR02
+L power:GND #PWR01
 U 1 1 5E429DF5
 P 2700 2800
-F 0 "#PWR02" H 2700 2550 50  0001 C CNN
+F 0 "#PWR01" H 2700 2550 50  0001 C CNN
 F 1 "GND" V 2705 2672 50  0000 R CNN
 F 2 "" H 2700 2800 50  0001 C CNN
@@
 	3000 3100 3000 3200
 $Comp
-L power:GND #PWR04
+L power:GND #PWR03
 U 1 1 5E425D93
 P 3000 3100
-F 0 "#PWR04" H 3000 2850 50  0001 C CNN
+F 0 "#PWR03" H 3000 2850 50  0001 C CNN
 F 1 "GND" V 3005 2972 50  0000 R CNN
 F 2 "" H 3000 3100 50  0001 C CNN
@@
 $EndComp
 $Comp
-L power:GND #PWR021
+L power:GND #PWR020
 U 1 1 5E4213E7
 P 7800 3300
-F 0 "#PWR021" H 7800 3050 50  0001 C CNN
+F 0 "#PWR020" H 7800 3050 50  0001 C CNN
 F 1 "GND" V 7805 3172 50  0000 R CNN
 F 2 "" H 7800 3300 50  0001 C CNN
@@
 	7800 2800 8250 2800
 $Comp
-L Device:R R8
+L Device:R R4
 U 1 1 5E41DC10
 P 8400 2800
-F 0 "R8" V 8193 2800 50  0000 C CNN
+F 0 "R4" V 8193 2800 50  0000 C CNN
 F 1 "100k" V 8284 2800 50  0000 C CNN
 F 2 "Resistor_SMD:R_0603_1608Metric" V 8330 2800 50  0001 C CNN
@@
 	4250 5200 4150 5200
 $Comp
-L Device:R R4
+L Device:R R2
 U 1 1 5E39AF39
 P 3150 3100
-F 0 "R4" V 2943 3100 50  0000 C CNN
+F 0 "R2" V 2943 3100 50  0000 C CNN
 F 1 "22k" V 3034 3100 50  0000 C CNN
 F 2 "Resistor_SMD:R_0603_1608Metric" V 3080 3100 50  0001 C CNN
@@
 F 2 "Capacitor_SMD:C_0603_1608Metric" H 7100 1900 50  0001 C CNN
 F 3 "~" H 7100 1900 50  0001 C CNN
+F 4 "C24452" H 7100 1900 50  0001 C CNN "LCSC"
+F 5 "CL10B104JB8NNNC" H 7100 1900 50  0001 C CNN "Part Number"
 	1    7100 1900
 	0    -1   -1   0
@@
 F 2 "Capacitor_SMD:C_0603_1608Metric" H 6650 1900 50  0001 C CNN
 F 3 "~" H 6650 1900 50  0001 C CNN
+F 4 "C24452" H 6650 1900 50  0001 C CNN "LCSC"
+F 5 "CL10B104JB8NNNC" H 6650 1900 50  0001 C CNN "Part Number"
 	1    6650 1900
 	0    -1   -1   0
@@
 F 2 "Capacitor_SMD:C_0603_1608Metric" H 7550 1900 50  0001 C CNN
 F 3 "~" H 7550 1900 50  0001 C CNN
+F 4 "C24452" H 7550 1900 50  0001 C CNN "LCSC"
+F 5 "CL10B104JB8NNNC" H 7550 1900 50  0001 C CNN "Part Number"
 	1    7550 1900
 	0    -1   -1   0
@@
 F 2 "Capacitor_SMD:C_0603_1608Metric" H 4350 1900 50  0001 C CNN
 F 3 "~" H 4350 1900 50  0001 C CNN
+F 4 "C24452" H 4350 1900 50  0001 C CNN "LCSC"
+F 5 "CL10B104JB8NNNC" H 4350 1900 50  0001 C CNN "Part Number"
 	1    4350 1900
 	0    -1   -1   0
@@
 F 2 "Capacitor_SMD:C_0603_1608Metric" H 3800 1900 50  0001 C CNN
 F 3 "~" H 3800 1900 50  0001 C CNN
+F 4 "C24452" H 3800 1900 50  0001 C CNN "LCSC"
+F 5 "CL10B104JB8NNNC" H 3800 1900 50  0001 C CNN "Part Number"
 	1    3800 1900
 	0    -1   -1   0
@@
 F 2 "Capacitor_SMD:C_0603_1608Metric" H 4700 1900 50  0001 C CNN
 F 3 "~" H 4700 1900 50  0001 C CNN
+F 4 "C24452" H 4700 1900 50  0001 C CNN "LCSC"
+F 5 "CL10B104JB8NNNC" H 4700 1900 50  0001 C CNN "Part Number"
 	1    4700 1900
 	0    -1   -1   0
@@
 	7450 1150 7450 1900
 $Comp
-L power:+3.3V #PWR03
+L power:+3.3V #PWR02
 U 1 1 5E277141
 P 2950 2200
-F 0 "#PWR03" H 2950 2050 50  0001 C CNN
+F 0 "#PWR02" H 2950 2050 50  0001 C CNN
 F 1 "+3.3V" H 2965 2373 50  0000 C CNN
 F 2 "" H 2950 2200 50  0001 C CNN
@@
 $EndComp
 $Comp
-L power:+3.3V #PWR020
+L power:+3.3V #PWR021
 U 1 1 5E280F4E
 P 7950 3200
-F 0 "#PWR020" H 7950 3050 50  0001 C CNN
+F 0 "#PWR021" H 7950 3050 50  0001 C CNN
 F 1 "+3.3V" H 7965 3373 50  0000 C CNN
 F 2 "" H 7950 3200 50  0001 C CNN
@@
 	3100 2200 3450 2200
 $Comp
-L power:+3.3V #PWR01
+L power:+3.3V #PWR05
 U 1 1 5E275074
 P 3700 950
-F 0 "#PWR01" H 3700 800 50  0001 C CNN
+F 0 "#PWR05" H 3700 800 50  0001 C CNN
 F 1 "+3.3V" H 3715 1123 50  0000 C CNN
 F 2 "" H 3700 950 50  0001 C CNN

Commit message: I might just have to stick with 1206/4 did some research, maybe time to make another minimal system board....
Parts:
- added C27, C28: 22uf/10v, Capacitor_Tantalum_SMD:CP_EIA-3216-18_Kemet-A, symbol Device:CP1
Connections:
- net +3V3: now also C27.1, C28.1
- net GND: now also C27.2, C28.2
Changed lines of the file:
@@
 	3700 1900 3700 2000
 Wire Wire Line
-	3700 1150 3700 1900
+	3700 1150 3700 1450
 Connection ~ 4250 1900
 Wire Wire Line
@@
 	6550 1900 6550 2000
 Wire Wire Line
-	6550 1150 6550 1900
+	6550 1150 6550 1450
 Connection ~ 7000 1900
 Wire Wire Line
@@
 Wire Wire Line
 	8150 2200 8300 2200
+$Comp
+L Device:CP1 C?
+U 1 1 5E48BFE2
+P 3550 1450
+AR Path="/5E1424B2/5E48BFE2" Ref="C?"  Part="1"
+AR Path="/5EC33E3D/5E48BFE2" Ref="C27"  Part="1"
+F 0 "C27" H 3665 1496 50  0000 L CNN
+F 1 "22uf/10v" H 3665 1405 50  0000 L CNN
+F 2 "Capacitor_Tantalum_SMD:CP_EIA-3216-18_Kemet-A" H 3550 1450 50  0001 C CNN
+F 3 "~" H 3550 1450 50  0001 C CNN
+	1    3550 1450
+	0    1    1    0
+$EndComp
+$Comp
+L power:GND #PWR0101
+U 1 1 5E48D2C3
+P 3400 1450
+F 0 "#PWR0101" H 3400 1200 50  0001 C CNN
+F 1 "GND" H 3405 1277 50  0000 C CNN
+F 2 "" H 3400 1450 50  0001 C CNN
+F 3 "" H 3400 1450 50  0001 C CNN
+	1    3400 1450
+	0    1    1    0
+$EndComp
+$Comp
+L Device:CP1 C?
+U 1 1 5E49004D
+P 6400 1450
+AR Path="/5E1424B2/5E49004D" Ref="C?"  Part="1"
+AR Path="/5EC33E3D/5E49004D" Ref="C28"  Part="1"
+F 0 "C28" H 6515 1496 50  0000 L CNN
+F 1 "22uf/10v" H 6515 1405 50  0000 L CNN
+F 2 "Capacitor_Tantalum_SMD:CP_EIA-3216-18_Kemet-A" H 6400 1450 50  0001 C CNN
+F 3 "~" H 6400 1450 50  0001 C CNN
+	1    6400 1450
+	0    1    1    0
+$EndComp
+$Comp
+L power:GND #PWR0102
+U 1 1 5E490053
+P 6250 1450
+F 0 "#PWR0102" H 6250 1200 50  0001 C CNN
+F 1 "GND" H 6255 1277 50  0000 C CNN
+F 2 "" H 6250 1450 50  0001 C CNN
+F 3 "" H 6250 1450 50  0001 C CNN
+	1    6250 1450
+	0    1    1    0
+$EndComp
+Connection ~ 3700 1450
+Wire Wire Line
+	3700 1450 3700 1900
+Connection ~ 6550 1450
+Wire Wire Line
+	6550 1450 6550 1900
 $EndSCHEMATC
