File: hardware/PCB/RGB.sch (KiCad schematic (older format))
At the start: 22 parts, among them U1 IS31FL3733-QFLS4-TR, U2 IS31FL3733-QFLS4-TR

Commit message: fixing the Tantalum
Parts:
- C27, C28: LCSC (none) -> C11366; Part Number (none) -> TAJA226K010RNJ
Changed lines of the file:
@@
 F 2 "Capacitor_Tantalum_SMD:CP_EIA-3216-18_Kemet-A" H 3550 1450 50  0001 C CNN
 F 3 "~" H 3550 1450 50  0001 C CNN
+F 4 "C11366" H 3550 1450 50  0001 C CNN "LCSC"
+F 5 "TAJA226K010RNJ" H 3550 1450 50  0001 C CNN "Part Number"
 	1    3550 1450
 	0    1    1    0
@@
 F 2 "Capacitor_Tantalum_SMD:CP_EIA-3216-18_Kemet-A" H 6400 1450 50  0001 C CNN
 F 3 "~" H 6400 1450 50  0001 C CNN
+F 4 "C11366" H 6400 1450 50  0001 C CNN "LCSC"
+F 5 "TAJA226K010RNJ" H 6400 1450 50  0001 C CNN "Part Number"
 	1    6400 1450
 	0    1    1    0

Commit message: Fix the button I can't buy... Change part selections for avalibiliby issues
Parts:
- C1, C10, C12, C14, C2, C4, C6, C8: LCSC C1623 -> C170149; Part Number CL10B474KA8NNNC -> CL10A474KB8NNNC
- C11, C13, C3, C5, C7, C9: LCSC C24452 -> C307348; Part Number CL10B104JB8NNNC -> CL10B104KB8WPNC
Changed lines of the file:
@@
 F 2 "Capacitor_SMD:C_0603_1608Metric" H 8150 2100 50  0001 C CNN
 F 3 "~" H 8150 2100 50  0001 C CNN
-F 4 "C1623" H 8150 2100 50  0001 C CNN "LCSC"
-F 5 "CL10B474KA8NNNC" H 8150 2100 50  0001 C CNN "Part Number"
+F 4 "C170149" H 8150 2100 50  0001 C CNN "LCSC"
+F 5 "CL10A474KB8NNNC" H 8150 2100 50  0001 C CNN "Part Number"
 	1    8150 2100
 	-1   0    0    -1
@@
 F 2 "Capacitor_SMD:C_0603_1608Metric" H 3100 2100 50  0001 C CNN
 F 3 "~" H 3100 2100 50  0001 C CNN
-F 4 "C1623" H 3100 2100 50  0001 C CNN "LCSC"
-F 5 "CL10B474KA8NNNC" H 3100 2100 50  0001 C CNN "Part Number"
+F 4 "C170149" H 3100 2100 50  0001 C CNN "LCSC"
+F 5 "CL10A474KB8NNNC" H 3100 2100 50  0001 C CNN "Part Number"
 	1    3100 2100
 	1    0    0    -1
@@
 F 2 "Capacitor_SMD:C_0603_1608Metric" H 7100 1900 50  0001 C CNN
 F 3 "~" H 7100 1900 50  0001 C CNN
-F 4 "C24452" H 7100 1900 50  0001 C CNN "LCSC"
-F 5 "CL10B104JB8NNNC" H 7100 1900 50  0001 C CNN "Part Number"
+F 4 "C307348" H 7100 1900 50  0001 C CNN "LCSC"
+F 5 "CL10B104KB8WPNC" H 7100 1900 50  0001 C CNN "Part Number"
 	1    7100 1900
 	0    -1   -1   0
@@
 F 2 "Capacitor_SMD:C_0603_1608Metric" H 7100 1150 50  0001 C CNN
 F 3 "~" H 7100 1150 50  0001 C CNN
-F 4 "C1623" H 7100 1150 50  0001 C CNN "LCSC"
-F 5 "CL10B474KA8NNNC" H 7100 1150 50  0001 C CNN "Part Number"
+F 4 "C170149" H 7100 1150 50  0001 C CNN "LCSC"
+F 5 "CL10A474KB8NNNC" H 7100 1150 50  0001 C CNN "Part Number"
 	1    7100 1150
 	0    -1   -1   0
@@
 F 2 "Capacitor_SMD:C_0603_1608Metric" H 6650 1900 50  0001 C CNN
 F 3 "~" H 6650 1900 50  0001 C CNN
-F 4 "C24452" H 6650 1900 50  0001 C CNN "LCSC"
-F 5 "CL10B104JB8NNNC" H 6650 1900 50  0001 C CNN "Part Number"
+F 4 "C307348" H 6650 1900 50  0001 C CNN "LCSC"
+F 5 "CL10B104KB8WPNC" H 6650 1900 50  0001 C CNN "Part Number"
 	1    6650 1900
 	0    -1   -1   0
@@
 F 2 "Capacitor_SMD:C_0603_1608Metric" H 6650 1150 50  0001 C CNN
 F 3 "~" H 6650 1150 50  0001 C CNN
-F 4 "C1623" H 6650 1150 50  0001 C CNN "LCSC"
-F 5 "CL10B474KA8NNNC" H 6650 1150 50  0001 C CNN "Part Number"
+F 4 "C170149" H 6650 1150 50  0001 C CNN "LCSC"
+F 5 "CL10A474KB8NNNC" H 6650 1150 50  0001 C CNN "Part Number"
 	1    6650 1150
 	0    -1   -1   0
@@
 F 2 "Capacitor_SMD:C_0603_1608Metric" H 7550 1900 50  0001 C CNN
 F 3 "~" H 7550 1900 50  0001 C CNN
-F 4 "C24452" H 7550 1900 50  0001 C CNN "LCSC"
-F 5 "CL10B104JB8NNNC" H 7550 1900 50  0001 C CNN "Part Number"
+F 4 "C307348" H 7550 1900 50  0001 C CNN "LCSC"
+F 5 "CL10B104KB8WPNC" H 7550 1900 50  0001 C CNN "Part Number"
 	1    7550 1900
 	0    -1   -1   0
@@
 F 2 "Capacitor_SMD:C_0603_1608Metric" H 7550 1150 50  0001 C CNN
 F 3 "~" H 7550 1150 50  0001 C CNN
-F 4 "C1623" H 7550 1150 50  0001 C CNN "LCSC"
-F 5 "CL10B474KA8NNNC" H 7550 1150 50  0001 C CNN "Part Number"
+F 4 "C170149" H 7550 1150 50  0001 C CNN "LCSC"
+F 5 "CL10A474KB8NNNC" H 7550 1150 50  0001 C CNN "Part Number"
 	1    7550 1150
 	0    -1   -1   0
@@
 F 2 "Capacitor_SMD:C_0603_1608Metric" H 4350 1900 50  0001 C CNN
 F 3 "~" H 4350 1900 50  0001 C CNN
-F 4 "C24452" H 4350 1900 50  0001 C CNN "LCSC"
-F 5 "CL10B104JB8NNNC" H 4350 1900 50  0001 C CNN "Part Number"
+F 4 "C307348" H 4350 1900 50  0001 C CNN "LCSC"
+F 5 "CL10B104KB8WPNC" H 4350 1900 50  0001 C CNN "Part Number"
 	1    4350 1900
 	0    -1   -1   0
@@
 F 2 "Capacitor_SMD:C_0603_1608Metric" H 4350 1150 50  0001 C CNN
 F 3 "~" H 4350 1150 50  0001 C CNN
-F 4 "C1623" H 4350 1150 50  0001 C CNN "LCSC"
-F 5 "CL10B474KA8NNNC" H 4350 1150 50  0001 C CNN "Part Number"
+F 4 "C170149" H 4350 1150 50  0001 C CNN "LCSC"
+F 5 "CL10A474KB8NNNC" H 4350 1150 50  0001 C CNN "Part Number"
 	1    4350 1150
 	0    -1   -1   0
@@
 F 2 "Capacitor_SMD:C_0603_1608Metric" H 3800 1900 50  0001 C CNN
 F 3 "~" H 3800 1900 50  0001 C CNN
-F 4 "C24452" H 3800 1900 50  0001 C CNN "LCSC"
-F 5 "CL10B104JB8NNNC" H 3800 1900 50  0001 C CNN "Part Number"
+F 4 "C307348" H 3800 1900 50  0001 C CNN "LCSC"
+F 5 "CL10B104KB8WPNC" H 3800 1900 50  0001 C CNN "Part Number"
 	1    3800 1900
 	0    -1   -1   0
@@
 F 2 "Capacitor_SMD:C_0603_1608Metric" H 3800 1150 50  0001 C CNN
 F 3 "~" H 3800 1150 50  0001 C CNN
-F 4 "C1623" H 3800 1150 50  0001 C CNN "LCSC"
-F 5 "CL10B474KA8NNNC" H 3800 1150 50  0001 C CNN "Part Number"
+F 4 "C170149" H 3800 1150 50  0001 C CNN "LCSC"
+F 5 "CL10A474KB8NNNC" H 3800 1150 50  0001 C CNN "Part Number"
 	1    3800 1150
 	0    -1   -1   0
@@
 F 2 "Capacitor_SMD:C_0603_1608Metric" H 4700 1900 50  0001 C CNN
 F 3 "~" H 4700 1900 50  0001 C CNN
-F 4 "C24452" H 4700 1900 50  0001 C CNN "LCSC"
-F 5 "CL10B104JB8NNNC" H 4700 1900 50  0001 C CNN "Part Number"
+F 4 "C307348" H 4700 1900 50  0001 C CNN "LCSC"
+F 5 "CL10B104KB8WPNC" H 4700 1900 50  0001 C CNN "Part Number"
 	1    4700 1900
 	0    -1   -1   0
@@
 F 2 "Capacitor_SMD:C_0603_1608Metric" H 4700 1150 50  0001 C CNN
 F 3 "~" H 4700 1150 50  0001 C CNN
-F 4 "C1623" H 4700 1150 50  0001 C CNN "LCSC"
-F 5 "CL10B474KA8NNNC" H 4700 1150 50  0001 C CNN "Part Number"
+F 4 "C170149" H 4700 1150 50  0001 C CNN "LCSC"
+F 5 "CL10A474KB8NNNC" H 4700 1150 50  0001 C CNN "Part Number"
 	1    4700 1150
 	0    -1   -1   0
