File: hardware/PCB/RGBMatrix2.sch (KiCad schematic (older format))
At the start: 27 parts

Commit message: Now it should be working just fine
Parts:
- D69, D70, D71, D72, D73, D74, D75, D76, D77, D78, D79, D80, D81, D82, D83, D84, D85, D86, D87, D88, D89, D90, D91, D92, D93, D94, D95: Footprint KiCad:XZMDKCBDDG45S9_fixed -> (none); Value XZMDKCBDDG45S9 -> (none)
Changed lines of the file:
@@
 F 2 "KiCad:XZMDKCBDDG45S9_fixed" H 1750 2350 50  0001 C CNN
 F 3 "~" H 1750 2350 50  0001 C CNN
-F 4 "KiCad:XZMDKCBDDG45S9_fixed" H 1750 2400 50  0001 C CNN "Footprint"
-F 5 "XZMDKCBDDG45S9" H 1750 2400 50  0001 C CNN "Value"
 	1    1750 2400
 	1    0    0    -1
@@
 F 2 "KiCad:XZMDKCBDDG45S9_fixed" H 2350 2350 50  0001 C CNN
 F 3 "~" H 2350 2350 50  0001 C CNN
-F 4 "KiCad:XZMDKCBDDG45S9_fixed" H 2350 2400 50  0001 C CNN "Footprint"
-F 5 "XZMDKCBDDG45S9" H 2350 2400 50  0001 C CNN "Value"
 	1    2350 2400
 	1    0    0    -1
@@
 F 2 "KiCad:XZMDKCBDDG45S9_fixed" H 2950 2350 50  0001 C CNN
 F 3 "~" H 2950 2350 50  0001 C CNN
-F 4 "KiCad:XZMDKCBDDG45S9_fixed" H 2950 2400 50  0001 C CNN "Footprint"
-F 5 "XZMDKCBDDG45S9" H 2950 2400 50  0001 C CNN "Value"
 	1    2950 2400
 	1    0    0    -1
@@
 F 2 "KiCad:XZMDKCBDDG45S9_fixed" H 3550 2350 50  0001 C CNN
 F 3 "~" H 3550 2350 50  0001 C CNN
-F 4 "KiCad:XZMDKCBDDG45S9_fixed" H 3550 2400 50  0001 C CNN "Footprint"
-F 5 "XZMDKCBDDG45S9" H 3550 2400 50  0001 C CNN "Value"
 	1    3550 2400
 	1    0    0    -1
@@
 F 2 "KiCad:XZMDKCBDDG45S9_fixed" H 4100 2350 50  0001 C CNN
 F 3 "~" H 4100 2350 50  0001 C CNN
-F 4 "KiCad:XZMDKCBDDG45S9_fixed" H 4100 2400 50  0001 C CNN "Footprint"
-F 5 "XZMDKCBDDG45S9" H 4100 2400 50  0001 C CNN "Value"
 	1    4100 2400
 	1    0    0    -1
@@
 F 2 "KiCad:XZMDKCBDDG45S9_fixed" H 4700 2350 50  0001 C CNN
 F 3 "~" H 4700 2350 50  0001 C CNN
-F 4 "KiCad:XZMDKCBDDG45S9_fixed" H 4700 2400 50  0001 C CNN "Footprint"
-F 5 "XZMDKCBDDG45S9" H 4700 2400 50  0001 C CNN "Value"
 	1    4700 2400
 	1    0    0    -1
@@
 F 2 "KiCad:XZMDKCBDDG45S9_fixed" H 5300 2350 50  0001 C CNN
 F 3 "~" H 5300 2350 50  0001 C CNN
-F 4 "KiCad:XZMDKCBDDG45S9_fixed" H 5300 2400 50  0001 C CNN "Footprint"
-F 5 "XZMDKCBDDG45S9" H 5300 2400 50  0001 C CNN "Value"
 	1    5300 2400
 	1    0    0    -1
@@
 F 2 "KiCad:XZMDKCBDDG45S9_fixed" H 5900 2350 50  0001 C CNN
 F 3 "~" H 5900 2350 50  0001 C CNN
-F 4 "KiCad:XZMDKCBDDG45S9_fixed" H 5900 2400 50  0001 C CNN "Footprint"
-F 5 "XZMDKCBDDG45S9" H 5900 2400 50  0001 C CNN "Value"
 	1    5900 2400
 	1    0    0    -1
@@
 F 2 "KiCad:XZMDKCBDDG45S9_fixed" H 6500 2350 50  0001 C CNN
 F 3 "~" H 6500 2350 50  0001 C CNN
-F 4 "KiCad:XZMDKCBDDG45S9_fixed" H 6500 2400 50  0001 C CNN "Footprint"
-F 5 "XZMDKCBDDG45S9" H 6500 2400 50  0001 C CNN "Value"
 	1    6500 2400
 	1    0    0    -1
@@
 F 2 "KiCad:XZMDKCBDDG45S9_fixed" H 7100 2350 50  0001 C CNN
 F 3 "~" H 7100 2350 50  0001 C CNN
-F 4 "KiCad:XZMDKCBDDG45S9_fixed" H 7100 2400 50  0001 C CNN "Footprint"
-F 5 "XZMDKCBDDG45S9" H 7100 2400 50  0001 C CNN "Value"
 	1    7100 2400
 	1    0    0    -1
@@
 F 2 "KiCad:XZMDKCBDDG45S9_fixed" H 7700 2350 50  0001 C CNN
 F 3 "~" H 7700 2350 50  0001 C CNN
-F 4 "KiCad:XZMDKCBDDG45S9_fixed" H 7700 2400 50  0001 C CNN "Footprint"
-F 5 "XZMDKCBDDG45S9" H 7700 2400 50  0001 C CNN "Value"
 	1    7700 2400
 	1    0    0    -1
@@
 F 2 "KiCad:XZMDKCBDDG45S9_fixed" H 8300 2350 50  0001 C CNN
 F 3 "~" H 8300 2350 50  0001 C CNN
-F 4 "KiCad:XZMDKCBDDG45S9_fixed" H 8300 2400 50  0001 C CNN "Footprint"
-F 5 "XZMDKCBDDG45S9" H 8300 2400 50  0001 C CNN "Value"
 	1    8300 2400
 	1    0    0    -1
@@
 F 2 "KiCad:XZMDKCBDDG45S9_fixed" H 8900 2350 50  0001 C CNN
 F 3 "~" H 8900 2350 50  0001 C CNN
-F 4 "KiCad:XZMDKCBDDG45S9_fixed" H 8900 2400 50  0001 C CNN "Footprint"
-F 5 "XZMDKCBDDG45S9" H 8900 2400 50  0001 C CNN "Value"
 	1    8900 2400
 	1    0    0    -1
@@
 F 2 "KiCad:XZMDKCBDDG45S9_fixed" H 9500 2350 50  0001 C CNN
 F 3 "~" H 9500 2350 50  0001 C CNN
-F 4 "KiCad:XZMDKCBDDG45S9_fixed" H 9500 2400 50  0001 C CNN "Footprint"
-F 5 "XZMDKCBDDG45S9" H 9500 2400 50  0001 C CNN "Value"
 	1    9500 2400
 	1    0    0    -1
@@
 F 2 "KiCad:XZMDKCBDDG45S9_fixed" H 9500 3400 50  0001 C CNN
 F 3 "~" H 9500 3400 50  0001 C CNN
-F 4 "KiCad:XZMDKCBDDG45S9_fixed" H 9500 3450 50  0001 C CNN "Footprint"
-F 5 "XZMDKCBDDG45S9" H 9500 3450 50  0001 C CNN "Value"
 	1    9500 3450
 	1    0    0    -1
@@
 F 2 "KiCad:XZMDKCBDDG45S9_fixed" H 8300 3400 50  0001 C CNN
 F 3 "~" H 8300 3400 50  0001 C CNN
-F 4 "KiCad:XZMDKCBDDG45S9_fixed" H 8300 3450 50  0001 C CNN "Footprint"
-F 5 "XZMDKCBDDG45S9" H 8300 3450 50  0001 C CNN "Value"
 	1    8300 3450
 	1    0    0    -1
@@
 F 2 "KiCad:XZMDKCBDDG45S9_fixed" H 7700 3400 50  0001 C CNN
 F 3 "~" H 7700 3400 50  0001 C CNN
-F 4 "KiCad:XZMDKCBDDG45S9_fixed" H 7700 3450 50  0001 C CNN "Footprint"
-F 5 "XZMDKCBDDG45S9" H 7700 3450 50  0001 C CNN "Value"
 	1    7700 3450
 	1    0    0    -1
@@
 F 2 "KiCad:XZMDKCBDDG45S9_fixed" H 7100 3400 50  0001 C CNN
 F 3 "~" H 7100 3400 50  0001 C CNN
-F 4 "KiCad:XZMDKCBDDG45S9_fixed" H 7100 3450 50  0001 C CNN "Footprint"
-F 5 "XZMDKCBDDG45S9" H 7100 3450 50  0001 C CNN "Value"
 	1    7100 3450
 	1    0    0    -1
@@
 F 2 "KiCad:XZMDKCBDDG45S9_fixed" H 6500 3400 50  0001 C CNN
 F 3 "~" H 6500 3400 50  0001 C CNN
-F 4 "KiCad:XZMDKCBDDG45S9_fixed" H 6500 3450 50  0001 C CNN "Footprint"
-F 5 "XZMDKCBDDG45S9" H 6500 3450 50  0001 C CNN "Value"
 	1    6500 3450
 	1    0    0    -1
@@
 F 2 "KiCad:XZMDKCBDDG45S9_fixed" H 5900 3400 50  0001 C CNN
 F 3 "~" H 5900 3400 50  0001 C CNN
-F 4 "KiCad:XZMDKCBDDG45S9_fixed" H 5900 3450 50  0001 C CNN "Footprint"
-F 5 "XZMDKCBDDG45S9" H 5900 3450 50  0001 C CNN "Value"
 	1    5900 3450
 	1    0    0    -1
@@
 F 2 "KiCad:XZMDKCBDDG45S9_fixed" H 4700 3400 50  0001 C CNN
 F 3 "~" H 4700 3400 50  0001 C CNN
-F 4 "KiCad:XZMDKCBDDG45S9_fixed" H 4700 3450 50  0001 C CNN "Footprint"
-F 5 "XZMDKCBDDG45S9" H 4700 3450 50  0001 C CNN "Value"
 	1    4700 3450
 	1    0    0    -1
@@
 F 2 "KiCad:XZMDKCBDDG45S9_fixed" H 4100 3400 50  0001 C CNN
 F 3 "~" H 4100 3400 50  0001 C CNN
-F 4 "KiCad:XZMDKCBDDG45S9_fixed" H 4100 3450 50  0001 C CNN "Footprint"
-F 5 "XZMDKCBDDG45S9" H 4100 3450 50  0001 C CNN "Value"
 	1    4100 3450
 	1    0    0    -1
@@
 F 2 "KiCad:XZMDKCBDDG45S9_fixed" H 3550 3400 50  0001 C CNN
 F 3 "~" H 3550 3400 50  0001 C CNN
-F 4 "KiCad:XZMDKCBDDG45S9_fixed" H 3550 3450 50  0001 C CNN "Footprint"
-F 5 "XZMDKCBDDG45S9" H 3550 3450 50  0001 C CNN "Value"
 	1    3550 3450
 	1    0    0    -1
@@
 F 2 "KiCad:XZMDKCBDDG45S9_fixed" H 2950 3400 50  0001 C CNN
 F 3 "~" H 2950 3400 50  0001 C CNN
-F 4 "KiCad:XZMDKCBDDG45S9_fixed" H 2950 3450 50  0001 C CNN "Footprint"
-F 5 "XZMDKCBDDG45S9" H 2950 3450 50  0001 C CNN "Value"
 	1    2950 3450
 	1    0    0    -1
@@
 F 2 "KiCad:XZMDKCBDDG45S9_fixed" H 2350 3400 50  0001 C CNN
 F 3 "~" H 2350 3400 50  0001 C CNN
-F 4 "KiCad:XZMDKCBDDG45S9_fixed" H 2350 3450 50  0001 C CNN "Footprint"
-F 5 "XZMDKCBDDG45S9" H 2350 3450 50  0001 C CNN "Value"
 	1    2350 3450
 	1    0    0    -1
@@
 F 2 "KiCad:XZMDKCBDDG45S9_fixed" H 1750 3400 50  0001 C CNN
 F 3 "~" H 1750 3400 50  0001 C CNN
-F 4 "KiCad:XZMDKCBDDG45S9_fixed" H 1750 3450 50  0001 C CNN "Footprint"
-F 5 "XZMDKCBDDG45S9" H 1750 3450 50  0001 C CNN "Value"
 	1    1750 3450
 	1    0    0    -1
@@
 F 2 "KiCad:XZMDKCBDDG45S9_fixed" H 8900 3400 50  0001 C CNN
 F 3 "~" H 8900 3400 50  0001 C CNN
-F 4 "KiCad:XZMDKCBDDG45S9_fixed" H 8900 3450 50  0001 C CNN "Footprint"
-F 5 "XZMDKCBDDG45S9" H 8900 3450 50  0001 C CNN "Value"
 	1    8900 3450
 	1    0    0    -1

Commit message: add in part number so I could use it for the bom
Parts:
- D69, D70, D71, D72, D73, D74, D75, D76, D77, D78, D79, D80, D81, D82, D83, D84, D85, D86, D87, D88, D89, D90, D91, D92, D93, D94, D95: Part Number (none) -> XZMDKCBDDG45S-9
Changed lines of the file:
@@
 F 1 "XZMDKCBDDG45S-9" H 1750 2806 50  0000 C CNN
 F 2 "KiCad:XZMDKCBDDG45S9_fixed" H 1750 2350 50  0001 C CNN
-F 3 "~" H 1750 2350 50  0001 C CNN
+F 3 "https://www.sunledusa.com/products/spec/XZMDKCBDDG45S-9.pdf" H 1750 2350 50  0001 C CNN
+F 4 "XZMDKCBDDG45S-9" H 1750 2400 50  0001 C CNN "Part Number"
 	1    1750 2400
 	1    0    0    -1
@@
 F 1 "XZMDKCBDDG45S-9" H 2350 2806 50  0000 C CNN
 F 2 "KiCad:XZMDKCBDDG45S9_fixed" H 2350 2350 50  0001 C CNN
-F 3 "~" H 2350 2350 50  0001 C CNN
+F 3 "https://www.sunledusa.com/products/spec/XZMDKCBDDG45S-9.pdf" H 2350 2350 50  0001 C CNN
+F 4 "XZMDKCBDDG45S-9" H 2350 2400 50  0001 C CNN "Part Number"
 	1    2350 2400
 	1    0    0    -1
@@
 F 1 "XZMDKCBDDG45S-9" H 2950 2806 50  0000 C CNN
 F 2 "KiCad:XZMDKCBDDG45S9_fixed" H 2950 2350 50  0001 C CNN
-F 3 "~" H 2950 2350 50  0001 C CNN
+F 3 "https://www.sunledusa.com/products/spec/XZMDKCBDDG45S-9.pdf" H 2950 2350 50  0001 C CNN
+F 4 "XZMDKCBDDG45S-9" H 2950 2400 50  0001 C CNN "Part Number"
 	1    2950 2400
 	1    0    0    -1
@@
 F 1 "XZMDKCBDDG45S-9" H 3550 2806 50  0000 C CNN
 F 2 "KiCad:XZMDKCBDDG45S9_fixed" H 3550 2350 50  0001 C CNN
-F 3 "~" H 3550 2350 50  0001 C CNN
+F 3 "https://www.sunledusa.com/products/spec/XZMDKCBDDG45S-9.pdf" H 3550 2350 50  0001 C CNN
+F 4 "XZMDKCBDDG45S-9" H 3550 2400 50  0001 C CNN "Part Number"
 	1    3550 2400
 	1    0    0    -1
@@
 F 1 "XZMDKCBDDG45S-9" H 4100 2806 50  0000 C CNN
 F 2 "KiCad:XZMDKCBDDG45S9_fixed" H 4100 2350 50  0001 C CNN
-F 3 "~" H 4100 2350 50  0001 C CNN
+F 3 "https://www.sunledusa.com/products/spec/XZMDKCBDDG45S-9.pdf" H 4100 2350 50  0001 C CNN
+F 4 "XZMDKCBDDG45S-9" H 4100 2400 50  0001 C CNN "Part Number"
 	1    4100 2400
 	1    0    0    -1
@@
 F 1 "XZMDKCBDDG45S-9" H 4700 2806 50  0000 C CNN
 F 2 "KiCad:XZMDKCBDDG45S9_fixed" H 4700 2350 50  0001 C CNN
-F 3 "~" H 4700 2350 50  0001 C CNN
+F 3 "https://www.sunledusa.com/products/spec/XZMDKCBDDG45S-9.pdf" H 4700 2350 50  0001 C CNN
+F 4 "XZMDKCBDDG45S-9" H 4700 2400 50  0001 C CNN "Part Number"
 	1    4700 2400
 	1    0    0    -1
@@
 F 1 "XZMDKCBDDG45S-9" H 5300 2806 50  0000 C CNN
 F 2 "KiCad:XZMDKCBDDG45S9_fixed" H 5300 2350 50  0001 C CNN
-F 3 "~" H 5300 2350 50  0001 C CNN
+F 3 "https://www.sunledusa.com/products/spec/XZMDKCBDDG45S-9.pdf" H 5300 2350 50  0001 C CNN
+F 4 "XZMDKCBDDG45S-9" H 5300 2400 50  0001 C CNN "Part Number"
 	1    5300 2400
 	1    0    0    -1
@@
 F 1 "XZMDKCBDDG45S-9" H 5900 2806 50  0000 C CNN
 F 2 "KiCad:XZMDKCBDDG45S9_fixed" H 5900 2350 50  0001 C CNN
-F 3 "~" H 5900 2350 50  0001 C CNN
+F 3 "https://www.sunledusa.com/products/spec/XZMDKCBDDG45S-9.pdf" H 5900 2350 50  0001 C CNN
+F 4 "XZMDKCBDDG45S-9" H 5900 2400 50  0001 C CNN "Part Number"
 	1    5900 2400
 	1    0    0    -1
@@
 F 1 "XZMDKCBDDG45S-9" H 6500 2806 50  0000 C CNN
 F 2 "KiCad:XZMDKCBDDG45S9_fixed" H 6500 2350 50  0001 C CNN
-F 3 "~" H 6500 2350 50  0001 C CNN
+F 3 "https://www.sunledusa.com/products/spec/XZMDKCBDDG45S-9.pdf" H 6500 2350 50  0001 C CNN
+F 4 "XZMDKCBDDG45S-9" H 6500 2400 50  0001 C CNN "Part Number"
 	1    6500 2400
 	1    0    0    -1
@@
 F 1 "XZMDKCBDDG45S-9" H 7100 2806 50  0000 C CNN
 F 2 "KiCad:XZMDKCBDDG45S9_fixed" H 7100 2350 50  0001 C CNN
-F 3 "~" H 7100 2350 50  0001 C CNN
+F 3 "https://www.sunledusa.com/products/spec/XZMDKCBDDG45S-9.pdf" H 7100 2350 50  0001 C CNN
+F 4 "XZMDKCBDDG45S-9" H 7100 2400 50  0001 C CNN "Part Number"
 	1    7100 2400
 	1    0    0    -1
@@
 F 1 "XZMDKCBDDG45S-9" H 7700 2806 50  0000 C CNN
 F 2 "KiCad:XZMDKCBDDG45S9_fixed" H 7700 2350 50  0001 C CNN
-F 3 "~" H 7700 2350 50  0001 C CNN
+F 3 "https://www.sunledusa.com/products/spec/XZMDKCBDDG45S-9.pdf" H 7700 2350 50  0001 C CNN
+F 4 "XZMDKCBDDG45S-9" H 7700 2400 50  0001 C CNN "Part Number"
 	1    7700 2400
 	1    0    0    -1
@@
 F 1 "XZMDKCBDDG45S-9" H 8300 2806 50  0000 C CNN
 F 2 "KiCad:XZMDKCBDDG45S9_fixed" H 8300 2350 50  0001 C CNN
-F 3 "~" H 8300 2350 50  0001 C CNN
+F 3 "https://www.sunledusa.com/products/spec/XZMDKCBDDG45S-9.pdf" H 8300 2350 50  0001 C CNN
+F 4 "XZMDKCBDDG45S-9" H 8300 2400 50  0001 C CNN "Part Number"
 	1    8300 2400
 	1    0    0    -1
@@
 F 1 "XZMDKCBDDG45S-9" H 8900 2806 50  0000 C CNN
 F 2 "KiCad:XZMDKCBDDG45S9_fixed" H 8900 2350 50  0001 C CNN
-F 3 "~" H 8900 2350 50  0001 C CNN
+F 3 "https://www.sunledusa.com/products/spec/XZMDKCBDDG45S-9.pdf" H 8900 2350 50  0001 C CNN
+F 4 "XZMDKCBDDG45S-9" H 8900 2400 50  0001 C CNN "Part Number"
 	1    8900 2400
 	1    0    0    -1
@@
 F 1 "XZMDKCBDDG45S-9" H 9500 2806 50  0000 C CNN
 F 2 "KiCad:XZMDKCBDDG45S9_fixed" H 9500 2350 50  0001 C CNN
-F 3 "~" H 9500 2350 50  0001 C CNN
+F 3 "https://www.sunledusa.com/products/spec/XZMDKCBDDG45S-9.pdf" H 9500 2350 50  0001 C CNN
+F 4 "XZMDKCBDDG45S-9" H 9500 2400 50  0001 C CNN "Part Number"
 	1    9500 2400
 	1    0    0    -1
@@
 F 1 "XZMDKCBDDG45S-9" H 9500 3856 50  0000 C CNN
 F 2 "KiCad:XZMDKCBDDG45S9_fixed" H 9500 3400 50  0001 C CNN
-F 3 "~" H 9500 3400 50  0001 C CNN
+F 3 "https://www.sunledusa.com/products/spec/XZMDKCBDDG45S-9.pdf" H 9500 3400 50  0001 C CNN
+F 4 "XZMDKCBDDG45S-9" H 9500 3450 50  0001 C CNN "Part Number"
 	1    9500 3450
 	1    0    0    -1
@@
 F 1 "XZMDKCBDDG45S-9" H 8300 3856 50  0000 C CNN
 F 2 "KiCad:XZMDKCBDDG45S9_fixed" H 8300 3400 50  0001 C CNN
-F 3 "~" H 8300 3400 50  0001 C CNN
+F 3 "https://www.sunledusa.com/products/spec/XZMDKCBDDG45S-9.pdf" H 8300 3400 50  0001 C CNN
+F 4 "XZMDKCBDDG45S-9" H 8300 3450 50  0001 C CNN "Part Number"
 	1    8300 3450
 	1    0    0    -1
@@
 F 1 "XZMDKCBDDG45S-9" H 7700 3856 50  0000 C CNN
 F 2 "KiCad:XZMDKCBDDG45S9_fixed" H 7700 3400 50  0001 C CNN
-F 3 "~" H 7700 3400 50  0001 C CNN
+F 3 "https://www.sunledusa.com/products/spec/XZMDKCBDDG45S-9.pdf" H 7700 3400 50  0001 C CNN
+F 4 "XZMDKCBDDG45S-9" H 7700 3450 50  0001 C CNN "Part Number"
 	1    7700 3450
 	1    0    0    -1
@@
 F 1 "XZMDKCBDDG45S-9" H 7100 3856 50  0000 C CNN
 F 2 "KiCad:XZMDKCBDDG45S9_fixed" H 7100 3400 50  0001 C CNN
-F 3 "~" H 7100 3400 50  0001 C CNN
+F 3 "https://www.sunledusa.com/products/spec/XZMDKCBDDG45S-9.pdf" H 7100 3400 50  0001 C CNN
+F 4 "XZMDKCBDDG45S-9" H 7100 3450 50  0001 C CNN "Part Number"
 	1    7100 3450
 	1    0    0    -1
@@
 F 1 "XZMDKCBDDG45S-9" H 6500 3856 50  0000 C CNN
 F 2 "KiCad:XZMDKCBDDG45S9_fixed" H 6500 3400 50  0001 C CNN
-F 3 "~" H 6500 3400 50  0001 C CNN
+F 3 "https://www.sunledusa.com/products/spec/XZMDKCBDDG45S-9.pdf" H 6500 3400 50  0001 C CNN
+F 4 "XZMDKCBDDG45S-9" H 6500 3450 50  0001 C CNN "Part Number"
 	1    6500 3450
 	1    0    0    -1
@@
 F 1 "XZMDKCBDDG45S-9" H 5900 3856 50  0000 C CNN
 F 2 "KiCad:XZMDKCBDDG45S9_fixed" H 5900 3400 50  0001 C CNN
-F 3 "~" H 5900 3400 50  0001 C CNN
+F 3 "https://www.sunledusa.com/products/spec/XZMDKCBDDG45S-9.pdf" H 5900 3400 50  0001 C CNN
+F 4 "XZMDKCBDDG45S-9" H 5900 3450 50  0001 C CNN "Part Number"
 	1    5900 3450
 	1    0    0    -1
@@
 F 1 "XZMDKCBDDG45S-9" H 4700 3856 50  0000 C CNN
 F 2 "KiCad:XZMDKCBDDG45S9_fixed" H 4700 3400 50  0001 C CNN
-F 3 "~" H 4700 3400 50  0001 C CNN
+F 3 "https://www.sunledusa.com/products/spec/XZMDKCBDDG45S-9.pdf" H 4700 3400 50  0001 C CNN
+F 4 "XZMDKCBDDG45S-9" H 4700 3450 50  0001 C CNN "Part Number"
 	1    4700 3450
 	1    0    0    -1
@@
 F 1 "XZMDKCBDDG45S-9" H 4100 3856 50  0000 C CNN
 F 2 "KiCad:XZMDKCBDDG45S9_fixed" H 4100 3400 50  0001 C CNN
-F 3 "~" H 4100 3400 50  0001 C CNN
+F 3 "https://www.sunledusa.com/products/spec/XZMDKCBDDG45S-9.pdf" H 4100 3400 50  0001 C CNN
+F 4 "XZMDKCBDDG45S-9" H 4100 3450 50  0001 C CNN "Part Number"
 	1    4100 3450
 	1    0    0    -1
@@
 F 1 "XZMDKCBDDG45S-9" H 3550 3856 50  0000 C CNN
 F 2 "KiCad:XZMDKCBDDG45S9_fixed" H 3550 3400 50  0001 C CNN
-F 3 "~" H 3550 3400 50  0001 C CNN
+F 3 "https://www.sunledusa.com/products/spec/XZMDKCBDDG45S-9.pdf" H 3550 3400 50  0001 C CNN
+F 4 "XZMDKCBDDG45S-9" H 3550 3450 50  0001 C CNN "Part Number"
 	1    3550 3450
 	1    0    0    -1
@@
 F 1 "XZMDKCBDDG45S-9" H 2950 3856 50  0000 C CNN
 F 2 "KiCad:XZMDKCBDDG45S9_fixed" H 2950 3400 50  0001 C CNN
-F 3 "~" H 2950 3400 50  0001 C CNN
+F 3 "https://www.sunledusa.com/products/spec/XZMDKCBDDG45S-9.pdf" H 2950 3400 50  0001 C CNN
+F 4 "XZMDKCBDDG45S-9" H 2950 3450 50  0001 C CNN "Part Number"
 	1    2950 3450
 	1    0    0    -1
@@
 F 1 "XZMDKCBDDG45S-9" H 2350 3856 50  0000 C CNN
 F 2 "KiCad:XZMDKCBDDG45S9_fixed" H 2350 3400 50  0001 C CNN
-F 3 "~" H 2350 3400 50  0001 C CNN
+F 3 "https://www.sunledusa.com/products/spec/XZMDKCBDDG45S-9.pdf" H 2350 3400 50  0001 C CNN
+F 4 "XZMDKCBDDG45S-9" H 2350 3450 50  0001 C CNN "Part Number"
 	1    2350 3450
 	1    0    0    -1
@@
 F 1 "XZMDKCBDDG45S-9" H 1750 3856 50  0000 C CNN
 F 2 "KiCad:XZMDKCBDDG45S9_fixed" H 1750 3400 50  0001 C CNN
-F 3 "~" H 1750 3400 50  0001 C CNN
+F 3 "https://www.sunledusa.com/products/spec/XZMDKCBDDG45S-9.pdf" H 1750 3400 50  0001 C CNN
+F 4 "XZMDKCBDDG45S-9" H 1750 3450 50  0001 C CNN "Part Number"
 	1    1750 3450
 	1    0    0    -1
@@
 F 1 "XZMDKCBDDG45S-9" H 8900 3856 50  0000 C CNN
 F 2 "KiCad:XZMDKCBDDG45S9_fixed" H 8900 3400 50  0001 C CNN
-F 3 "~" H 8900 3400 50  0001 C CNN
+F 3 "https://www.sunledusa.com/products/spec/XZMDKCBDDG45S-9.pdf" H 8900 3400 50  0001 C CNN
+F 4 "XZMDKCBDDG45S-9" H 8900 3450 50  0001 C CNN "Part Number"
 	1    8900 3450
 	1    0    0    -1

Commit message: update render, remove useless files, fix the decoupeling
Parts:
- renumbered D69 to D110, D70 to D111, D71 to D112, D72 to D113, D73 to D114, D74 to D115, D75 to D116, D76 to D117, D77 to D118, D78 to D119, D79 to D120, D80 to D121, D81 to D122, D82 to D123, D83 to D124, D84 to D125, D85 to D126, D86 to D127, D87 to D128, D88 to D129, D89 to D130, D90 to D131, D91 to D132, D92 to D133, D93 to D134, D94 to D135, D95 to D136
