File: hardware/PCB/RGBMatrix2.sch (KiCad schematic (older format))
At the start: 27 parts

Commit message: Remove some unused
Parts:
- D110, D111, D112, D113, D114, D115, D116, D117, D118, D119, D120, D121, D122, D123, D124, D125, D126, D127, D128, D129, D130, D131, D132, D133, D134, D135, D136: footprint KiCad:RGB_LED_1205 -> KiCad:RGB_LED_1204_reverse
Changed lines of the file:
@@
 F 0 "D110" H 2150 3747 50  0000 C CNN
 F 1 "RABG" H 2150 3656 50  0000 C CNN
-F 2 "KiCad:RGB_LED_1205" H 2150 3200 50  0001 C CNN
+F 2 "KiCad:RGB_LED_1204_reverse" H 2150 3200 50  0001 C CNN
 F 3 "https://datasheet.lcsc.com/szlcsc/1912111437_MEIHUA-MHT150RGBCT_C409782.pdf" H 2150 3200 50  0001 C CNN
 F 4 "MHT150RGBCT" H 2150 3250 50  0001 C CNN "Part Number"
@@
 F 0 "D112" H 2750 3747 50  0000 C CNN
 F 1 "RABG" H 2750 3656 50  0000 C CNN
-F 2 "KiCad:RGB_LED_1205" H 2750 3200 50  0001 C CNN
+F 2 "KiCad:RGB_LED_1204_reverse" H 2750 3200 50  0001 C CNN
 F 3 "https://datasheet.lcsc.com/szlcsc/1912111437_MEIHUA-MHT150RGBCT_C409782.pdf" H 2750 3200 50  0001 C CNN
 F 4 "MHT150RGBCT" H 2750 3250 50  0001 C CNN "Part Number"
@@
 F 0 "D114" H 3350 3747 50  0000 C CNN
 F 1 "RABG" H 3350 3656 50  0000 C CNN
-F 2 "KiCad:RGB_LED_1205" H 3350 3200 50  0001 C CNN
+F 2 "KiCad:RGB_LED_1204_reverse" H 3350 3200 50  0001 C CNN
 F 3 "https://datasheet.lcsc.com/szlcsc/1912111437_MEIHUA-MHT150RGBCT_C409782.pdf" H 3350 3200 50  0001 C CNN
 F 4 "MHT150RGBCT" H 3350 3250 50  0001 C CNN "Part Number"
@@
 F 0 "D116" H 3950 3747 50  0000 C CNN
 F 1 "RABG" H 3950 3656 50  0000 C CNN
-F 2 "KiCad:RGB_LED_1205" H 3950 3200 50  0001 C CNN
+F 2 "KiCad:RGB_LED_1204_reverse" H 3950 3200 50  0001 C CNN
 F 3 "https://datasheet.lcsc.com/szlcsc/1912111437_MEIHUA-MHT150RGBCT_C409782.pdf" H 3950 3200 50  0001 C CNN
 F 4 "MHT150RGBCT" H 3950 3250 50  0001 C CNN "Part Number"
@@
 F 0 "D118" H 4500 3747 50  0000 C CNN
 F 1 "RABG" H 4500 3656 50  0000 C CNN
-F 2 "KiCad:RGB_LED_1205" H 4500 3200 50  0001 C CNN
+F 2 "KiCad:RGB_LED_1204_reverse" H 4500 3200 50  0001 C CNN
 F 3 "https://datasheet.lcsc.com/szlcsc/1912111437_MEIHUA-MHT150RGBCT_C409782.pdf" H 4500 3200 50  0001 C CNN
 F 4 "MHT150RGBCT" H 4500 3250 50  0001 C CNN "Part Number"
@@
 F 0 "D120" H 5100 3747 50  0000 C CNN
 F 1 "RABG" H 5100 3656 50  0000 C CNN
-F 2 "KiCad:RGB_LED_1205" H 5100 3200 50  0001 C CNN
+F 2 "KiCad:RGB_LED_1204_reverse" H 5100 3200 50  0001 C CNN
 F 3 "https://datasheet.lcsc.com/szlcsc/1912111437_MEIHUA-MHT150RGBCT_C409782.pdf" H 5100 3200 50  0001 C CNN
 F 4 "MHT150RGBCT" H 5100 3250 50  0001 C CNN "Part Number"
@@
 F 0 "D122" H 5700 3747 50  0000 C CNN
 F 1 "RABG" H 5700 3656 50  0000 C CNN
-F 2 "KiCad:RGB_LED_1205" H 5700 3200 50  0001 C CNN
+F 2 "KiCad:RGB_LED_1204_reverse" H 5700 3200 50  0001 C CNN
 F 3 "https://datasheet.lcsc.com/szlcsc/1912111437_MEIHUA-MHT150RGBCT_C409782.pdf" H 5700 3200 50  0001 C CNN
 F 4 "MHT150RGBCT" H 5700 3250 50  0001 C CNN "Part Number"
@@
 F 0 "D123" H 6300 3747 50  0000 C CNN
 F 1 "RABG" H 6300 3656 50  0000 C CNN
-F 2 "KiCad:RGB_LED_1205" H 6300 3200 50  0001 C CNN
+F 2 "KiCad:RGB_LED_1204_reverse" H 6300 3200 50  0001 C CNN
 F 3 "https://datasheet.lcsc.com/szlcsc/1912111437_MEIHUA-MHT150RGBCT_C409782.pdf" H 6300 3200 50  0001 C CNN
 F 4 "MHT150RGBCT" H 6300 3250 50  0001 C CNN "Part Number"
@@
 F 0 "D125" H 6900 3747 50  0000 C CNN
 F 1 "RABG" H 6900 3656 50  0000 C CNN
-F 2 "KiCad:RGB_LED_1205" H 6900 3200 50  0001 C CNN
+F 2 "KiCad:RGB_LED_1204_reverse" H 6900 3200 50  0001 C CNN
 F 3 "https://datasheet.lcsc.com/szlcsc/1912111437_MEIHUA-MHT150RGBCT_C409782.pdf" H 6900 3200 50  0001 C CNN
 F 4 "MHT150RGBCT" H 6900 3250 50  0001 C CNN "Part Number"
@@
 F 0 "D127" H 7500 3747 50  0000 C CNN
 F 1 "RABG" H 7500 3656 50  0000 C CNN
-F 2 "KiCad:RGB_LED_1205" H 7500 3200 50  0001 C CNN
+F 2 "KiCad:RGB_LED_1204_reverse" H 7500 3200 50  0001 C CNN
 F 3 "https://datasheet.lcsc.com/szlcsc/1912111437_MEIHUA-MHT150RGBCT_C409782.pdf" H 7500 3200 50  0001 C CNN
 F 4 "MHT150RGBCT" H 7500 3250 50  0001 C CNN "Part Number"
@@
 F 0 "D129" H 8100 3747 50  0000 C CNN
 F 1 "RABG" H 8100 3656 50  0000 C CNN
-F 2 "KiCad:RGB_LED_1205" H 8100 3200 50  0001 C CNN
+F 2 "KiCad:RGB_LED_1204_reverse" H 8100 3200 50  0001 C CNN
 F 3 "https://datasheet.lcsc.com/szlcsc/1912111437_MEIHUA-MHT150RGBCT_C409782.pdf" H 8100 3200 50  0001 C CNN
 F 4 "MHT150RGBCT" H 8100 3250 50  0001 C CNN "Part Number"
@@
 F 0 "D131" H 8700 3747 50  0000 C CNN
 F 1 "RABG" H 8700 3656 50  0000 C CNN
-F 2 "KiCad:RGB_LED_1205" H 8700 3200 50  0001 C CNN
+F 2 "KiCad:RGB_LED_1204_reverse" H 8700 3200 50  0001 C CNN
 F 3 "https://datasheet.lcsc.com/szlcsc/1912111437_MEIHUA-MHT150RGBCT_C409782.pdf" H 8700 3200 50  0001 C CNN
 F 4 "MHT150RGBCT" H 8700 3250 50  0001 C CNN "Part Number"
@@
 F 0 "D133" H 9300 3747 50  0000 C CNN
 F 1 "RABG" H 9300 3656 50  0000 C CNN
-F 2 "KiCad:RGB_LED_1205" H 9300 3200 50  0001 C CNN
+F 2 "KiCad:RGB_LED_1204_reverse" H 9300 3200 50  0001 C CNN
 F 3 "https://datasheet.lcsc.com/szlcsc/1912111437_MEIHUA-MHT150RGBCT_C409782.pdf" H 9300 3200 50  0001 C CNN
 F 4 "MHT150RGBCT" H 9300 3250 50  0001 C CNN "Part Number"
@@
 F 0 "D135" H 9900 3747 50  0000 C CNN
 F 1 "RABG" H 9900 3656 50  0000 C CNN
-F 2 "KiCad:RGB_LED_1205" H 9900 3200 50  0001 C CNN
+F 2 "KiCad:RGB_LED_1204_reverse" H 9900 3200 50  0001 C CNN
 F 3 "https://datasheet.lcsc.com/szlcsc/1912111437_MEIHUA-MHT150RGBCT_C409782.pdf" H 9900 3200 50  0001 C CNN
 F 4 "MHT150RGBCT" H 9900 3250 50  0001 C CNN "Part Number"
@@
 F 0 "D136" H 9900 4797 50  0000 C CNN
 F 1 "RABG" H 9900 4706 50  0000 C CNN
-F 2 "KiCad:RGB_LED_1205" H 9900 4250 50  0001 C CNN
+F 2 "KiCad:RGB_LED_1204_reverse" H 9900 4250 50  0001 C CNN
 F 3 "https://datasheet.lcsc.com/szlcsc/1912111437_MEIHUA-MHT150RGBCT_C409782.pdf" H 9900 4250 50  0001 C CNN
 F 4 "MHT150RGBCT" H 9900 4300 50  0001 C CNN "Part Number"
@@
 F 0 "D132" H 8700 4797 50  0000 C CNN
 F 1 "RABG" H 8700 4706 50  0000 C CNN
-F 2 "KiCad:RGB_LED_1205" H 8700 4250 50  0001 C CNN
+F 2 "KiCad:RGB_LED_1204_reverse" H 8700 4250 50  0001 C CNN
 F 3 "https://datasheet.lcsc.com/szlcsc/1912111437_MEIHUA-MHT150RGBCT_C409782.pdf" H 8700 4250 50  0001 C CNN
 F 4 "MHT150RGBCT" H 8700 4300 50  0001 C CNN "Part Number"
@@
 F 0 "D130" H 8100 4797 50  0000 C CNN
 F 1 "RABG" H 8100 4706 50  0000 C CNN
-F 2 "KiCad:RGB_LED_1205" H 8100 4250 50  0001 C CNN
+F 2 "KiCad:RGB_LED_1204_reverse" H 8100 4250 50  0001 C CNN
 F 3 "https://datasheet.lcsc.com/szlcsc/1912111437_MEIHUA-MHT150RGBCT_C409782.pdf" H 8100 4250 50  0001 C CNN
 F 4 "MHT150RGBCT" H 8100 4300 50  0001 C CNN "Part Number"
@@
 F 0 "D128" H 7500 4797 50  0000 C CNN
 F 1 "RABG" H 7500 4706 50  0000 C CNN
-F 2 "KiCad:RGB_LED_1205" H 7500 4250 50  0001 C CNN
+F 2 "KiCad:RGB_LED_1204_reverse" H 7500 4250 50  0001 C CNN
 F 3 "https://datasheet.lcsc.com/szlcsc/1912111437_MEIHUA-MHT150RGBCT_C409782.pdf" H 7500 4250 50  0001 C CNN
 F 4 "MHT150RGBCT" H 7500 4300 50  0001 C CNN "Part Number"
@@
 F 0 "D126" H 6900 4797 50  0000 C CNN
 F 1 "RABG" H 6900 4706 50  0000 C CNN
-F 2 "KiCad:RGB_LED_1205" H 6900 4250 50  0001 C CNN
+F 2 "KiCad:RGB_LED_1204_reverse" H 6900 4250 50  0001 C CNN
 F 3 "https://datasheet.lcsc.com/szlcsc/1912111437_MEIHUA-MHT150RGBCT_C409782.pdf" H 6900 4250 50  0001 C CNN
 F 4 "MHT150RGBCT" H 6900 4300 50  0001 C CNN "Part Number"
@@
 F 0 "D124" H 6300 4797 50  0000 C CNN
 F 1 "RABG" H 6300 4706 50  0000 C CNN
-F 2 "KiCad:RGB_LED_1205" H 6300 4250 50  0001 C CNN
+F 2 "KiCad:RGB_LED_1204_reverse" H 6300 4250 50  0001 C CNN
 F 3 "https://datasheet.lcsc.com/szlcsc/1912111437_MEIHUA-MHT150RGBCT_C409782.pdf" H 6300 4250 50  0001 C CNN
 F 4 "MHT150RGBCT" H 6300 4300 50  0001 C CNN "Part Number"
@@
 F 0 "D121" H 5100 4797 50  0000 C CNN
 F 1 "RABG" H 5100 4706 50  0000 C CNN
-F 2 "KiCad:RGB_LED_1205" H 5100 4250 50  0001 C CNN
+F 2 "KiCad:RGB_LED_1204_reverse" H 5100 4250 50  0001 C CNN
 F 3 "https://datasheet.lcsc.com/szlcsc/1912111437_MEIHUA-MHT150RGBCT_C409782.pdf" H 5100 4250 50  0001 C CNN
 F 4 "MHT150RGBCT" H 5100 4300 50  0001 C CNN "Part Number"
@@
 F 0 "D119" H 4500 4797 50  0000 C CNN
 F 1 "RABG" H 4500 4706 50  0000 C CNN
-F 2 "KiCad:RGB_LED_1205" H 4500 4250 50  0001 C CNN
+F 2 "KiCad:RGB_LED_1204_reverse" H 4500 4250 50  0001 C CNN
 F 3 "https://datasheet.lcsc.com/szlcsc/1912111437_MEIHUA-MHT150RGBCT_C409782.pdf" H 4500 4250 50  0001 C CNN
 F 4 "MHT150RGBCT" H 4500 4300 50  0001 C CNN "Part Number"
@@
 F 0 "D117" H 3950 4797 50  0000 C CNN
 F 1 "RABG" H 3950 4706 50  0000 C CNN
-F 2 "KiCad:RGB_LED_1205" H 3950 4250 50  0001 C CNN
+F 2 "KiCad:RGB_LED_1204_reverse" H 3950 4250 50  0001 C CNN
 F 3 "https://datasheet.lcsc.com/szlcsc/1912111437_MEIHUA-MHT150RGBCT_C409782.pdf" H 3950 4250 50  0001 C CNN
 F 4 "MHT150RGBCT" H 3950 4300 50  0001 C CNN "Part Number"
@@
 F 0 "D115" H 3350 4797 50  0000 C CNN
 F 1 "RABG" H 3350 4706 50  0000 C CNN
-F 2 "KiCad:RGB_LED_1205" H 3350 4250 50  0001 C CNN
+F 2 "KiCad:RGB_LED_1204_reverse" H 3350 4250 50  0001 C CNN
 F 3 "https://datasheet.lcsc.com/szlcsc/1912111437_MEIHUA-MHT150RGBCT_C409782.pdf" H 3350 4250 50  0001 C CNN
 F 4 "MHT150RGBCT" H 3350 4300 50  0001 C CNN "Part Number"
@@
 F 0 "D113" H 2750 4797 50  0000 C CNN
 F 1 "RABG" H 2750 4706 50  0000 C CNN
-F 2 "KiCad:RGB_LED_1205" H 2750 4250 50  0001 C CNN
+F 2 "KiCad:RGB_LED_1204_reverse" H 2750 4250 50  0001 C CNN
 F 3 "https://datasheet.lcsc.com/szlcsc/1912111437_MEIHUA-MHT150RGBCT_C409782.pdf" H 2750 4250 50  0001 C CNN
 F 4 "MHT150RGBCT" H 2750 4300 50  0001 C CNN "Part Number"
@@
 F 0 "D111" H 2150 4797 50  0000 C CNN
 F 1 "RABG" H 2150 4706 50  0000 C CNN
-F 2 "KiCad:RGB_LED_1205" H 2150 4250 50  0001 C CNN
+F 2 "KiCad:RGB_LED_1204_reverse" H 2150 4250 50  0001 C CNN
 F 3 "https://datasheet.lcsc.com/szlcsc/1912111437_MEIHUA-MHT150RGBCT_C409782.pdf" H 2150 4250 50  0001 C CNN
 F 4 "MHT150RGBCT" H 2150 4300 50  0001 C CNN "Part Number"
@@
 F 0 "D134" H 9300 4797 50  0000 C CNN
 F 1 "RABG" H 9300 4706 50  0000 C CNN
-F 2 "KiCad:RGB_LED_1205" H 9300 4250 50  0001 C CNN
+F 2 "KiCad:RGB_LED_1204_reverse" H 9300 4250 50  0001 C CNN
 F 3 "https://datasheet.lcsc.com/szlcsc/1912111437_MEIHUA-MHT150RGBCT_C409782.pdf" H 9300 4250 50  0001 C CNN
 F 4 "MHT150RGBCT" H 9300 4300 50  0001 C CNN "Part Number"

Commit message: It is the last update of 1206 RGB design, going to switch LED again, correct the 1206 name
Parts:
- D110, D111, D112, D113, D114, D115, D116, D117, D118, D119, D120, D121, D122, D123, D124, D125, D126, D127, D128, D129, D130, D131, D132, D133, D134, D135, D136: footprint KiCad:RGB_LED_1204_reverse -> KiCad:RGB_LED_1206_reverse
