File: hardware/PCB/RGBMatrix2.sch (KiCad schematic (older format))
At the start: 27 parts

Commit message: fix some detail for 1.0
Parts:
- renumbered D112 to D111, D114 to D112, D116 to D113, D118 to D114, D120 to D115, D122 to D116, D123 to D117, D125 to D118, D127 to D119, D129 to D120, D131 to D121, D133 to D122, D135 to D123, D111 to D124, D113 to D125, D115 to D126, D117 to D127, D119 to D128, D121 to D129, D124 to D130, D126 to D131, D128 to D132, D130 to D133, D132 to D134, D134 to D135
Changed lines of the file:
@@
 P 2750 3250
 AR Path="/5EC33E3D/5EC48B37/5ECF7D8D" Ref="D?"  Part="1"
-AR Path="/5EC33E3D/5E12F961/5ECF7D8D" Ref="D112"  Part="1"
-F 0 "D112" H 2750 3747 50  0000 C CNN
+AR Path="/5EC33E3D/5E12F961/5ECF7D8D" Ref="D111"  Part="1"
+F 0 "D111" H 2750 3747 50  0000 C CNN
 F 1 "RABG" H 2750 3656 50  0000 C CNN
 F 2 "KiCad:RGB_LED_1206_reverse" H 2750 3200 50  0001 C CNN
@@
 P 3350 3250
 AR Path="/5EC33E3D/5EC48B37/5ED08C1C" Ref="D?"  Part="1"
-AR Path="/5EC33E3D/5E12F961/5ED08C1C" Ref="D114"  Part="1"
-F 0 "D114" H 3350 3747 50  0000 C CNN
+AR Path="/5EC33E3D/5E12F961/5ED08C1C" Ref="D112"  Part="1"
+F 0 "D112" H 3350 3747 50  0000 C CNN
 F 1 "RABG" H 3350 3656 50  0000 C CNN
 F 2 "KiCad:RGB_LED_1206_reverse" H 3350 3200 50  0001 C CNN
@@
 P 3950 3250
 AR Path="/5EC33E3D/5EC48B37/5ED19532" Ref="D?"  Part="1"
-AR Path="/5EC33E3D/5E12F961/5ED19532" Ref="D116"  Part="1"
-F 0 "D116" H 3950 3747 50  0000 C CNN
+AR Path="/5EC33E3D/5E12F961/5ED19532" Ref="D113"  Part="1"
+F 0 "D113" H 3950 3747 50  0000 C CNN
 F 1 "RABG" H 3950 3656 50  0000 C CNN
 F 2 "KiCad:RGB_LED_1206_reverse" H 3950 3200 50  0001 C CNN
@@
 P 4500 3250
 AR Path="/5EC33E3D/5EC48B37/5ED2A1D2" Ref="D?"  Part="1"
-AR Path="/5EC33E3D/5E12F961/5ED2A1D2" Ref="D118"  Part="1"
-F 0 "D118" H 4500 3747 50  0000 C CNN
+AR Path="/5EC33E3D/5E12F961/5ED2A1D2" Ref="D114"  Part="1"
+F 0 "D114" H 4500 3747 50  0000 C CNN
 F 1 "RABG" H 4500 3656 50  0000 C CNN
 F 2 "KiCad:RGB_LED_1206_reverse" H 4500 3200 50  0001 C CNN
@@
 P 5100 3250
 AR Path="/5EC33E3D/5EC48B37/5ED3AE35" Ref="D?"  Part="1"
-AR Path="/5EC33E3D/5E12F961/5ED3AE35" Ref="D120"  Part="1"
-F 0 "D120" H 5100 3747 50  0000 C CNN
+AR Path="/5EC33E3D/5E12F961/5ED3AE35" Ref="D115"  Part="1"
+F 0 "D115" H 5100 3747 50  0000 C CNN
 F 1 "RABG" H 5100 3656 50  0000 C CNN
 F 2 "KiCad:RGB_LED_1206_reverse" H 5100 3200 50  0001 C CNN
@@
 P 5700 3250
 AR Path="/5EC33E3D/5EC48B37/5ED4B8F9" Ref="D?"  Part="1"
-AR Path="/5EC33E3D/5E12F961/5ED4B8F9" Ref="D122"  Part="1"
-F 0 "D122" H 5700 3747 50  0000 C CNN
+AR Path="/5EC33E3D/5E12F961/5ED4B8F9" Ref="D116"  Part="1"
+F 0 "D116" H 5700 3747 50  0000 C CNN
 F 1 "RABG" H 5700 3656 50  0000 C CNN
 F 2 "KiCad:RGB_LED_1206_reverse" H 5700 3200 50  0001 C CNN
@@
 P 6300 3250
 AR Path="/5EC33E3D/5EC48B37/5ED5C37B" Ref="D?"  Part="1"
-AR Path="/5EC33E3D/5E12F961/5ED5C37B" Ref="D123"  Part="1"
-F 0 "D123" H 6300 3747 50  0000 C CNN
+AR Path="/5EC33E3D/5E12F961/5ED5C37B" Ref="D117"  Part="1"
+F 0 "D117" H 6300 3747 50  0000 C CNN
 F 1 "RABG" H 6300 3656 50  0000 C CNN
 F 2 "KiCad:RGB_LED_1206_reverse" H 6300 3200 50  0001 C CNN
@@
 P 6900 3250
 AR Path="/5EC33E3D/5EC48B37/5ED6CA4B" Ref="D?"  Part="1"
-AR Path="/5EC33E3D/5E12F961/5ED6CA4B" Ref="D125"  Part="1"
-F 0 "D125" H 6900 3747 50  0000 C CNN
+AR Path="/5EC33E3D/5E12F961/5ED6CA4B" Ref="D118"  Part="1"
+F 0 "D118" H 6900 3747 50  0000 C CNN
 F 1 "RABG" H 6900 3656 50  0000 C CNN
 F 2 "KiCad:RGB_LED_1206_reverse" H 6900 3200 50  0001 C CNN
@@
 P 7500 3250
 AR Path="/5EC33E3D/5EC48B37/5ED7D671" Ref="D?"  Part="1"
-AR Path="/5EC33E3D/5E12F961/5ED7D671" Ref="D127"  Part="1"
-F 0 "D127" H 7500 3747 50  0000 C CNN
+AR Path="/5EC33E3D/5E12F961/5ED7D671" Ref="D119"  Part="1"
+F 0 "D119" H 7500 3747 50  0000 C CNN
 F 1 "RABG" H 7500 3656 50  0000 C CNN
 F 2 "KiCad:RGB_LED_1206_reverse" H 7500 3200 50  0001 C CNN
@@
 P 8100 3250
 AR Path="/5EC33E3D/5EC48B37/5ED8E3BC" Ref="D?"  Part="1"
-AR Path="/5EC33E3D/5E12F961/5ED8E3BC" Ref="D129"  Part="1"
-F 0 "D129" H 8100 3747 50  0000 C CNN
+AR Path="/5EC33E3D/5E12F961/5ED8E3BC" Ref="D120"  Part="1"
+F 0 "D120" H 8100 3747 50  0000 C CNN
 F 1 "RABG" H 8100 3656 50  0000 C CNN
 F 2 "KiCad:RGB_LED_1206_reverse" H 8100 3200 50  0001 C CNN
@@
 P 8700 3250
 AR Path="/5EC33E3D/5EC48B37/5ED9EECC" Ref="D?"  Part="1"
-AR Path="/5EC33E3D/5E12F961/5ED9EECC" Ref="D131"  Part="1"
-F 0 "D131" H 8700 3747 50  0000 C CNN
+AR Path="/5EC33E3D/5E12F961/5ED9EECC" Ref="D121"  Part="1"
+F 0 "D121" H 8700 3747 50  0000 C CNN
 F 1 "RABG" H 8700 3656 50  0000 C CNN
 F 2 "KiCad:RGB_LED_1206_reverse" H 8700 3200 50  0001 C CNN
@@
 P 9300 3250
 AR Path="/5EC33E3D/5EC48B37/5EDAF8D0" Ref="D?"  Part="1"
-AR Path="/5EC33E3D/5E12F961/5EDAF8D0" Ref="D133"  Part="1"
-F 0 "D133" H 9300 3747 50  0000 C CNN
+AR Path="/5EC33E3D/5E12F961/5EDAF8D0" Ref="D122"  Part="1"
+F 0 "D122" H 9300 3747 50  0000 C CNN
 F 1 "RABG" H 9300 3656 50  0000 C CNN
 F 2 "KiCad:RGB_LED_1206_reverse" H 9300 3200 50  0001 C CNN
@@
 P 9900 3250
 AR Path="/5EC33E3D/5EC48B37/5EDC0468" Ref="D?"  Part="1"
-AR Path="/5EC33E3D/5E12F961/5EDC0468" Ref="D135"  Part="1"
-F 0 "D135" H 9900 3747 50  0000 C CNN
+AR Path="/5EC33E3D/5E12F961/5EDC0468" Ref="D123"  Part="1"
+F 0 "D123" H 9900 3747 50  0000 C CNN
 F 1 "RABG" H 9900 3656 50  0000 C CNN
 F 2 "KiCad:RGB_LED_1206_reverse" H 9900 3200 50  0001 C CNN
@@
 P 8700 4300
 AR Path="/5EC33E3D/5EC48B37/5EE13AA6" Ref="D?"  Part="1"
-AR Path="/5EC33E3D/5E12F961/5EE13AA6" Ref="D132"  Part="1"
-F 0 "D132" H 8700 4797 50  0000 C CNN
+AR Path="/5EC33E3D/5E12F961/5EE13AA6" Ref="D134"  Part="1"
+F 0 "D134" H 8700 4797 50  0000 C CNN
 F 1 "RABG" H 8700 4706 50  0000 C CNN
 F 2 "KiCad:RGB_LED_1206_reverse" H 8700 4250 50  0001 C CNN
@@
 P 8100 4300
 AR Path="/5EC33E3D/5EC48B37/5EE24547" Ref="D?"  Part="1"
-AR Path="/5EC33E3D/5E12F961/5EE24547" Ref="D130"  Part="1"
-F 0 "D130" H 8100 4797 50  0000 C CNN
+AR Path="/5EC33E3D/5E12F961/5EE24547" Ref="D133"  Part="1"
+F 0 "D133" H 8100 4797 50  0000 C CNN
 F 1 "RABG" H 8100 4706 50  0000 C CNN
 F 2 "KiCad:RGB_LED_1206_reverse" H 8100 4250 50  0001 C CNN
@@
 P 7500 4300
 AR Path="/5EC33E3D/5EC48B37/5EE34C17" Ref="D?"  Part="1"
-AR Path="/5EC33E3D/5E12F961/5EE34C17" Ref="D128"  Part="1"
-F 0 "D128" H 7500 4797 50  0000 C CNN
+AR Path="/5EC33E3D/5E12F961/5EE34C17" Ref="D132"  Part="1"
+F 0 "D132" H 7500 4797 50  0000 C CNN
 F 1 "RABG" H 7500 4706 50  0000 C CNN
 F 2 "KiCad:RGB_LED_1206_reverse" H 7500 4250 50  0001 C CNN
@@
 P 6900 4300
 AR Path="/5EC33E3D/5EC48B37/5EE45875" Ref="D?"  Part="1"
-AR Path="/5EC33E3D/5E12F961/5EE45875" Ref="D126"  Part="1"
-F 0 "D126" H 6900 4797 50  0000 C CNN
+AR Path="/5EC33E3D/5E12F961/5EE45875" Ref="D131"  Part="1"
+F 0 "D131" H 6900 4797 50  0000 C CNN
 F 1 "RABG" H 6900 4706 50  0000 C CNN
 F 2 "KiCad:RGB_LED_1206_reverse" H 6900 4250 50  0001 C CNN
@@
 P 6300 4300
 AR Path="/5EC33E3D/5EC48B37/5EE56B5B" Ref="D?"  Part="1"
-AR Path="/5EC33E3D/5E12F961/5EE56B5B" Ref="D124"  Part="1"
-F 0 "D124" H 6300 4797 50  0000 C CNN
+AR Path="/5EC33E3D/5E12F961/5EE56B5B" Ref="D130"  Part="1"
+F 0 "D130" H 6300 4797 50  0000 C CNN
 F 1 "RABG" H 6300 4706 50  0000 C CNN
 F 2 "KiCad:RGB_LED_1206_reverse" H 6300 4250 50  0001 C CNN
@@
 P 5100 4300
 AR Path="/5EC33E3D/5EC48B37/5EE68DA5" Ref="D?"  Part="1"
-AR Path="/5EC33E3D/5E12F961/5EE68DA5" Ref="D121"  Part="1"
-F 0 "D121" H 5100 4797 50  0000 C CNN
+AR Path="/5EC33E3D/5E12F961/5EE68DA5" Ref="D129"  Part="1"
+F 0 "D129" H 5100 4797 50  0000 C CNN
 F 1 "RABG" H 5100 4706 50  0000 C CNN
 F 2 "KiCad:RGB_LED_1206_reverse" H 5100 4250 50  0001 C CNN
@@
 P 4500 4300
 AR Path="/5EC33E3D/5EC48B37/5EE797FA" Ref="D?"  Part="1"
-AR Path="/5EC33E3D/5E12F961/5EE797FA" Ref="D119"  Part="1"
-F 0 "D119" H 4500 4797 50  0000 C CNN
+AR Path="/5EC33E3D/5E12F961/5EE797FA" Ref="D128"  Part="1"
+F 0 "D128" H 4500 4797 50  0000 C CNN
 F 1 "RABG" H 4500 4706 50  0000 C CNN
 F 2 "KiCad:RGB_LED_1206_reverse" H 4500 4250 50  0001 C CNN
@@
 P 3950 4300
 AR Path="/5EC33E3D/5EC48B37/5EE8A2F6" Ref="D?"  Part="1"
-AR Path="/5EC33E3D/5E12F961/5EE8A2F6" Ref="D117"  Part="1"
-F 0 "D117" H 3950 4797 50  0000 C CNN
+AR Path="/5EC33E3D/5E12F961/5EE8A2F6" Ref="D127"  Part="1"
+F 0 "D127" H 3950 4797 50  0000 C CNN
 F 1 "RABG" H 3950 4706 50  0000 C CNN
 F 2 "KiCad:RGB_LED_1206_reverse" H 3950 4250 50  0001 C CNN
@@
 P 3350 4300
 AR Path="/5EC33E3D/5EC48B37/5EEAC0EB" Ref="D?"  Part="1"
-AR Path="/5EC33E3D/5E12F961/5EEAC0EB" Ref="D115"  Part="1"
-F 0 "D115" H 3350 4797 50  0000 C CNN
+AR Path="/5EC33E3D/5E12F961/5EEAC0EB" Ref="D126"  Part="1"
+F 0 "D126" H 3350 4797 50  0000 C CNN
 F 1 "RABG" H 3350 4706 50  0000 C CNN
 F 2 "KiCad:RGB_LED_1206_reverse" H 3350 4250 50  0001 C CNN
@@
 P 2750 4300
 AR Path="/5EC33E3D/5EC48B37/5EEBC7BB" Ref="D?"  Part="1"
-AR Path="/5EC33E3D/5E12F961/5EEBC7BB" Ref="D113"  Part="1"
-F 0 "D113" H 2750 4797 50  0000 C CNN
+AR Path="/5EC33E3D/5E12F961/5EEBC7BB" Ref="D125"  Part="1"
+F 0 "D125" H 2750 4797 50  0000 C CNN
 F 1 "RABG" H 2750 4706 50  0000 C CNN
 F 2 "KiCad:RGB_LED_1206_reverse" H 2750 4250 50  0001 C CNN
@@
 P 2150 4300
 AR Path="/5EC33E3D/5EC48B37/5EECD5B2" Ref="D?"  Part="1"
-AR Path="/5EC33E3D/5E12F961/5EECD5B2" Ref="D111"  Part="1"
-F 0 "D111" H 2150 4797 50  0000 C CNN
+AR Path="/5EC33E3D/5E12F961/5EECD5B2" Ref="D124"  Part="1"
+F 0 "D124" H 2150 4797 50  0000 C CNN
 F 1 "RABG" H 2150 4706 50  0000 C CNN
 F 2 "KiCad:RGB_LED_1206_reverse" H 2150 4250 50  0001 C CNN
@@
 P 9300 4300
 AR Path="/5EC33E3D/5EC48B37/5EE030A2" Ref="D?"  Part="1"
-AR Path="/5EC33E3D/5E12F961/5EE030A2" Ref="D134"  Part="1"
-F 0 "D134" H 9300 4797 50  0000 C CNN
+AR Path="/5EC33E3D/5E12F961/5EE030A2" Ref="D135"  Part="1"
+F 0 "D135" H 9300 4797 50  0000 C CNN
 F 1 "RABG" H 9300 4706 50  0000 C CNN
 F 2 "KiCad:RGB_LED_1206_reverse" H 9300 4250 50  0001 C CNN
