File: hardware/PCB/PCB.kicad_pcb (KiCad board)
At the start: 2 copper layers, 282.7 x 117.3 mm, 254 parts, among them J1 473460001, SW1 B3U-1000P, SW2 B3U-1000P, U1 IS31FL3733-QFLS4-TR, U2 IS31FL3733-QFLS4-TR, U3 AZ1117CH-3.3TRG1, U4 STM32F303CCT6, Y1 8Mhz20pF

Commit message: attempt to remove some extra values
Routing:
- net GND: vias 17 -> 16
Changed lines of the file:
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@@
     (thickness 1.6)
     (drawings 300)
-    (tracks 3154)
+    (tracks 3153)
     (zones 0)
     (modules 254)
@@
     (tags capacitor)
     (attr smd)
-    (fp_text reference C19 (at 0 -1.17 90) (layer F.SilkS)
+    (fp_text reference C19 (at 0 1.15 90) (layer F.SilkS)
       (effects (font (size 1 1) (thickness 0.15)))
     )
@@
   (segment (start 234.8166 185.68033) (end 234.28627 185.15) (width 0.25) (layer F.Cu) (net 1))
   (via (at 96.425 134.7) (size 0.6) (drill 0.3) (layers F.Cu B.Cu) (net 1))
-  (via (at 114.548 85.302) (size 0.8) (drill 0.4) (layers F.Cu B.Cu) (net 1))
   (via (at 121.025 88.95) (size 0.6) (drill 0.3) (layers F.Cu B.Cu) (net 1))
   (via (at 122.025 88.95) (size 0.6) (drill 0.3) (layers F.Cu B.Cu) (net 1))

Commit message: update render, remove useless files, fix the decoupeling
Parts:
- removed the R11 at (141.4, 91.6)
- removed the R16 at (126.4, 91.0)
- added C24: 10nF, Capacitor_SMD:C_0402_1005Metric, F.Cu at (139.6, 90.8)
- added C25: 1uf, Capacitor_SMD:C_0402_1005Metric, F.Cu at (140.6, 90.8)
- added R10: 1K, Resistor_SMD:R_0402_1005Metric, F.Cu at (142.8, 93.0)
- added R13: 10K, Resistor_SMD:R_0402_1005Metric, F.Cu at (126.4, 91.0)
- C23: renamed from C21; value 100nF -> 4.7uf
- Key1, Key10, Key11, Key12, Key13, Key14, Key15, Key16, Key17, Key18, Key19, Key2, Key20, Key21, Key22, Key23, Key24, Key25, Key26, Key27, Key28, Key29, Key3, Key30, Key31, Key32, Key33, Key34, Key35, Key36, Key37, Key38, Key39, Key4, Key40, Key41, Key42, Key43, Key44, Key45, Key46, Key47, Key48, Key49, Key5, Key50, Key51, Key52, Key53, Key54, Key55, Key56, Key57, Key58, Key59, Key6, Key60, Key61, Key62, Key63, Key64, Key65, Key66, Key67, Key68, Key7, Key8, Key9: value CPG151101S03 -> Switch
- moved C19 14.6 mm to (126.5, 95.5), turned to 90 degrees
- renumbered C22 to C17, C23 to C18, C17 to C19, C18 to C20, C19 to C21, C20 to C22, C24 to C26, D127 to D100, D128 to D101, D129 to D102, D130 to D103, D131 to D104, D132 to D105, D133 to D106, D134 to D107, D135 to D108, D136 to D109, D69 to D110, D70 to D111, D71 to D112, D72 to D113, D73 to D114, D74 to D115, D75 to D116, D76 to D117, D77 to D118, D78 to D119, D79 to D120, D80 to D121, D81 to D122, D82 to D123, D83 to D124, D84 to D125, D85 to D126, D86 to D127, D87 to D128, D88 to D129, D89 to D130, D90 to D131, D91 to D132, D92 to D133, D93 to D134, D94 to D135, D95 to D136, D96 to D69, D97 to D70, D98 to D71, D99 to D72, D100 to D73, D101 to D74, D102 to D75, D103 to D76, D104 to D77, D105 to D78, D106 to D79, D107 to D80, D108 to D81, D109 to D82, D110 to D83, D111 to D84, D112 to D85, D113 to D86, D114 to D87, D115 to D88, D116 to D89, D117 to D90, D118 to D91, D119 to D92, D120 to D93, D121 to D94, D122 to D95, D123 to D96, D124 to D97, D125 to D98, D126 to D99, R10 to R11, R13 to R12, R12 to R14, R14 to R16
Connections:
- net Net-(C22-Pad2) renamed /SMT32/OSC_IN
- U4 pad 6: Net-(R11-Pad1) -> /SMT32/OSC_OUT
Routing:
- net /SMT32/OSC_OUT: track 0.00 -> 5.85 mm
- net Net-(R11-Pad1): track 4.46 -> 0.00 mm
- net GND: vias 16 -> 28

Commit message: minor changes
Parts:
- moved C22 1.57 mm to (139.5, 95.3)
- moved C17 0.87 mm to (142.0, 95.6), turned to 45 degrees
- moved C20 0.73 mm to (137.4, 97.0), turned to 0 degrees
- moved R10 0.50 mm to (142.3, 93.0), turned to 0 degrees
- moved C19 0.10 mm to (126.3, 95.5)
- moved C23 0.10 mm to (127.3, 95.5)
Routing:
- net +3V3: track 401.5 -> 388.3 mm
- net /SMT32/COL1: track 119.2 -> 117.8 mm
- net /SMT32/OSC_OUT: track 5.85 -> 4.67 mm
- net Net-(C18-Pad2): track 3.48 -> 4.00 mm

Commit message: Move the Crystal and made a keepout ring
Parts:
- moved C26 9.82 mm to (141.6, 90.8), turned to 270 degrees
- moved SW1 6.28 mm to (144.6, 90.8)
- moved C18 5.60 mm to (147.1, 94.8), turned to 180 degrees
- moved Y1 3.72 mm to (144.6, 97.2), turned to 0 degrees
- moved R10 3.08 mm to (145.2, 94.3), turned to 270 degrees
- moved C17 1.19 mm to (142.4, 94.5), turned to 0 degrees
- moved C22 0.78 mm to (138.9, 95.9), turned to 270 degrees
Routing:
- net GND: track 24.0 -> 63.8 mm, vias 28 -> 42
- net Net-(C26-Pad2): track 17.0 -> 10.5 mm, vias 2 -> 0
- net /SMT32/OSC_OUT: track 4.67 -> 8.29 mm
- net +3V3: track 388.3 -> 390.4 mm
- net /SMT32/COL4: track 126.0 -> 127.6 mm
- net /SMT32/COL6: track 164.9 -> 166.5 mm
- net /SMT32/COL5: track 145.5 -> 147.0 mm
- net /SMT32/COL7: track 184.5 -> 186.0 mm
- net /SMT32/COL14: track 327.3 -> 328.3 mm
- net /SMT32/COL13: track 307.1 -> 308.1 mm
- net /SMT32/COL12: track 287.2 -> 288.2 mm
- net /SMT32/COL8: track 186.3 -> 187.4 mm
- net /SMT32/COL10: track 249.8 -> 250.8 mm
- net /SMT32/COL11: track 266.9 -> 268.0 mm
- net /SMT32/COL9: track 228.4 -> 229.5 mm

Commit message: small improvements (cap distance)
Parts:
- moved C4 6.72 mm to (101.3, 146.9)
- moved C5 6.72 mm to (102.3, 146.9)
- moved C2 1.77 mm to (96.4, 134.7), turned to 45 degrees
- moved C1 1.10 mm to (97.8, 136.1), turned to 225 degrees
- moved C11 0.94 mm to (234.0, 179.4), turned to 90 degrees
- moved R2 0.73 mm to (94.8, 133.7)
- moved R3 0.73 mm to (93.8, 133.7)
- moved C3 0.46 mm to (97.1, 135.4), turned to 45 degrees
- moved C10 0.19 mm to (235.0, 179.4), turned to 90 degrees
Routing:
- net /RGB/RGBmatrix2/COL8: track 61.7 -> 40.9 mm
- net /RGB/RGBmatrix2/ROW4: track 285.1 -> 279.3 mm
- net /RGB/RGBmatrix2/ROW6: track 287.3 -> 282.5 mm
- net +3V3: track 390.4 -> 386.3 mm
- net /SMT32/ROW4: track 387.3 -> 383.8 mm
- net /RGB/RGBmatrix2/COL7: track 26.7 -> 29.2 mm
- net /RGB/RGBmatrix2/ROW5: track 275.4 -> 273.2 mm
- net /RGB/RGBmatrix2/COL9: track 61.1 -> 59.8 mm
- net /RGB/RGBmatrix/ROW6: track 307.6 -> 306.4 mm
- net /RGB/RGBmatrix2/COL4: track 96.4 -> 95.3 mm
- net /RGB/RGBmatrix2/COL10: track 79.4 -> 78.5 mm
- net /SMT32/I2C2_SDA: track 271.0 -> 271.9 mm
- net /RGB/RGBmatrix2/COL12: track 116.3 -> 115.5 mm
- net /SMT32/I2C2_SCL: track 275.2 -> 275.9 mm
- net /RGB/RGBmatrix2/COL6: track 64.3 -> 63.7 mm
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
Commit message: vias, don't know why but people put them.... so i put them there just in case
Routing:
- net GND: track 63.7 -> 58.9 mm, vias 33 -> 182
- net /SMT32/COL14: track 328.3 -> 323.8 mm
- net /RGB/SYNC: track 206.6 -> 202.6 mm
- net /SMT32/I2C2_SDA: track 271.9 -> 268.0 mm
- net /SMT32/I2C2_SCL: track 275.9 -> 272.0 mm
- net /RGB/LED_EN_PIN: track 290.4 -> 286.5 mm
