File: hardware/PCB/PCB.kicad_pcb (KiCad board)
At the start: 2 copper layers, 282.7 x 117.3 mm, 252 parts, among them J1 473460001, J2 1.27mm STDC14, SW1 B3U-1000P, U1 IS31FL3733-QFLS4-TR, U2 IS31FL3733-QFLS4-TR, U3 AZ1117CH-3.3TRG1, U4 STM32F303CCT6, Y1 8Mhz 20pf

Commit message: I have fish memory
Parts:
- D100, D101, D102, D103, D104, D105, D106, D107, D108, D109, D110, D111, D112, D113, D114, D115, D116, D117, D118, D119, D120, D121, D122, D123, D124, D125, D126, D127, D128, D129, D130, D131, D132, D133, D134, D135, D136, D69, D70, D71, D72, D73, D74, D75, D76, D77, D78, D79, D80, D81, D82, D83, D84, D85, D86, D87, D88, D89, D90, D91, D92, D93, D94, D95, D96, D97, D98, D99: value XZMDKCBDDG45S-9 -> RABG

Commit message: I don't know why but i can't count
Other:
- board text added: "NHW68 Rev:0.3 MIT License Copyright (c) 2019 Yifei Ding https://github.com/dingyifei/NHW68/"
- board text removed: "NHW68 Rev:0.2 MIT License Copyright (c) 2019 Yifei Ding https://github.com/dingyifei/NHW68/"
Changed lines of the file:
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@@
     )
   )
-  (gr_text "NHW68\nRev:0.2\nMIT License\nCopyright (c) 2019 Yifei Ding\nhttps://github.com/dingyifei/NHW68/" (at 357.04 93.28) (layer F.SilkS)
+  (gr_text "NHW68\nRev:0.3\nMIT License\nCopyright (c) 2019 Yifei Ding\nhttps://github.com/dingyifei/NHW68/" (at 357.04 93.28) (layer F.SilkS)
     (effects (font (size 1.5 1.5) (thickness 0.2)) (justify right))
   )
@@
     (effects (font (size 1.5 1.5) (thickness 0.2)))
   )
-  (gr_text "NHW68\nRev:0.2\nMIT License\nCopyright (c) 2019 Yifei Ding\nhttps://github.com/dingyifei/NHW68/" (at 357.08 93.27) (layer B.SilkS)
+  (gr_text "NHW68\nRev:0.3\nMIT License\nCopyright (c) 2019 Yifei Ding\nhttps://github.com/dingyifei/NHW68/" (at 357.08 93.27) (layer B.SilkS)
     (effects (font (size 1.5 1.5) (thickness 0.2)) (justify left mirror))
   )

Commit message: changed something
Parts:
- C21: value 22uf -> 10uf
- U3: value AZ1117CH-3.3TRG1 -> LD1117AG-33-AB3-A-R; footprint Package_TO_SOT_SMD:SOT-223-3_TabPin2 -> Package_TO_SOT_SMD:SOT-89-3
- moved C21 7.12 mm to (110.9, 89.7), turned to 0 degrees
- moved U3 0.82 mm to (110.4, 92.8)
- moved C16 0.48 mm to (109.3, 88.7)
Routing:
- net GND: vias 304 -> 305

Commit message: changed to 0603
Parts:
- removed R17, R18: 0, Resistor_SMD:R_0402_1005Metric
- C1, C10, C11, C12, C13, C14, C15, C16, C17, C18, C19, C2, C20, C21, C22, C23, C24, C25, C26, C3, C4, C5, C6, C7, C8, C9: footprint Capacitor_SMD:C_0402_1005Metric -> Capacitor_SMD:C_0603_1608Metric
- R1, R10, R11, R12, R13, R14, R15, R16, R4, R7, R8, R9: footprint Resistor_SMD:R_0402_1005Metric -> Resistor_SMD:R_0603_1608Metric
- moved R4 10.6 mm to (97.4, 126.1), turned to 180 degrees
- moved R11 9.20 mm to (145.3, 98.5)
- moved R12 8.88 mm to (117.7, 92.6), turned to 315 degrees
- moved R14 7.85 mm to (118.8, 91.5), turned to 315 degrees
- moved R9 7.84 mm to (113.9, 90.9)
- moved R1 7.62 mm to (96.2, 147.1), turned to 270 degrees
- moved C14 6.52 mm to (226.2, 187.4), turned to 45 degrees
- moved C12 5.63 mm to (224.9, 185.5), turned to 90 degrees
- moved C8 4.67 mm to (225.8, 178.7), turned to 180 degrees
- moved C23 3.94 mm to (123.6, 96.9), turned to 270 degrees
- moved C25 3.65 mm to (145.5, 89.6)
- moved C17 3.56 mm to (142.8, 95.5), turned to 180 degrees
- moved R8 3.39 mm to (233.3, 189.2), turned to 45 degrees
- moved R7 3.10 mm to (225.6, 181.7), turned to 180 degrees
- moved C11 2.50 mm to (231.7, 178.3)
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Connections:
- net Net-(R12-Pad2) renamed /SMT32/D+
- net Net-(R14-Pad2) renamed /SMT32/D-
- R13 pad 2: Net-(R13-Pad2) -> /SMT32/I2C2_SDA
- R15 pad 2: Net-(R15-Pad2) -> /SMT32/I2C2_SCL
- U4 pad 30: Net-(R15-Pad2) -> /SMT32/I2C2_SCL
- U4 pad 31: Net-(R13-Pad2) -> /SMT32/I2C2_SDA
Routing:
- net /SMT32/I2C2_SDA: track 261.0 -> 281.4 mm, vias 2 -> 4
- net /SMT32/I2C2_SCL: track 263.2 -> 283.1 mm, vias 2 -> 4
- net Net-(R13-Pad2): track 19.4 -> 0.00 mm, vias 2 -> 0
- net Net-(R15-Pad2): track 18.7 -> 0.00 mm, vias 2 -> 0
- net Net-(R4-Pad1): track 1.22 -> 15.5 mm, vias 0 -> 2
- net /SMT32/BOOT0: track 3.38 -> 12.7 mm
- net /SMT32/D+: track 2.11 -> 11.0 mm
- net /SMT32/USB_D-: track 13.3 -> 4.52 mm
- net /SMT32/USB_D+: track 15.3 -> 6.72 mm
- net +5V: track 12.4 -> 20.9 mm
- net /SMT32/D-: track 2.13 -> 10.5 mm
- net Net-(R1-Pad1): track 1.24 -> 8.80 mm, vias 0 -> 2
- net /RGB/RGBmatrix/COL13: track 90.0 -> 85.9 mm
- net /SMT32/OSC_IN: track 9.61 -> 7.05 mm
- net Net-(R8-Pad1): track 1.29 -> 3.78 mm
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
Commit message: Rev 0.5
1. Use a better 1205 LED (much chaper on LCSC)
2. Fix the crystal CL, Rext
3. did a better job on wiring (but might come with power issues?)
4. fix the key position (0.01mm shifted so its a big fix)
5. generate better bom files
6. add in LCSC and part number so easier to source
0.4 is gone
Parts:
- C21: value 10uf -> 22uf
- D100, D101, D102, D103, D104, D105, D106, D107, D108, D109, D110, D111, D112, D113, D114, D115, D116, D117, D118, D119, D120, D121, D122, D123, D124, D125, D126, D127, D128, D129, D130, D131, D132, D133, D134, D135, D136, D69, D70, D71, D72, D73, D74, D75, D76, D77, D78, D79, D80, D81, D82, D83, D84, D85, D86, D87, D88, D89, D90, D91, D92, D93, D94, D95, D96, D97, D98, D99: footprint KiCad:XZMDKCBDDG45S9_fixed -> KiCad:RGB_LED_1205
- J1: value 473460001 -> 47346-0001
- R10: value 1K -> 1.5K
- R4, R7: value 20k -> 22k
- U3: value LD1117AG-33-AB3-A-R -> AZ1117CH-3.3TRG1; footprint Package_TO_SOT_SMD:SOT-89-3 -> Package_TO_SOT_SMD:SOT-223-3_TabPin2
- moved R4 9.71 mm to (100.6, 135.3), turned to 90 degrees
- moved R1 9.28 mm to (93.9, 138.1), turned to 90 degrees
- moved U3 7.78 mm to (102.0, 90.6), turned to 180 degrees
- moved C5 7.19 mm to (106.6, 143.7), turned to 270 degrees
- moved C4 5.09 mm to (105.1, 143.7), turned to 270 degrees
- moved C17 3.12 mm to (139.8, 94.8), turned to 0 degrees
- moved C7 3.05 mm to (102.9, 134.2), turned to 0 degrees
- moved C21 2.39 mm to (107.9, 90.7)
- moved R9 2.38 mm to (114.2, 93.3)
- moved C9 2.12 mm to (227.4, 178.8), turned to 225 degrees
- moved C6 1.43 mm to (102.9, 135.7), turned to 0 degrees
- moved C8 1.07 mm to (226.3, 177.8), turned to 225 degrees
- moved R12 1.06 mm to (116.7, 92.7)
- moved R14 1.06 mm to (117.7, 91.6)
- moved R16 1.00 mm to (120.9, 97.9)
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Connections:
- U1 pad 11: /RGB/RGBmatrix/ROW3 -> /RGB/RGBmatrix/ROW1
- U1 pad 13: /RGB/RGBmatrix/ROW7 -> /RGB/RGBmatrix/ROW9
- U1 pad 15: /RGB/RGBmatrix/ROW9 -> /RGB/RGBmatrix/ROW7
- U1 pad 19: /RGB/RGBmatrix/COL4 -> /RGB/RGBmatrix/COL13
- U1 pad 21: /RGB/RGBmatrix/COL5 -> /RGB/RGBmatrix/COL4
- U1 pad 22: /RGB/RGBmatrix/COL6 -> /RGB/RGBmatrix/COL5
- U1 pad 23: /RGB/RGBmatrix/COL7 -> /RGB/RGBmatrix/COL6
- U1 pad 24: /RGB/RGBmatrix/COL8 -> /RGB/RGBmatrix/COL7
- U1 pad 25: /RGB/RGBmatrix/COL9 -> /RGB/RGBmatrix/COL8
- U1 pad 26: /RGB/RGBmatrix/COL10 -> /RGB/RGBmatrix/COL9
- U1 pad 27: /RGB/RGBmatrix/COL11 -> /RGB/RGBmatrix/COL10
- U1 pad 28: /RGB/RGBmatrix/COL12 -> /RGB/RGBmatrix/COL11
- U1 pad 30: /RGB/RGBmatrix/COL13 -> /RGB/RGBmatrix/COL12
- U1 pad 6: /RGB/RGBmatrix/ROW4 -> /RGB/RGBmatrix/ROW6
- U1 pad 8: /RGB/RGBmatrix/ROW6 -> /RGB/RGBmatrix/ROW4
- U1 pad 9: /RGB/RGBmatrix/ROW1 -> /RGB/RGBmatrix/ROW3
- U2 pad 11: /RGB/RGBmatrix2/ROW6 -> /RGB/RGBmatrix2/ROW4
- U2 pad 16: /RGB/RGBmatrix2/COL1 -> /RGB/RGBmatrix2/COL6
- U2 pad 17: /RGB/RGBmatrix2/COL2 -> /RGB/RGBmatrix2/COL5
- U2 pad 18: /RGB/RGBmatrix2/COL3 -> /RGB/RGBmatrix2/COL4
- U2 pad 19: /RGB/RGBmatrix2/COL4 -> /RGB/RGBmatrix2/COL3
- U2 pad 21: /RGB/RGBmatrix2/COL5 -> /RGB/RGBmatrix2/COL2
- U2 pad 22: /RGB/RGBmatrix2/COL6 -> /RGB/RGBmatrix2/COL1
- U2 pad 9: /RGB/RGBmatrix2/ROW4 -> /RGB/RGBmatrix2/ROW6
Routing:
- net /SMT32/ROW4: track 394.9 -> 350.5 mm
- net /SMT32/ROW3: track 373.3 -> 331.0 mm
- net /SMT32/ROW1: track 333.9 -> 293.9 mm
- net /SMT32/ROW2: track 345.8 -> 314.2 mm
- net /SMT32/ROW5: track 403.2 -> 379.0 mm
- net /RGB/RGBmatrix/ROW3: track 332.2 -> 308.5 mm, vias 0 -> 28
- net GND: track 49.4 -> 26.8 mm, vias 47 -> 31
- net /RGB/RGBmatrix/ROW6: track 305.2 -> 288.4 mm, vias 0 -> 28
- net /RGB/RGBmatrix/COL13: track 85.9 -> 72.1 mm, vias 4 -> 5
- net Net-(R4-Pad1): track 15.5 -> 2.24 mm, vias 2 -> 0
- net /RGB/RGBmatrix2/ROW3: track 297.4 -> 284.5 mm, vias 2 -> 30
- net /RGB/RGBmatrix/COL3: track 267.2 -> 279.5 mm, vias 4 -> 6
- net /RGB/RGBmatrix2/ROW6: track 282.7 -> 270.8 mm, vias 2 -> 24
- net /RGB/RGBmatrix/ROW9: track 273.5 -> 261.8 mm, vias 0 -> 26
- net /RGB/RGBmatrix/COL1: track 308.4 -> 319.2 mm, vias 3 -> 5
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Other:
- board text added: "NHW68 Rev:0.5 MIT License Copyright (c) 2019 Yifei Ding https://github.com/dingyifei/NHW68/"
- board text removed: "NHW68 Rev:0.3 MIT License Copyright (c) 2019 Yifei Ding https://github.com/dingyifei/NHW68/"

Commit message: rev 0.5 fixed
Parts:
- C17, C18: value 20pF -> 10pF
- J2: footprint Connector_PinSocket_1.27mm:PinSocket_2x07_P1.27mm_Vertical_SMD -> Connector_PinHeader_1.27mm:PinHeader_2x07_P1.27mm_Vertical
- R11: value 100K -> 100k
- moved J2 4.15 mm to (154.6, 90.4)
Routing:
- net GND: track 26.8 -> 289.2 mm, vias 31 -> 383
- net +3V3: track 402.6 -> 414.9 mm, vias 16 -> 15
- net /RGB/LED_EN_PIN: track 285.6 -> 292.7 mm
- net /SMT32/NRST: track 23.2 -> 29.8 mm, vias 0 -> 2
- net /SMT32/I2C2_SCL: track 283.1 -> 287.3 mm
- net /SMT32/VCP_TX: track 23.3 -> 26.2 mm
- net /SMT32/SWDIO: track 29.4 -> 31.6 mm
- net /SMT32/SWCLK: track 35.3 -> 37.4 mm
- net /SMT32/JTDR: track 31.8 -> 33.7 mm, vias 0 -> 1
- net /SMT32/I2C2_SDA: track 281.3 -> 283.2 mm
- net /SMT32/VCP_RX: track 25.8 -> 24.1 mm, vias 2 -> 0
- net /RGB/SYNC: track 200.9 -> 200.0 mm
