File: hardware/PCB/PCB.kicad_pcb (KiCad board)
At the start: 2 copper layers, 282.7 x 117.3 mm, 250 parts, among them J1 47346-0001, J2 1.27mm STDC14, SW1 B3U-1000P, U1 IS31FL3733-QFLS4-TR, U2 IS31FL3733-QFLS4-TR, U3 AZ1117CH-3.3TRG1, U4 STM32F303CCT6, Y1 8Mhz 20pf

Commit message: 0.6 I hate these auto generated code from STM32Cube
1. ready for the firmware nightmare
2. adjust the M3 screw holes
3. add tooling holes for future PCBA
4. if nothing go wrong, this will be the V1 after testing
Parts:
- added H1: M3Mount, MountingHole:MountingHole_3.2mm_M3_DIN965, F.Cu at (90.1, 89.0)
- added H2: M3Mount, MountingHole:MountingHole_3.2mm_M3_DIN965, F.Cu at (226.3, 87.8)
- added H3: M3Mount, MountingHole:MountingHole_3.2mm_M3_DIN965, F.Cu at (362.5, 89.0)
- added H4: M3Mount, MountingHole:MountingHole_3.2mm_M3_DIN965, F.Cu at (90.1, 195.9)
- added H5: M3Mount, MountingHole:MountingHole_3.2mm_M3_DIN965, F.Cu at (226.3, 197.0)
- added H6: M3Mount, MountingHole:MountingHole_3.2mm_M3_DIN965, F.Cu at (362.5, 195.9)
- added H7: M3Mount, KiCad:JLC_SMT_ToolingHole, F.Cu at (232.2, 199.3)
- added H8: M3Mount, KiCad:JLC_SMT_ToolingHole, F.Cu at (365.8, 189.6)
- added H9: M3Mount, KiCad:JLC_SMT_ToolingHole, F.Cu at (86.7, 94.3)
- moved R4 3.98 mm to (230.0, 191.4), turned to 270 degrees
- moved C19 0.09 mm to (148.8, 90.1)
- renumbered C26 to C19, C19 to C20, C20 to C21, C21 to C22, C22 to C23, C23 to C24, C24 to C25, C25 to C26, R14 to R10, R15 to R11, R13 to R12, R4 to R2, R7 to R3, R8 to R4, R11 to R5, R9 to R6, R10 to R7, R16 to R8, R12 to R9
Routing:
- net (no net): track 0.00 -> 272.2 mm, vias 0 -> 3
- net GND: track 289.2 -> 26.8 mm, vias 383 -> 246
- net Net-(R4-Pad1): track 3.78 -> 2.25 mm
- net /RGB/RGBmatrix2/ROW3: track 284.7 -> 283.4 mm
- net /SMT32/ROW5: track 379.0 -> 378.1 mm
- net +3V3: track 414.9 -> 414.3 mm
- net /SMT32/ROW2: track 314.2 -> 313.6 mm
- net /SMT32/JTDO: track 34.0 -> 33.5 mm
- net /SMT32/NRST: track 29.8 -> 29.6 mm, vias 2 -> 1
Other:
- outline, holes or cut-outs redrawn
- board text added: "NHW68 Rev:0.6 MIT License Copyright (c) 2019 Yifei Ding https://github.com/dingyifei/NHW68/"
- board text removed: "NHW68 Rev:0.5 MIT License Copyright (c) 2019 Yifei Ding https://github.com/dingyifei/NHW68/"

Commit message: fix some minor detail, I guess its v0.7
Parts:
- moved J1 0.73 mm to (115.0, 87.2)
- moved C16 0.50 mm to (109.0, 88.3), turned to 270 degrees
Routing:
- net /SMT32/USB_D+: track 6.72 -> 5.99 mm
- net /SMT32/USB_D-: track 4.20 -> 3.48 mm
Other:
- board text added: "NHW68 Rev:0.7 MIT License Copyright (c) 2019 Yifei Ding https://github.com/dingyifei/NHW68/"
- board text removed: "NHW68 Rev:0.6 MIT License Copyright (c) 2019 Yifei Ding https://github.com/dingyifei/NHW68/"
Changed lines of the file:
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@@
     (thickness 1.6)
     (drawings 295)
-    (tracks 3144)
+    (tracks 3145)
     (zones 0)
     (modules 259)
@@
     (title NHW68)
     (date 2020-02-10)
-    (rev 0.6)
+    (rev 0.7)
   )
   (layers
@@
   )
   (setup
-    (last_trace_width 0.3)
+    (last_trace_width 0.4)
     (user_trace_width 0.128)
     (user_trace_width 0.2)
@@
       (drillshape 0)
       (scaleselection 1)
-      (outputdirectory "output/"))
+      (outputdirectory "output/Gerber/"))
   )
   (net 0 "")
@@
   )
   (module Capacitor_SMD:C_0603_1608Metric (layer F.Cu)
-    (at 108.55 88.32)
+    (at 109.05 88.35 270)
     (descr "Capacitor SMD 0603 (1608 Metric), square (rectangular) end terminal, IPC_7351 nominal, (Body size source: http://www.tortai-tech.com/upload/download/2011102023233369053.pdf), generated with kicad-footprint-generator")
     (tags capacitor)
     (attr smd)
-    (fp_text reference C16 (at 0 -1.43) (layer F.SilkS)
+    (fp_text reference C16 (at 0 -1.43 90) (layer F.SilkS)
       (effects (font (size 0.85 0.7) (thickness 0.155)))
     )
-    (fp_text value 10uf (at 0 1.43) (layer F.Fab)
+    (fp_text value 10uf (at 0 1.43 90) (layer F.Fab)
       (effects (font (size 1 1) (thickness 0.15)))
     )
-    (fp_text user %R (at 0 0) (layer F.Fab)
+    (fp_text user %R (at 0 0 90) (layer F.Fab)
       (effects (font (size 1 1) (thickness 0.15)))
     )
@@
     (fp_line (start -0.8 -0.4) (end 0.8 -0.4) (layer F.Fab) (width 0.1))
     (fp_line (start -0.8 0.4) (end -0.8 -0.4) (layer F.Fab) (width 0.1))
-    (pad 2 smd roundrect (at 0.7875 0) (size 0.875 0.95) (layers F.Cu F.Paste F.Mask) (roundrect_rratio 0.25)
+    (pad 2 smd roundrect (at 0.7875 0 270) (size 0.875 0.95) (layers F.Cu F.Paste F.Mask) (roundrect_rratio 0.25)
       (net 1 GND))
-    (pad 1 smd roundrect (at -0.7875 0) (size 0.875 0.95) (layers F.Cu F.Paste F.Mask) (roundrect_rratio 0.25)
+    (pad 1 smd roundrect (at -0.7875 0 270) (size 0.875 0.95) (layers F.Cu F.Paste F.Mask) (roundrect_rratio 0.25)
       (net 53 +5V))
     (model ${KISYS3DMOD}/Capacitor_SMD.3dshapes/C_0603_1608Metric.wrl
@@
   )
   (module Connector_USB:USB_Micro-B_Molex_47346-0001 (layer F.Cu)
-    (at 114.975 86.425 180)
+    (at 114.975 87.15 180)
     (descr "Micro USB B receptable with flange, bottom-mount, SMD, right-angle (http://www.molex.com/pdm_docs/sd/473460001_sd.pdf)")
     (tags "Micro B USB SMD")
@@
   (gr_line (start 243.3348 118.840351) (end 243.3348 133.840351) (layer Eco1.User) (width 0.15))
   (gr_line (start 92.966085 90.789728) (end 92.966085 193.0398) (layer B.SilkS) (width 0.16))
-  (gr_text "NHW68\nRev:0.6\nMIT License\nCopyright (c) 2019 Yifei Ding\nhttps://github.com/dingyifei/NHW68/" (at 357.04 93.28) (layer F.SilkS)
+  (gr_text "NHW68\nRev:0.7\nMIT License\nCopyright (c) 2019 Yifei Ding\nhttps://github.com/dingyifei/NHW68/" (at 357.04 93.28) (layer F.SilkS)
     (effects (font (size 1.5 1.5) (thickness 0.2)) (justify right))
   )
@@
     (effects (font (size 1.5 1.5) (thickness 0.2)))
   )
-  (gr_text "NHW68\nRev:0.6\nMIT License\nCopyright (c) 2019 Yifei Ding\nhttps://github.com/dingyifei/NHW68/" (at 357.08 93.27) (layer B.SilkS)
+  (gr_text "NHW68\nRev:0.7\nMIT License\nCopyright (c) 2019 Yifei Ding\nhttps://github.com/dingyifei/NHW68/" (at 357.08 93.27) (layer B.SilkS)
     (effects (font (size 1.5 1.5) (thickness 0.2)) (justify left mirror))
   )
@@
   (segment (start 136.085637 92.299363) (end 136.085637 92.333225) (width 0.25) (layer F.Cu) (net 1))
   (via (at 136.085637 92.333225) (size 0.6) (drill 0.3) (layers F.Cu B.Cu) (net 1))
-  (via (at 113.69 89.04) (size 0.6) (drill 0.3) (layers F.Cu B.Cu) (net 1))
+  (via (at 113.69 89.75) (size 0.6) (drill 0.3) (layers F.Cu B.Cu) (net 1))
   (via (at 136.48 97.77) (size 0.6) (drill 0.3) (layers F.Cu B.Cu) (net 1))
-  (via (at 110.23 88.32) (size 0.6) (drill 0.3) (layers F.Cu B.Cu) (net 1))
+  (via (at 107.9 89.15) (size 0.6) (drill 0.3) (layers F.Cu B.Cu) (net 1))
   (via (at 127.63 94.85) (size 0.6) (drill 0.3) (layers F.Cu B.Cu) (net 1))
   (via (at 130.88 87.05) (size 0.6) (drill 0.3) (layers F.Cu B.Cu) (net 1))
@@
   (via (at 116.38 189.0675) (size 0.6) (drill 0.3) (layers F.Cu B.Cu) (net 1))
   (via (at 117.88 116.3175) (size 0.6) (drill 0.3) (layers F.Cu B.Cu) (net 1))
-  (via (at 118.63 89.3175) (size 0.6) (drill 0.3) (layers F.Cu B.Cu) (net 1))
+  (via (at 120.2 91.95) (size 0.6) (drill 0.3) (layers F.Cu B.Cu) (net 1))
   (via (at 116.36 148.76) (size 0.6) (drill 0.3) (layers F.Cu B.Cu) (net 1))
   (via (at 120.13 168.0675) (size 0.6) (drill 0.3) (layers F.Cu B.Cu) (net 1))
@@
   (segment (start 129.9765 88.05) (end 130.362 88.4355) (width 0.3) (layer F.Cu) (net 52) (status 20))
   (segment (start 129.2175 88.05) (end 129.9765 88.05) (width 0.3) (layer F.Cu) (net 52) (status 10))
-  (segment (start 107.7425 88.34) (end 107.7625 88.32) (width 0.4) (layer F.Cu) (net 53) (status 30))
-  (segment (start 105.14 88.34) (end 107.7425 88.34) (width 0.4) (layer F.Cu) (net 53) (status 30))
-  (segment (start 116.154999 86.674999) (end 109.407501 86.674999) (width 0.4) (layer F.Cu) (net 53))
-  (segment (start 116.275 87.885) (end 116.275 86.795) (width 0.4) (layer F.Cu) (net 53) (status 10))
-  (segment (start 109.407501 86.674999) (end 107.7625 88.32) (width 0.4) (layer F.Cu) (net 53) (status 20))
-  (segment (start 116.275 86.795) (end 116.154999 86.674999) (width 0.4) (layer F.Cu) (net 53))
+  (segment (start 116.154999 87.399999) (end 116.275 87.52) (width 0.4) (layer F.Cu) (net 53))
+  (segment (start 109.525 87.5625) (end 109.687501 87.399999) (width 0.4) (layer F.Cu) (net 53))
+  (segment (start 116.275 87.52) (end 116.275 88.61) (width 0.4) (layer F.Cu) (net 53))
+  (segment (start 109.687501 87.399999) (end 116.154999 87.399999) (width 0.4) (layer F.Cu) (net 53))
+  (segment (start 109.05 87.5625) (end 109.525 87.5625) (width 0.4) (layer F.Cu) (net 53))
+  (segment (start 105.9175 87.5625) (end 105.14 88.34) (width 0.4) (layer F.Cu) (net 53))
+  (segment (start 109.05 87.5625) (end 105.9175 87.5625) (width 0.4) (layer F.Cu) (net 53))
   (segment (start 113.834249 109.69) (end 113.974599 109.83035) (width 0.3) (layer F.Cu) (net 54) (status 30))
   (segment (start 94.924599 108.28035) (end 95.334949 107.87) (width 0.3) (layer F.Cu) (net 54))
@@
   (segment (start 88.16 109.31) (end 88.16 137.49) (width 0.25) (layer F.Cu) (net 75))
   (segment (start 98.62 98.85) (end 88.16 109.31) (width 0.25) (layer F.Cu) (net 75))
-  (segment (start 116.093153 91.484055) (end 115 90.390902) (width 0.3) (layer F.Cu) (net 76))
-  (segment (start 115 88.945001) (end 114.975 88.920001) (width 0.3) (layer F.Cu) (net 76))
-  (segment (start 116.093153 92.133153) (end 116.093153 91.484055) (width 0.3) (layer F.Cu) (net 76) (status 10))
-  (segment (start 115 90.390902) (end 115 88.945001) (width 0.3) (layer F.Cu) (net 76))
-  (segment (start 114.975 88.920001) (end 114.975 87.885) (width 0.3) (layer F.Cu) (net 76) (status 20))
   (segment (start 115.753806 92.4725) (end 116.093153 92.133153) (width 0.2) (layer F.Cu) (net 76) (status 20))
   (segment (start 114.23 92.4725) (end 115.753806 92.4725) (width 0.2) (layer F.Cu) (net 76) (status 10))
-  (segment (start 115.625 88.920001) (end 115.625 87.885) (width 0.3) (layer F.Cu) (net 77) (status 20))
-  (segment (start 117.156516 91.05979) (end 116.517418 91.05979) (width 0.3) (layer F.Cu) (net 77) (status 10))
+  (segment (start 116.093153 92.133153) (end 116.093153 91.484055) (width 0.3) (layer F.Cu) (net 76))
+  (segment (start 116.093153 91.484055) (end 115 90.390902) (width 0.3) (layer F.Cu) (net 76))
+  (segment (start 115 90.390902) (end 115 89.670001) (width 0.3) (layer F.Cu) (net 76))
+  (segment (start 114.975 89.645001) (end 114.975 88.61) (width 0.3) (layer F.Cu) (net 76))
+  (segment (start 115 89.670001) (end 114.975 89.645001) (width 0.3) (layer F.Cu) (net 76))
+  (segment (start 115.625 89.645001) (end 115.625 88.61) (width 0.3) (layer F.Cu) (net 77))
+  (segment (start 115.6 89.670001) (end 115.625 89.645001) (width 0.3) (layer F.Cu) (net 77))
   (segment (start 116.517418 91.05979) (end 115.6 90.142372) (width 0.3) (layer F.Cu) (net 77))
-  (segment (start 115.6 88.945001) (end 115.625 88.920001) (width 0.3) (layer F.Cu) (net 77))
-  (segment (start 115.6 90.142372) (end 115.6 88.945001) (width 0.3) (layer F.Cu) (net 77))
+  (segment (start 115.6 90.142372) (end 115.6 89.670001) (width 0.3) (layer F.Cu) (net 77))
+  (segment (start 117.156516 91.05979) (end 116.517418 91.05979) (width 0.3) (layer F.Cu) (net 77))
   (segment (start 94.241916 138.8875) (end 93.94 138.8875) (width 0.2) (layer F.Cu) (net 87) (status 30))
   (segment (start 95.466243 140.111827) (end 94.241916 138.8875) (width 0.2) (layer F.Cu) (net 87) (status 30))

Commit message: Remove some unused
Parts:
- D100, D101, D102, D103, D104, D105, D106, D107, D108, D109, D110, D111, D112, D113, D114, D115, D116, D117, D118, D119, D120, D121, D122, D123, D124, D125, D126, D127, D128, D129, D130, D131, D132, D133, D134, D135, D136, D69, D70, D71, D72, D73, D74, D75, D76, D77, D78, D79, D80, D81, D82, D83, D84, D85, D86, D87, D88, D89, D90, D91, D92, D93, D94, D95, D96, D97, D98, D99: footprint KiCad:RGB_LED_1205 -> KiCad:RGB_LED_1204_reverse
- H7, H8, H9: value M3Mount -> tooling
Connections:
- J1 pad 4: Net-(J1-Pad4) -> (no net)
- J2 pad 1: Net-(J2-Pad1) -> (no net)
- J2 pad 2: Net-(J2-Pad2) -> (no net)
- J2 pad 9: Net-(J2-Pad9) -> (no net)
- U1 pad 1: Net-(U1-Pad1) -> (no net)
- U1 pad 2: Net-(U1-Pad2) -> (no net)
- U1 pad 3: Net-(U1-Pad3) -> (no net)
- U1 pad 32: Net-(U1-Pad32) -> (no net)
- U1 pad 33: Net-(U1-Pad33) -> (no net)
- U1 pad 36: Net-(U1-Pad36) -> (no net)
- U1 pad 4: Net-(U1-Pad4) -> (no net)
- U1 pad 45: Net-(U1-Pad45) -> (no net)
- U2 pad 1: Net-(U2-Pad1) -> (no net)
- U2 pad 2: Net-(U2-Pad2) -> (no net)
- U2 pad 3: Net-(U2-Pad3) -> (no net)
- U2 pad 32: Net-(U2-Pad32) -> (no net)
- U2 pad 33: Net-(U2-Pad33) -> (no net)
- U2 pad 36: Net-(U2-Pad36) -> (no net)
- U2 pad 4: Net-(U2-Pad4) -> (no net)
- U2 pad 45: Net-(U2-Pad45) -> (no net)
- U2 pad 6: Net-(U2-Pad6) -> (no net)
- U2 pad 7: Net-(U2-Pad7) -> (no net)
- U2 pad 8: Net-(U2-Pad8) -> (no net)
- U4 pad 2: Net-(U4-Pad2) -> (no net)
- U4 pad 21: Net-(U4-Pad21) -> (no net)
- U4 pad 3: Net-(U4-Pad3) -> (no net)
- U4 pad 4: Net-(U4-Pad4) -> (no net)
- U4 pad 45: Net-(U4-Pad45) -> (no net)

Commit message: It is the last update of 1206 RGB design, going to switch LED again, correct the 1206 name
Parts:
- D100, D101, D102, D103, D104, D105, D106, D107, D108, D109, D110, D111, D112, D113, D114, D115, D116, D117, D118, D119, D120, D121, D122, D123, D124, D125, D126, D127, D128, D129, D130, D131, D132, D133, D134, D135, D136, D69, D70, D71, D72, D73, D74, D75, D76, D77, D78, D79, D80, D81, D82, D83, D84, D85, D86, D87, D88, D89, D90, D91, D92, D93, D94, D95, D96, D97, D98, D99: footprint KiCad:RGB_LED_1204_reverse -> KiCad:RGB_LED_1206_reverse

Commit message: I might just have to stick with 1206/4 did some research, maybe time to make another minimal system board....
Parts:
- added C27: 22uf/10v, Capacitor_Tantalum_SMD:CP_EIA-3216-18_Kemet-A, F.Cu at (79.6, 131.9)
- added C28: 22uf/10v, Capacitor_Tantalum_SMD:CP_EIA-3216-18_Kemet-A, F.Cu at (221.0, 183.5)
- C22: value 22uf -> 22uf/10v; footprint Capacitor_SMD:C_0603_1608Metric -> Capacitor_Tantalum_SMD:CP_EIA-3216-18_Kemet-A
- moved C22 2.05 mm to (109.8, 91.4)
- moved C1 0.44 mm to (97.7, 135.8)
- moved C3 0.44 mm to (96.7, 134.7)
- moved C2 0.44 mm to (95.6, 133.6)
- moved R3 0.43 mm to (225.2, 181.7)
Routing:
- net /RGB/RGBmatrix2/COL6: track 54.8 -> 44.5 mm, vias 4 -> 3
- net /RGB/RGBmatrix/COL13: track 72.1 -> 63.3 mm, vias 5 -> 4
- net /RGB/RGBmatrix2/ROW2: track 287.5 -> 296.0 mm
- net /RGB/RGBmatrix/ROW2: track 313.4 -> 321.1 mm
- net /RGB/RGBmatrix/ROW8: track 264.4 -> 272.0 mm
- net /RGB/RGBmatrix2/ROW5: track 274.4 -> 281.8 mm, vias 3 -> 2
- net /RGB/RGBmatrix/ROW5: track 294.0 -> 301.3 mm
- net /RGB/RGBmatrix/COL8: track 167.6 -> 160.6 mm
- net /RGB/RGBmatrix/COL6: track 206.5 -> 199.5 mm
- net /RGB/RGBmatrix/COL9: track 148.9 -> 141.9 mm
- net /RGB/RGBmatrix/COL11: track 111.5 -> 104.6 mm
- net /RGB/RGBmatrix/COL7: track 186.9 -> 179.9 mm
- net /RGB/RGBmatrix/COL10: track 130.2 -> 123.3 mm
- net /RGB/RGBmatrix/COL12: track 93.3 -> 86.4 mm
- net /RGB/RGBmatrix/ROW3: track 308.5 -> 315.3 mm
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
Commit message: fixing the Tantalum
Parts:
- moved C27 17.5 mm to (95.8, 125.2), turned to 0 degrees
Routing:
- net +3V3: track 420.0 -> 427.4 mm, vias 15 -> 16
