File: hardware/PCB/RGBmatrix.sch (KiCad schematic (older format))
At the start: 41 parts

Commit message: It is the last update of 1206 RGB design, going to switch LED again, correct the 1206 name
Parts:
- D100, D101, D102, D103, D104, D105, D106, D107, D108, D109, D69, D70, D71, D72, D73, D74, D75, D76, D77, D78, D79, D80, D81, D82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: footprint KiCad:RGB_LED_1204_reverse -> KiCad:RGB_LED_1206_reverse

Commit message: fix some detail for 1.0
Parts:
- renumbered D80 to D100, D83 to D101, D86 to D102, D89 to D103, D92 to D104, D95 to D105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
