File: hardware/PCB/PCB.sch (KiCad schematic (older format))
At the start: 9 parts

Commit message: fix some detail for 1.0
Parts:
- renumbered H3 to H2, H5 to H3, H2 to H4, H4 to H5
Changed lines of the file:
@@
 	6250 4950 5200 4950
 $Comp
-L Mechanical:MountingHole H4
+L Mechanical:MountingHole H5
 U 1 1 5E422B05
 P 1600 4700
-F 0 "H4" H 1700 4746 50  0000 L CNN
+F 0 "H5" H 1700 4746 50  0000 L CNN
 F 1 "M3Mount" H 1700 4655 50  0000 L CNN
 F 2 "MountingHole:MountingHole_3.2mm_M3_DIN965" H 1600 4700 50  0001 C CNN
@@
 $EndComp
 $Comp
-L Mechanical:MountingHole H2
+L Mechanical:MountingHole H4
 U 1 1 5E423012
 P 950 4700
-F 0 "H2" H 1050 4746 50  0000 L CNN
+F 0 "H4" H 1050 4746 50  0000 L CNN
 F 1 "M3Mount" H 1050 4655 50  0000 L CNN
 F 2 "MountingHole:MountingHole_3.2mm_M3_DIN965" H 950 4700 50  0001 C CNN
@@
 $EndComp
 $Comp
-L Mechanical:MountingHole H3
+L Mechanical:MountingHole H2
 U 1 1 5E42389A
 P 1600 4350
-F 0 "H3" H 1700 4396 50  0000 L CNN
+F 0 "H2" H 1700 4396 50  0000 L CNN
 F 1 "M3Mount" H 1700 4305 50  0000 L CNN
 F 2 "MountingHole:MountingHole_3.2mm_M3_DIN965" H 1600 4350 50  0001 C CNN
@@
 $EndComp
 $Comp
-L Mechanical:MountingHole H5
+L Mechanical:MountingHole H3
 U 1 1 5E4291CD
 P 2300 4350
-F 0 "H5" H 2400 4396 50  0000 L CNN
+F 0 "H3" H 2400 4396 50  0000 L CNN
 F 1 "M3Mount" H 2400 4305 50  0000 L CNN
 F 2 "MountingHole:MountingHole_3.2mm_M3_DIN965" H 2300 4350 50  0001 C CNN

Commit message: Non-RGB
Changed lines of the file:
@@
 $Descr A4 11693 8268
 encoding utf-8
-Sheet 1 6
+Sheet 1 3
 Title "NHW68"
 Date "2020-04-06"
@@
 $EndSheet
 $Sheet
-S 7450 3100 600  350
-U 5EC33E3D
-F0 "RGB" 50
-F1 "RGB.sch" 50
-F2 "SCL" I L 7450 3150 50
-F3 "SDA" I L 7450 3250 50
-F4 "LED_EN_PIN" I L 7450 3350 50
-$EndSheet
-$Sheet
 S 6250 2800 800  2250
 U 5E1424B2
@@
 $EndSheet
 Wire Wire Line
-	7050 3150 7450 3150
-Wire Wire Line
-	7450 3250 7050 3250
-Wire Wire Line
-	7050 3350 7450 3350
-Wire Wire Line
 	6250 3150 5200 3150
