File: hardware/PCB/switch.sch (KiCad schematic (older format))
At the start: 136 parts

Commit message: Code kinda works
Parts:
- D1, D10, D11, D12, D13, D14, D15, D16, D17, D18, D19, D2, D20, D21, D22, D23, D24, D25, D26, D27, D28, D29, D3, D30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: LCSC C118873 -> C110221

Commit message: fix some detail for 1.0
Parts:
- renumbered D45 to D10, D50 to D11, D55 to D12, D60 to D13, D65 to D14, D2 to D15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
