File: hardware/testing/RGB.sch (KiCad schematic (older format))
At the start: 2 parts

Commit message: starting the testing PCB
Parts:
- removed U?: IS31FL3731-QF, Package_DFN_QFN:QFN-28-1EP_4x4mm_P0.4mm_EP2.3x2.3mm, symbol Driver_LED:IS31FL3731-QF
- added C1, C4, C6, C8: 0.47μF, Capacitor_SMD:C_0402_1005Metric, symbol Device:C_Small
- added C3: 22μF/10V, Capacitor_Tantalum_SMD:CP_EIA-3216-18_Kemet-A, symbol Device:CP1_Small
- added C5, C7, C9: 0.1μF, Capacitor_SMD:C_0402_1005Metric, symbol Device:C_Small
- added R16, R23: 100k, Resistor_SMD:R_0402_1005Metric, symbol Device:R
- added R17, R18: 1k, Resistor_SMD:R_0402_1005Metric, symbol Device:R
- added R19: 20k, Resistor_SMD:R_0402_1005Metric, symbol Device:R
- U2: renamed from U?; footprint Package_DFN_QFN:QFN-48-1EP_6x6mm_P0.4mm_EP4.2x4.2mm -> Package_DFN_QFN:QFN-48-1EP_6x6mm_P0.4mm_EP4.2x4.2mm_ThermalVias; Footprint (none) -> Package_DFN_QFN:QFN-48-1EP_6x6mm_P0.4mm_EP4.2x4.2mm_Thermal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; Value (none) -> IS31FL7377
Connections:
- net labels added: +3.3V, GND, LED_EN_PIN, SCL, SDA, SYNC
- wire segments 0 -> 38
- no-connect marks 0 -> 6
Other:
- moved on the sheet: U2
