File: hardware/testing/RGBMatrix2.sch (KiCad schematic (older format))
At the start: 30 parts

Commit message: starting the testing PCB
Parts:
- removed D? (x30): LED_RGB, symbol Device:LED_RGB
- added D69, D70, D71, D72, D73, D74, D75, D76, D77, D78, D79, D80, D81, D82, D83, D84, D85, D86, D87, D88, D89, D90, D91, D92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: LED_RABG, KiCad:XZMDKCBDDG45S9_fixed, symbol Device:LED_RABG
Connections:
- net labels removed: COL15
- wire segments 330 -> 243
