File: hardware/testing/RGBmatrix.sch (KiCad schematic (older format))
At the start: 45 parts

Commit message: starting the testing PCB
Parts:
- removed D? (x45): LED_RGB, symbol Device:LED_RGB
- added D100, D101, D102, D103, D104, D105, D106, D107, D108, D109, D110, D111, D112, D113, D114, D115, D116, D117, D118, D119, D120, D121, D122, D123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: LED_RABG, KiCad:XZMDKCBDDG45S9_fixed, symbol Device:LED_RABG
Connections:
- net labels removed: COL15
- wire segments 495 -> 369
