File: hardware/testing/keyboard.kicad_pcb (KiCad board)
At the start: 2 copper layers, 166.4 x 109.2 mm, 33 parts

Commit message: starting the testing PCB
Parts:
- removed U_Main1: proton_c, proton_c:proton_c
- added C17: 1μF, Capacitor_SMD:C_0402_1005Metric, B.Cu at (119.3, 88.3)
- added C18: 0.1μF, Capacitor_SMD:C_0402_1005Metric, B.Cu at (119.3, 87.3)
- added C19: 0.01μF, Capacitor_SMD:C_0402_1005Metric, B.Cu at (122.7, 84.4)
- added C20: 1μF, Capacitor_SMD:C_0402_1005Metric, B.Cu at (122.7, 86.3)
- added C21: 20pF, Capacitor_SMD:C_0402_1005Metric, B.Cu at (86.7, 86.6)
- added C22: 20pF, Capacitor_SMD:C_0402_1005Metric, B.Cu at (89.5, 86.6)
- added C23: 1μF, Capacitor_SMD:C_0402_1005Metric, B.Cu at (95.0, 90.8)
- added C24: 0.1μF, Capacitor_SMD:C_0402_1005Metric, B.Cu at (127.4, 88.0)
- added C25: 0.1μF, Capacitor_SMD:C_0402_1005Metric, B.Cu at (126.4, 88.0)
- added C26: 0.1μF, Capacitor_SMD:C_0402_1005Metric, B.Cu at (125.4, 88.0)
- added C27: 0.1μF, Capacitor_SMD:C_0402_1005Metric, B.Cu at (124.4, 88.0)
- added CherryMX17: SW_SPST, TestPoint:TestPoint_2Pads_Pitch2.54mm_Drill0.8mm, F.Cu at (209.6, 109.4)
- added CherryMX18: SW_SPST, TestPoint:TestPoint_2Pads_Pitch2.54mm_Drill0.8mm, F.Cu at (209.6, 128.4)
- added CherryMX19: SW_SPST, TestPoint:TestPoint_2Pads_Pitch2.54mm_Drill0.8mm, F.Cu at (209.6, 147.5)
- added CherryMX20: SW_SPST, TestPoint:TestPoint_2Pads_Pitch2.54mm_Drill0.8mm, F.Cu at (209.6, 166.5)
- added CherryMX21: SW_SPST, TestPoint:TestPoint_2Pads_Pitch2.54mm_Drill0.8mm, F.Cu at (228.7, 90.3)
- added CherryMX22: SW_SPST, TestPoint:TestPoint_2Pads_Pitch2.54mm_Drill0.8mm, F.Cu at (228.7, 109.4)
- added CherryMX23: SW_SPST, TestPoint:TestPoint_2Pads_Pitch2.54mm_Drill0.8mm, F.Cu at (228.7, 128.4)
- added CherryMX24: SW_SPST, TestPoint:TestPoint_2Pads_Pitch2.54mm_Drill0.8mm, F.Cu at (228.7, 147.5)
- added CherryMX25: SW_SPST, TestPoint:TestPoint_2Pads_Pitch2.54mm_Drill0.8mm, F.Cu at (228.7, 166.5)
- added CherryMX26: SW_SPST, TestPoint:TestPoint_2Pads_Pitch2.54mm_Drill0.8mm, F.Cu at (243.0, 90.3)
- added CherryMX27: SW_SPST, TestPoint:TestPoint_2Pads_Pitch2.54mm_Drill0.8mm, F.Cu at (243.0, 109.4)
- added CherryMX28: SW_SPST, TestPoint:TestPoint_2Pads_Pitch2.54mm_Drill0.8mm, F.Cu at (243.0, 128.4)
- added CherryMX29: SW_SPST, TestPoint:TestPoint_2Pads_Pitch2.54mm_Drill0.8mm, F.Cu at (243.0, 147.5)
- added CherryMX30: SW_SPST, TestPoint:TestPoint_2Pads_Pitch2.54mm_Drill0.8mm, F.Cu at (252.5, 166.5)
- added CherryMX31: SW_SPST, TestPoint:TestPoint_2Pads_Pitch2.54mm_Drill0.8mm, F.Cu at (262.0, 90.3)
- added CherryMX32: SW_SPST, TestPoint:TestPoint_2Pads_Pitch2.54mm_Drill0.8mm, F.Cu at (262.0, 109.4)
- added CherryMX33: SW_SPST, TestPoint:TestPoint_2Pads_Pitch2.54mm_Drill0.8mm, F.Cu at (262.0, 128.4)
- added CherryMX34: SW_SPST, TestPoint:TestPoint_2Pads_Pitch2.54mm_Drill0.8mm, F.Cu at (262.0, 147.5)
- added CherryMX35: SW_SPST, TestPoint:TestPoint_2Pads_Pitch2.54mm_Drill0.8mm, F.Cu at (281.1, 90.3)
- added CherryMX36: SW_SPST, TestPoint:TestPoint_2Pads_Pitch2.54mm_Drill0.8mm, F.Cu at (281.1, 109.4)
- added CherryMX37: SW_SPST, TestPoint:TestPoint_2Pads_Pitch2.54mm_Drill0.8mm, F.Cu at (281.1, 128.4)
- added CherryMX38: SW_SPST, TestPoint:TestPoint_2Pads_Pitch2.54mm_Drill0.8mm, F.Cu at (281.1, 147.5)
- added CherryMX39: SW_SPST, TestPoint:TestPoint_2Pads_Pitch2.54mm_Drill0.8mm, F.Cu at (281.1, 166.5)
- added CherryMX40: SW_SPST, TestPoint:TestPoint_2Pads_Pitch2.54mm_Drill0.8mm, F.Cu at (300.1, 90.3)
- added CherryMX41: SW_SPST, TestPoint:TestPoint_2Pads_Pitch2.54mm_Drill0.8mm, F.Cu at (300.1, 109.4)
- added CherryMX42: SW_SPST, TestPoint:TestPoint_2Pads_Pitch2.54mm_Drill0.8mm, F.Cu at (300.1, 128.4)
- added CherryMX43: SW_SPST, TestPoint:TestPoint_2Pads_Pitch2.54mm_Drill0.8mm, F.Cu at (300.1, 147.5)
- added CherryMX44: SW_SPST, TestPoint:TestPoint_2Pads_Pitch2.54mm_Drill0.8mm, F.Cu at (300.1, 166.5)
- added CherryMX45: SW_SPST, TestPoint:TestPoint_2Pads_Pitch2.54mm_Drill0.8mm, F.Cu at (319.2, 90.3)
- added CherryMX46: SW_SPST, TestPoint:TestPoint_2Pads_Pitch2.54mm_Drill0.8mm, F.Cu at (319.2, 109.4)
- added CherryMX47: SW_SPST, TestPoint:TestPoint_2Pads_Pitch2.54mm_Drill0.8mm, F.Cu at (319.2, 128.4)
- added CherryMX48: SW_SPST, TestPoint:TestPoint_2Pads_Pitch2.54mm_Drill0.8mm, F.Cu at (319.2, 147.5)
- added CherryMX49: SW_SPST, TestPoint:TestPoint_2Pads_Pitch2.54mm_Drill0.8mm, F.Cu at (319.2, 166.5)
- added CherryMX50: SW_SPST, TestPoint:TestPoint_2Pads_Pitch2.54mm_Drill0.8mm, F.Cu at (338.2, 90.3)
- added CherryMX51: SW_SPST, TestPoint:TestPoint_2Pads_Pitch2.54mm_Drill0.8mm, F.Cu at (338.2, 109.4)
- added CherryMX52: SW_SPST, TestPoint:TestPoint_2Pads_Pitch2.54mm_Drill0.8mm, F.Cu at (338.2, 128.4)
- added CherryMX53: SW_SPST, TestPoint:TestPoint_2Pads_Pitch2.54mm_Drill0.8mm, F.Cu at (338.2, 147.5)
- added CherryMX54: SW_SPST, TestPoint:TestPoint_2Pads_Pitch2.54mm_Drill0.8mm, F.Cu at (338.2, 166.5)
- added CherryMX55: SW_SPST, TestPoint:TestPoint_2Pads_Pitch2.54mm_Drill0.8mm, F.Cu at (357.3, 90.3)
- added CherryMX56: SW_SPST, TestPoint:TestPoint_2Pads_Pitch2.54mm_Drill0.8mm, F.Cu at (357.3, 109.4)
- added CherryMX57: SW_SPST, TestPoint:TestPoint_2Pads_Pitch2.54mm_Drill0.8mm, F.Cu at (357.3, 128.4)
- added CherryMX58: SW_SPST, TestPoint:TestPoint_2Pads_Pitch2.54mm_Drill0.8mm, F.Cu at (357.3, 147.5)
- added CherryMX59: SW_SPST, TestPoint:TestPoint_2Pads_Pitch2.54mm_Drill0.8mm, F.Cu at (358.0, 171.1)
- added CherryMX60: SW_SPST, TestPoint:TestPoint_2Pads_Pitch2.54mm_Drill0.8mm, F.Cu at (376.3, 90.3)
- added CherryMX61: SW_SPST, TestPoint:TestPoint_2Pads_Pitch2.54mm_Drill0.8mm, F.Cu at (376.3, 109.4)
- added CherryMX62: SW_SPST, TestPoint:TestPoint_2Pads_Pitch2.54mm_Drill0.8mm, F.Cu at (385.8, 128.4)
- added CherryMX63: SW_SPST, TestPoint:TestPoint_2Pads_Pitch2.54mm_Drill0.8mm, F.Cu at (376.3, 147.5)
- added CherryMX64: SW_SPST, TestPoint:TestPoint_2Pads_Pitch2.54mm_Drill0.8mm, F.Cu at (376.3, 166.5)
- added CherryMX65: SW_SPST, TestPoint:TestPoint_2Pads_Pitch2.54mm_Drill0.8mm, F.Cu at (395.4, 90.3)
- added CherryMX66: SW_SPST, TestPoint:TestPoint_2Pads_Pitch2.54mm_Drill0.8mm, F.Cu at (395.4, 109.4)
- added CherryMX67: SW_SPST, TestPoint:TestPoint_2Pads_Pitch2.54mm_Drill0.8mm, F.Cu at (395.4, 147.5)
- added CherryMX68: SW_SPST, TestPoint:TestPoint_2Pads_Pitch2.54mm_Drill0.8mm, F.Cu at (395.4, 166.5)
- added D17: 1N4148W, Diode_SMD:D_SOD-523, B.Cu at (203.3, 111.4)
- added D18: 1N4148W, Diode_SMD:D_SOD-523, B.Cu at (203.3, 130.5)
- added D19: 1N4148W, Diode_SMD:D_SOD-523, B.Cu at (203.3, 149.5)
- added D20: 1N4148W, Diode_SMD:D_SOD-523, B.Cu at (203.3, 168.6)
- added D21: 1N4148W, Diode_SMD:D_SOD-523, B.Cu at (222.4, 92.4)
- added D22: 1N4148W, Diode_SMD:D_SOD-523, B.Cu at (222.4, 111.4)
- added D23: 1N4148W, Diode_SMD:D_SOD-523, B.Cu at (222.4, 130.5)
- added D24: 1N4148W, Diode_SMD:D_SOD-523, B.Cu at (222.4, 149.5)
- added D25: 1N4148W, Diode_SMD:D_SOD-523, B.Cu at (222.4, 168.6)
- added D26: 1N4148W, Diode_SMD:D_SOD-523, B.Cu at (236.7, 92.4)
- added D27: 1N4148W, Diode_SMD:D_SOD-523, B.Cu at (236.7, 111.4)
- added D28: 1N4148W, Diode_SMD:D_SOD-523, B.Cu at (236.7, 130.5)
- added D29: 1N4148W, Diode_SMD:D_SOD-523, B.Cu at (236.7, 149.5)
- added D30: 1N4148W, Diode_SMD:D_SOD-523, B.Cu at (246.2, 168.6)
- added D31: 1N4148W, Diode_SMD:D_SOD-523, B.Cu at (255.7, 92.4)
- added D32: 1N4148W, Diode_SMD:D_SOD-523, B.Cu at (255.7, 111.4)
- added D33: 1N4148W, Diode_SMD:D_SOD-523, B.Cu at (255.7, 130.5)
- added D34: 1N4148W, Diode_SMD:D_SOD-523, B.Cu at (255.7, 149.5)
- added D35: 1N4148W, Diode_SMD:D_SOD-523, B.Cu at (274.8, 92.4)
- added D36: 1N4148W, Diode_SMD:D_SOD-523, B.Cu at (274.8, 111.4)
- added D37: 1N4148W, Diode_SMD:D_SOD-523, B.Cu at (274.8, 130.5)
- added D38: 1N4148W, Diode_SMD:D_SOD-523, B.Cu at (274.8, 149.5)
- added D39: 1N4148W, Diode_SMD:D_SOD-523, B.Cu at (274.8, 168.6)
- added D40: 1N4148W, Diode_SMD:D_SOD-523, B.Cu at (293.8, 92.4)
- added D41: 1N4148W, Diode_SMD:D_SOD-523, B.Cu at (293.8, 111.4)
- added D42: 1N4148W, Diode_SMD:D_SOD-523, B.Cu at (293.8, 130.5)
- added D43: 1N4148W, Diode_SMD:D_SOD-523, B.Cu at (293.8, 149.5)
- added D44: 1N4148W, Diode_SMD:D_SOD-523, B.Cu at (293.8, 168.6)
- added D45: 1N4148W, Diode_SMD:D_SOD-523, B.Cu at (312.9, 92.4)
- added D46: 1N4148W, Diode_SMD:D_SOD-523, B.Cu at (312.9, 111.4)
- added D47: 1N4148W, Diode_SMD:D_SOD-523, B.Cu at (312.9, 130.5)
- added D48: 1N4148W, Diode_SMD:D_SOD-523, B.Cu at (312.9, 149.5)
- added D49: 1N4148W, Diode_SMD:D_SOD-523, B.Cu at (312.9, 168.6)
- added D50: 1N4148W, Diode_SMD:D_SOD-523, B.Cu at (331.9, 92.4)
- added D51: 1N4148W, Diode_SMD:D_SOD-523, B.Cu at (331.9, 111.4)
- added D52: 1N4148W, Diode_SMD:D_SOD-523, B.Cu at (331.9, 130.5)
- added D53: 1N4148W, Diode_SMD:D_SOD-523, B.Cu at (331.9, 149.5)
- added D54: 1N4148W, Diode_SMD:D_SOD-523, B.Cu at (331.9, 168.6)
- added D55: 1N4148W, Diode_SMD:D_SOD-523, B.Cu at (351.0, 92.4)
- added D56: 1N4148W, Diode_SMD:D_SOD-523, B.Cu at (351.0, 111.4)
- added D57: 1N4148W, Diode_SMD:D_SOD-523, B.Cu at (351.0, 130.5)
- added D58: 1N4148W, Diode_SMD:D_SOD-523, B.Cu at (351.0, 149.5)
- added D59: 1N4148W, Diode_SMD:D_SOD-523, B.Cu at (351.0, 168.6)
- added D60: 1N4148W, Diode_SMD:D_SOD-523, B.Cu at (370.0, 92.4)
- added D61: 1N4148W, Diode_SMD:D_SOD-523, B.Cu at (370.0, 111.4)
- added D62: 1N4148W, Diode_SMD:D_SOD-523, B.Cu at (379.6, 130.5)
- added D63: 1N4148W, Diode_SMD:D_SOD-523, B.Cu at (370.0, 149.5)
- added D64: 1N4148W, Diode_SMD:D_SOD-523, B.Cu at (370.0, 168.6)
- added D65: 1N4148W, Diode_SMD:D_SOD-523, B.Cu at (389.1, 92.4)
- added D66: 1N4148W, Diode_SMD:D_SOD-523, B.Cu at (389.1, 111.4)
- added D67: 1N4148W, Diode_SMD:D_SOD-523, B.Cu at (389.1, 149.5)
- added D68: 1N4148W, Diode_SMD:D_SOD-523, B.Cu at (389.1, 168.6)
- added D96: BAT60JFILM, Diode_SMD:D_SOD-323, B.Cu at (122.7, 88.5)
- added J1: USB_B_Micro, Connector_USB:USB_Micro-B_Molex-105017-0001, F.Cu at (112.7, 83.2)
- added R25: 1.5K, Resistor_SMD:R_0402_1005Metric, B.Cu at (109.3, 90.4)
- added R26: 22, Resistor_SMD:R_0402_1005Metric, B.Cu at (108.8, 93.1)
- added R27: 22, Resistor_SMD:R_0402_1005Metric, B.Cu at (108.8, 92.1)
- added R28: 100K, Resistor_SMD:R_0402_1005Metric, B.Cu at (101.0, 97.8)
- added R29: 1K, Resistor_SMD:R_0402_1005Metric, B.Cu at (90.6, 91.4)
- added SW1: SW_DIP_x01, Button_Switch_SMD:SW_SPST_B3U-1000P, B.Cu at (95.4, 96.5)
- added TP1: TestPoint, TestPoint:TestPoint_Pad_D1.0mm, B.Cu at (130.5, 86.4)
- added TP2: TestPoint, TestPoint:TestPoint_Pad_D1.0mm, B.Cu at (117.4, 86.2)
- added TP5: TestPoint, TestPoint:TestPoint_Pad_D1.0mm, B.Cu at (130.5, 89.5)
- added U1: STM32F303CCTx, Package_QFP:LQFP-48_7x7mm_P0.5mm, B.Cu at (101.7, 91.6)
- added U4: LD3985M33R, Package_TO_SOT_SMD:SOT-23-5, B.Cu at (119.8, 85.4)
- added Y1: YSX530GA, Crystal:Crystal_SMD_5032-2Pin_5.0x3.2mm, B.Cu at (88.1, 89.0)
- CherryMX1, CherryMX10, CherryMX11, CherryMX12, CherryMX13, CherryMX14, CherryMX15, CherryMX16, CherryMX2, CherryMX3, CherryMX4, CherryMX5, CherryMX6, CherryMX7, CherryMX8, CherryMX9: footprint Button_Switch_Keyboard:SW_Cherry_MX_1.00u_Plate -> TestPoint:TestPoint_2Pads_Pitch2.54mm_Drill0.8mm
- D1, D10, D11, D12, D13, D14, D15, D16, D2, D3, D4, D5, D6, D7, D8, D9: footprint Diode_SMD:D_SOD-123 -> Diode_SMD:D_SOD-523; moved to B.Cu
- moved CherryMX13 102.8 mm to (190.6, 128.4), turned to 180 degrees
- moved D13 102.7 mm to (184.3, 130.5), turned to 270 degrees
- moved CherryMX5 97.4 mm to (152.5, 166.5), turned to 180 degrees
- moved CherryMX9 87.7 mm to (171.5, 147.5), turned to 180 degrees
- moved D5 84.3 mm to (146.2, 168.6), turned to 270 degrees
- moved CherryMX4 84.1 mm to (152.5, 147.5), turned to 180 degrees
- moved D9 80.1 mm to (165.2, 149.5), turned to 270 degrees
- moved D16 74.4 mm to (203.3, 92.4), turned to 270 degrees
- moved CherryMX14 73.8 mm to (190.6, 147.5), turned to 180 degrees
- moved CherryMX10 73.1 mm to (171.5, 166.5), turned to 180 degrees
- moved D14 71.0 mm to (184.3, 149.5), turned to 270 degrees
- moved D4 70.7 mm to (146.2, 149.5), turned to 270 degrees
- moved CherryMX16 62.0 mm to (209.6, 90.3), turned to 180 degrees
- moved CherryMX3 61.5 mm to (152.5, 128.4), turned to 180 degrees
- moved D10 60.5 mm to (165.2, 168.6), turned to 270 degrees
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Connections:
- CherryMX1 pad 1: /switch/ROW1 -> /SMT32/ROW1
- CherryMX10 pad 1: /switch/ROW2 -> /SMT32/ROW5
- CherryMX11 pad 1: /switch/ROW3 -> /SMT32/ROW1
- CherryMX12 pad 1: /switch/ROW4 -> /SMT32/ROW2
- CherryMX13 pad 1: /switch/ROW1 -> /SMT32/ROW3
- CherryMX14 pad 1: /switch/ROW2 -> /SMT32/ROW4
- CherryMX15 pad 1: /switch/ROW3 -> /SMT32/ROW5
- CherryMX16 pad 1: /switch/ROW4 -> /SMT32/ROW1
- CherryMX2 pad 1: /switch/ROW2 -> /SMT32/ROW2
- CherryMX3 pad 1: /switch/ROW3 -> /SMT32/ROW3
- CherryMX4 pad 1: /switch/ROW4 -> /SMT32/ROW4
- CherryMX5 pad 1: /switch/ROW1 -> /SMT32/ROW5
- CherryMX6 pad 1: /switch/ROW2 -> /SMT32/ROW1
- CherryMX7 pad 1: /switch/ROW3 -> /SMT32/ROW2
- CherryMX8 pad 1: /switch/ROW4 -> /SMT32/ROW3
- CherryMX9 pad 1: /switch/ROW1 -> /SMT32/ROW4
- D1 pad 1: /switch/COL1 -> /SMT32/COL14
- D10 pad 1: /switch/COL3 -> /SMT32/COL13
- D11 pad 1: /switch/COL3 -> /SMT32/COL12
- D12 pad 1: /switch/COL3 -> /SMT32/COL12
- D13 pad 1: /switch/COL4 -> /SMT32/COL12
- D14 pad 1: /switch/COL4 -> /SMT32/COL12
- D15 pad 1: /switch/COL4 -> /SMT32/COL12
- D16 pad 1: /switch/COL4 -> /SMT32/COL11
- D2 pad 1: /switch/COL1 -> /SMT32/COL14
- D3 pad 1: /switch/COL1 -> /SMT32/COL14
- D4 pad 1: /switch/COL1 -> /SMT32/COL14
- D5 pad 1: /switch/COL2 -> /SMT32/COL14
- D6 pad 1: /switch/COL2 -> /SMT32/COL13
- D7 pad 1: /switch/COL2 -> /SMT32/COL13
- D8 pad 1: /switch/COL2 -> /SMT32/COL13
- D9 pad 1: /switch/COL3 -> /SMT32/COL13
Routing:
- net /switch/COL4: track 182.3 -> 0.00 mm
- net /switch/ROW1: track 181.7 -> 0.00 mm
- net /switch/COL3: track 173.6 -> 0.00 mm
- net /switch/ROW2: track 157.4 -> 0.00 mm
- net /switch/COL2: track 138.1 -> 0.00 mm, vias 1 -> 0
- net /switch/ROW3: track 130.9 -> 0.00 mm
- net /switch/COL1: track 125.9 -> 0.00 mm, vias 1 -> 0
- net GND: track 0.00 -> 95.0 mm, vias 0 -> 7
- net /switch/ROW4: track 93.1 -> 0.00 mm
- net +3V3: track 0.00 -> 49.2 mm
- net Net-(U_Main1-PadGND): track 20.3 -> 0.00 mm
- net Net-(C21-Pad2): track 0.00 -> 16.1 mm
- net Net-(CherryMX3-Pad2): track 15.7 -> 0.00 mm
- net Net-(CherryMX2-Pad2): track 15.7 -> 0.00 mm
- net Net-(CherryMX9-Pad2): track 15.7 -> 0.00 mm
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Other:
- board size 166.4 x 109.2 mm -> 100 x 100 mm
- net class Default: clearance 0.2 -> 0.15; trace_width 0.25 -> 0.3; via_drill 0.4 -> 0.35
- net class Power added: clearance 0.15, trace_width 0.3, via_dia 0.8, via_drill 0.35
- net class RGB_Power added: clearance 0.15, trace_width 0.2, via_dia 0.8, via_drill 0.35
- net class Signal added: clearance 0.15, trace_width 0.2, via_dia 0.6, via_drill 0.35
- rule trace_clearance: 0.2 -> 0.15
- rule trace_min: 0.2 -> 0.127
- rule via_min_size: 0.4 -> 0.6

Commit message: remove useless files
Parts:
- moved CherryMX59 282.5 mm to (78.9, 127.2)
- moved CherryMX6 79.2 mm to (94.1, 106.9)
- moved D1 3.59 mm to (76.6, 106.9), turned to 0 degrees
Changed lines of the file:
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@@
   )
   (module TestPoint:TestPoint_2Pads_Pitch2.54mm_Drill0.8mm (layer F.Cu)
-    (at 358.013 171.1325)
+    (at 78.9305 127.1905)
     (descr "Test point with 2 pins, pitch 2.54mm, drill diameter 0.8mm")
     (tags "CONN DEV")
@@
   )
   (module Diode_SMD:D_SOD-523 (layer B.Cu)
-    (at 79.248 104.394 270)
+    (at 76.6445 106.8705)
     (descr "http://www.diodes.com/datasheets/ap02001.pdf p.144")
     (tags "Diode SOD523")
     (attr smd)
-    (fp_text reference D1 (at 0 1.3 90) (layer B.SilkS)
+    (fp_text reference D1 (at 0 1.3) (layer B.SilkS)
       (effects (font (size 1 1) (thickness 0.15)) (justify mirror))
     )
-    (fp_text value 1N4148W (at 0 -1.4 90) (layer B.Fab)
+    (fp_text value 1N4148W (at 0 -1.4) (layer B.Fab)
       (effects (font (size 1 1) (thickness 0.15)) (justify mirror))
     )
@@
     (fp_line (start 1.25 0.7) (end 1.25 -0.7) (layer B.CrtYd) (width 0.05))
     (fp_line (start -1.15 0.6) (end -1.15 -0.6) (layer B.SilkS) (width 0.12))
-    (fp_text user %R (at 0 1.3 90) (layer B.Fab)
+    (fp_text user %R (at 0 1.3) (layer B.Fab)
       (effects (font (size 1 1) (thickness 0.15)) (justify mirror))
     )
-    (pad 1 smd rect (at -0.7 0 90) (size 0.6 0.7) (layers B.Cu B.Paste B.Mask)
+    (pad 1 smd rect (at -0.7 0 180) (size 0.6 0.7) (layers B.Cu B.Paste B.Mask)
       (net 89 /SMT32/COL14))
-    (pad 2 smd rect (at 0.7 0 90) (size 0.6 0.7) (layers B.Cu B.Paste B.Mask)
+    (pad 2 smd rect (at 0.7 0 180) (size 0.6 0.7) (layers B.Cu B.Paste B.Mask)
       (net 2 "Net-(CherryMX1-Pad2)"))
     (model ${KISYS3DMOD}/Diode_SMD.3dshapes/D_SOD-523.wrl
@@
   )
   (module TestPoint:TestPoint_2Pads_Pitch2.54mm_Drill0.8mm (layer F.Cu)
-    (at 171.528151 90.34585 180)
+    (at 94.107 106.8705 180)
     (descr "Test point with 2 pins, pitch 2.54mm, drill diameter 0.8mm")
     (tags "CONN DEV")

Commit message: making testing PCB, making sure the DFU mode is correct
Parts:
- removed CherryMX1, CherryMX10, CherryMX11, CherryMX12, CherryMX13, CherryMX14, CherryMX15, CherryMX16, CherryMX17, CherryMX18, CherryMX19, CherryMX2, CherryMX20, CherryMX21, CherryMX22, CherryMX23, CherryMX24, CherryMX25, CherryMX26, CherryMX27, CherryMX28, CherryMX29, CherryMX3, CherryMX30, CherryMX31, CherryMX32, CherryMX33, CherryMX34, CherryMX35, CherryMX36, CherryMX37, CherryMX38, CherryMX39, CherryMX4, CherryMX40, CherryMX41, CherryMX42, CherryMX43, CherryMX44, CherryMX45, CherryMX46, CherryMX47, CherryMX48, CherryMX49, CherryMX5, CherryMX50, CherryMX51, CherryMX52, CherryMX53, CherryMX54, CherryMX55, CherryMX56, CherryMX57, CherryMX58, CherryMX59, CherryMX6, CherryMX60, CherryMX61, CherryMX62, CherryMX63, CherryMX64, CherryMX65, CherryMX66, CherryMX67, CherryMX68, CherryMX7, CherryMX8, CherryMX9: SW_SPST, TestPoint:TestPoint_2Pads_Pitch2.54mm_Drill0.8mm
- added R1: 100K, Resistor_SMD:R_0402_1005Metric, B.Cu at (147.1, 54.7)
- added R2: 100K, Resistor_SMD:R_0402_1005Metric, B.Cu at (148.1, 54.7)
- added SW10: CherryMX, TestPoint:TestPoint_2Pads_Pitch2.54mm_Drill0.8mm, B.Cu at (151.6, 105.6)
- added SW11: CherryMX, TestPoint:TestPoint_2Pads_Pitch2.54mm_Drill0.8mm, B.Cu at (147.9, 74.8)
- added SW12: CherryMX, TestPoint:TestPoint_2Pads_Pitch2.54mm_Drill0.8mm, B.Cu at (147.9, 82.5)
- added SW13: CherryMX, TestPoint:TestPoint_2Pads_Pitch2.54mm_Drill0.8mm, B.Cu at (147.9, 90.2)
- added SW14: CherryMX, TestPoint:TestPoint_2Pads_Pitch2.54mm_Drill0.8mm, B.Cu at (147.9, 97.9)
- added SW15: CherryMX, TestPoint:TestPoint_2Pads_Pitch2.54mm_Drill0.8mm, B.Cu at (147.9, 105.6)
- added SW16: CherryMX, TestPoint:TestPoint_2Pads_Pitch2.54mm_Drill0.8mm, B.Cu at (144.2, 74.8)
- added SW17: CherryMX, TestPoint:TestPoint_2Pads_Pitch2.54mm_Drill0.8mm, B.Cu at (144.2, 82.5)
- added SW18: CherryMX, TestPoint:TestPoint_2Pads_Pitch2.54mm_Drill0.8mm, B.Cu at (144.2, 90.2)
- added SW19: CherryMX, TestPoint:TestPoint_2Pads_Pitch2.54mm_Drill0.8mm, B.Cu at (144.2, 97.9)
- added SW2: CherryMX, TestPoint:TestPoint_2Pads_Pitch2.54mm_Drill0.8mm, B.Cu at (155.3, 82.5)
- added SW20: CherryMX, TestPoint:TestPoint_2Pads_Pitch2.54mm_Drill0.8mm, B.Cu at (144.2, 105.6)
- added SW21: CherryMX, TestPoint:TestPoint_2Pads_Pitch2.54mm_Drill0.8mm, B.Cu at (140.5, 74.8)
- added SW22: CherryMX, TestPoint:TestPoint_2Pads_Pitch2.54mm_Drill0.8mm, B.Cu at (140.5, 82.5)
- added SW23: CherryMX, TestPoint:TestPoint_2Pads_Pitch2.54mm_Drill0.8mm, B.Cu at (140.5, 90.2)
- added SW24: CherryMX, TestPoint:TestPoint_2Pads_Pitch2.54mm_Drill0.8mm, B.Cu at (140.5, 97.9)
- added SW25: CherryMX, TestPoint:TestPoint_2Pads_Pitch2.54mm_Drill0.8mm, B.Cu at (140.5, 105.6)
- added SW26: CherryMX, TestPoint:TestPoint_2Pads_Pitch2.54mm_Drill0.8mm, B.Cu at (136.8, 74.8)
- added SW27: CherryMX, TestPoint:TestPoint_2Pads_Pitch2.54mm_Drill0.8mm, B.Cu at (136.8, 82.5)
- added SW28: CherryMX, TestPoint:TestPoint_2Pads_Pitch2.54mm_Drill0.8mm, B.Cu at (136.8, 90.2)
- added SW29: CherryMX, TestPoint:TestPoint_2Pads_Pitch2.54mm_Drill0.8mm, B.Cu at (136.8, 97.9)
- added SW3: CherryMX, TestPoint:TestPoint_2Pads_Pitch2.54mm_Drill0.8mm, B.Cu at (155.3, 90.2)
- added SW30: CherryMX, TestPoint:TestPoint_2Pads_Pitch2.54mm_Drill0.8mm, B.Cu at (136.8, 105.6)
- added SW31: CherryMX, TestPoint:TestPoint_2Pads_Pitch2.54mm_Drill0.8mm, B.Cu at (133.1, 74.8)
- added SW32: CherryMX, TestPoint:TestPoint_2Pads_Pitch2.54mm_Drill0.8mm, B.Cu at (133.1, 82.5)
- added SW33: CherryMX, TestPoint:TestPoint_2Pads_Pitch2.54mm_Drill0.8mm, B.Cu at (133.1, 90.2)
- added SW34: CherryMX, TestPoint:TestPoint_2Pads_Pitch2.54mm_Drill0.8mm, B.Cu at (133.1, 97.9)
- added SW35: CherryMX, TestPoint:TestPoint_2Pads_Pitch2.54mm_Drill0.8mm, B.Cu at (129.4, 74.8)
- added SW36: CherryMX, TestPoint:TestPoint_2Pads_Pitch2.54mm_Drill0.8mm, B.Cu at (129.4, 82.5)
- added SW37: CherryMX, TestPoint:TestPoint_2Pads_Pitch2.54mm_Drill0.8mm, B.Cu at (129.4, 90.2)
- added SW38: CherryMX, TestPoint:TestPoint_2Pads_Pitch2.54mm_Drill0.8mm, B.Cu at (129.4, 97.9)
- added SW39: CherryMX, TestPoint:TestPoint_2Pads_Pitch2.54mm_Drill0.8mm, B.Cu at (129.4, 105.6)
- added SW4: CherryMX, TestPoint:TestPoint_2Pads_Pitch2.54mm_Drill0.8mm, B.Cu at (155.3, 97.9)
- added SW40: CherryMX, TestPoint:TestPoint_2Pads_Pitch2.54mm_Drill0.8mm, B.Cu at (125.7, 74.8)
- added SW41: CherryMX, TestPoint:TestPoint_2Pads_Pitch2.54mm_Drill0.8mm, B.Cu at (125.7, 82.5)
- added SW42: CherryMX, TestPoint:TestPoint_2Pads_Pitch2.54mm_Drill0.8mm, B.Cu at (125.7, 90.2)
- added SW43: CherryMX, TestPoint:TestPoint_2Pads_Pitch2.54mm_Drill0.8mm, B.Cu at (125.7, 97.9)
- added SW44: CherryMX, TestPoint:TestPoint_2Pads_Pitch2.54mm_Drill0.8mm, B.Cu at (125.7, 105.6)
- added SW45: CherryMX, TestPoint:TestPoint_2Pads_Pitch2.54mm_Drill0.8mm, B.Cu at (122.0, 74.8)
- added SW46: CherryMX, TestPoint:TestPoint_2Pads_Pitch2.54mm_Drill0.8mm, B.Cu at (122.0, 82.5)
- added SW47: CherryMX, TestPoint:TestPoint_2Pads_Pitch2.54mm_Drill0.8mm, B.Cu at (122.0, 90.2)
- added SW48: CherryMX, TestPoint:TestPoint_2Pads_Pitch2.54mm_Drill0.8mm, B.Cu at (122.0, 97.9)
- added SW49: CherryMX, TestPoint:TestPoint_2Pads_Pitch2.54mm_Drill0.8mm, B.Cu at (122.0, 105.6)
- added SW5: CherryMX, TestPoint:TestPoint_2Pads_Pitch2.54mm_Drill0.8mm, B.Cu at (155.3, 105.6)
- added SW50: CherryMX, TestPoint:TestPoint_2Pads_Pitch2.54mm_Drill0.8mm, B.Cu at (118.3, 74.8)
- added SW51: CherryMX, TestPoint:TestPoint_2Pads_Pitch2.54mm_Drill0.8mm, B.Cu at (118.3, 82.5)
- added SW52: CherryMX, TestPoint:TestPoint_2Pads_Pitch2.54mm_Drill0.8mm, B.Cu at (118.3, 90.2)
- added SW53: CherryMX, TestPoint:TestPoint_2Pads_Pitch2.54mm_Drill0.8mm, B.Cu at (118.3, 97.9)
- added SW54: CherryMX, TestPoint:TestPoint_2Pads_Pitch2.54mm_Drill0.8mm, B.Cu at (118.3, 105.6)
- added SW55: CherryMX, TestPoint:TestPoint_2Pads_Pitch2.54mm_Drill0.8mm, B.Cu at (114.6, 74.8)
- added SW56: CherryMX, TestPoint:TestPoint_2Pads_Pitch2.54mm_Drill0.8mm, B.Cu at (114.6, 82.5)
- added SW57: CherryMX, TestPoint:TestPoint_2Pads_Pitch2.54mm_Drill0.8mm, B.Cu at (114.6, 90.2)
- added SW58: CherryMX, TestPoint:TestPoint_2Pads_Pitch2.54mm_Drill0.8mm, B.Cu at (114.6, 97.9)
- added SW59: CherryMX, TestPoint:TestPoint_2Pads_Pitch2.54mm_Drill0.8mm, B.Cu at (114.6, 105.6)
- added SW6: CherryMX, TestPoint:TestPoint_2Pads_Pitch2.54mm_Drill0.8mm, B.Cu at (151.6, 74.8)
- added SW60: CherryMX, TestPoint:TestPoint_2Pads_Pitch2.54mm_Drill0.8mm, B.Cu at (110.9, 74.8)
- added SW61: CherryMX, TestPoint:TestPoint_2Pads_Pitch2.54mm_Drill0.8mm, B.Cu at (110.9, 82.5)
- added SW62: CherryMX, TestPoint:TestPoint_2Pads_Pitch2.54mm_Drill0.8mm, B.Cu at (110.9, 90.2)
- added SW63: CherryMX, TestPoint:TestPoint_2Pads_Pitch2.54mm_Drill0.8mm, B.Cu at (110.9, 97.9)
- added SW64: CherryMX, TestPoint:TestPoint_2Pads_Pitch2.54mm_Drill0.8mm, B.Cu at (110.9, 105.6)
- added SW65: CherryMX, TestPoint:TestPoint_2Pads_Pitch2.54mm_Drill0.8mm, B.Cu at (107.2, 74.8)
- added SW66: CherryMX, TestPoint:TestPoint_2Pads_Pitch2.54mm_Drill0.8mm, B.Cu at (107.2, 82.5)
- added SW67: CherryMX, TestPoint:TestPoint_2Pads_Pitch2.54mm_Drill0.8mm, B.Cu at (107.2, 97.9)
- added SW68: CherryMX, TestPoint:TestPoint_2Pads_Pitch2.54mm_Drill0.8mm, B.Cu at (107.2, 105.6)
- added SW7: CherryMX, TestPoint:TestPoint_2Pads_Pitch2.54mm_Drill0.8mm, B.Cu at (151.6, 82.5)
- added SW8: CherryMX, TestPoint:TestPoint_2Pads_Pitch2.54mm_Drill0.8mm, B.Cu at (151.6, 90.2)
- added SW9: CherryMX, TestPoint:TestPoint_2Pads_Pitch2.54mm_Drill0.8mm, B.Cu at (151.6, 97.9)
- added SW_debug_1: SW_DIP_x01, TestPoint:TestPoint_2Pads_Pitch2.54mm_Drill0.8mm, B.Cu at (124.1, 58.2)
- added TP3: TestPoint, TestPoint:TestPoint_Pad_D2.0mm, B.Cu at (151.4, 65.4)
- added TP4: TestPoint, TestPoint:TestPoint_Pad_D2.0mm, B.Cu at (151.4, 61.4)
- added TP6: TestPoint, TestPoint:TestPoint_Pad_D2.0mm, B.Cu at (151.4, 57.3)
- SW1: value SW_DIP_x01 -> CherryMX; footprint Button_Switch_SMD:SW_SPST_B3U-1000P -> TestPoint:TestPoint_2Pads_Pitch2.54mm_Drill0.8mm
- TP1, TP2, TP5: footprint TestPoint:TestPoint_Pad_D1.0mm -> TestPoint:TestPoint_Pad_D2.0mm
- moved D68 290.0 mm to (107.2, 100.5)
- moved D67 287.5 mm to (107.2, 92.8)
- moved D66 283.9 mm to (107.2, 77.4)
- moved D65 282.8 mm to (107.2, 69.7)
- moved D62 272.5 mm to (110.9, 85.1)
- moved D64 267.9 mm to (110.9, 100.5)
- moved D63 265.3 mm to (110.9, 92.8)
- moved D61 261.4 mm to (110.9, 77.4)
- moved D60 260.1 mm to (110.9, 69.7)
- moved D59 246.0 mm to (114.6, 100.5)
- moved D58 243.1 mm to (114.6, 92.8)
- moved D57 240.7 mm to (114.6, 85.1)
- moved D56 238.8 mm to (114.6, 77.4)
- moved D55 237.5 mm to (114.6, 69.7)
- moved D54 224.2 mm to (118.3, 100.5)
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Connections:
- net /SMT32/LED_EN_PIN renamed Net-(U1-Pad34)
- D1 pad 2: Net-(CherryMX1-Pad2) -> Net-(D1-Pad2)
- SW1 pad 1: GND -> /SMT32/ROW1
- SW1 pad 2: Net-(C23-Pad2) -> Net-(D1-Pad2)
Routing:
- net /SMT32/ROW5: track 3.54 -> 94.6 mm, vias 1 -> 0
- net /SMT32/ROW4: track 3.34 -> 86.6 mm, vias 1 -> 0
- net /SMT32/COL1: track 0.12 -> 74.4 mm, vias 0 -> 2
- net /SMT32/ROW3: track 3.55 -> 75.0 mm, vias 1 -> 0
- net /SMT32/COL2: track 0.00 -> 71.0 mm, vias 0 -> 2
- net /SMT32/ROW2: track 3.77 -> 72.3 mm, vias 2 -> 0
- net /SMT32/COL14: track 0.00 -> 65.4 mm, vias 0 -> 2
- net /SMT32/COL13: track 0.00 -> 62.5 mm, vias 0 -> 2
- net /SMT32/COL10: track 0.00 -> 61.6 mm, vias 0 -> 2
- net /SMT32/ROW1: track 3.93 -> 64.4 mm, vias 1 -> 0
- net /SMT32/COL12: track 0.00 -> 60.0 mm, vias 0 -> 2
- net /SMT32/COL4: track 0.00 -> 58.8 mm, vias 0 -> 2
- net /SMT32/COL11: track 0.00 -> 58.0 mm, vias 0 -> 2
- net /SMT32/COL9: track 0.00 -> 57.1 mm, vias 0 -> 2
- net /SMT32/COL3: track 1.31 -> 58.0 mm, vias 1 -> 2
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- added copper zone on F.Cu, net GND
Other:
- rule trace_min: 0.127 -> 0.13
