File: hardware/testing/testing.sch (KiCad schematic (older format))
At the start: 0 parts

Commit message: small changes
Changed lines of the file:
@@
 $Descr A4 11693 8268
 encoding utf-8
-Sheet 1 3
+Sheet 1 4
 Title ""
 Date ""
@@
 Wire Wire Line
 	5500 4600 4450 4600
+$Sheet
+S 7250 2600 750  1650
+U 5E2317EE
+F0 "SpareParts" 50
+F1 "SpareParts.sch" 50
+$EndSheet
 $EndSCHEMATC
