File: hardware/testing/SMT32.sch (KiCad schematic (older format))
At the start: 25 parts, among them J1 USB_B_Micro, SW1 SW_DIP_x01, U1 STM32F303CCTx, U4 LD3985M33R, Y1 YSX530GA

Commit message: making testing PCB, making sure the DFU mode is correct
Parts:
- added R1, R2: 100K, Resistor_SMD:R_0402_1005Metric, symbol Device:R
- added TP3, TP4, TP6: TestPoint, TestPoint:TestPoint_Pad_D2.0mm, symbol Connector:TestPoint
- SW_debug_1: renamed from SW1; footprint Button_Switch_SMD:SW_SPST_B3U-1000P -> TestPoint:TestPoint_2Pads_Pitch2.54mm_Drill0.8mm
- TP1, TP2, TP5: footprint TestPoint:TestPoint_Pad_D1.0mm -> TestPoint:TestPoint_Pad_D2.0mm
Connections:
- net +3V3: now also R1.1, R2.1
- net at U1.29 (PA8): now also R2.2, TP6.1
- net at U1.30 (PA9): now also R1.2, TP4.1
- net at U1.31 (PA10): now also TP3.1
- net LED_EN_PIN: no longer names the net of U1.34 (PA13)
- no-connect marks 9 -> 12
Changed lines of the file:
@@
 Connection ~ 5600 2550
 $Comp
-L Switch:SW_DIP_x01 SW1
+L Switch:SW_DIP_x01 SW_debug_1
 U 1 1 5E234436
 P 5600 2250
-F 0 "SW1" V 5554 2380 50  0000 L CNN
+F 0 "SW_debug_1" V 5554 2380 50  0000 L CNN
 F 1 "SW_DIP_x01" V 5645 2380 50  0000 L CNN
-F 2 "Button_Switch_SMD:SW_SPST_B3U-1000P" H 5600 2250 50  0001 C CNN
+F 2 "TestPoint:TestPoint_2Pads_Pitch2.54mm_Drill0.8mm" H 5600 2250 50  0001 C CNN
 F 3 "~" H 5600 2250 50  0001 C CNN
 	1    5600 2250
@@
 Text HLabel 6400 4050 0    50   Input ~ 0
 ROW4
-NoConn ~ 7700 4450
 NoConn ~ 6400 5150
-Text HLabel 7700 4950 2    50   Input ~ 0
-LED_EN_PIN
 Wire Wire Line
 	1500 2550 1600 2550
@@
 F 0 "TP2" H 2008 1868 50  0000 L CNN
 F 1 "TestPoint" H 2008 1777 50  0000 L CNN
-F 2 "TestPoint:TestPoint_Pad_D1.0mm" H 2150 1750 50  0001 C CNN
+F 2 "TestPoint:TestPoint_Pad_D2.0mm" H 2150 1750 50  0001 C CNN
 F 3 "~" H 2150 1750 50  0001 C CNN
 	1    1950 1750
@@
 F 0 "TP1" H 1558 2668 50  0000 L CNN
 F 1 "TestPoint" H 1558 2577 50  0000 L CNN
-F 2 "TestPoint:TestPoint_Pad_D1.0mm" H 1700 2550 50  0001 C CNN
+F 2 "TestPoint:TestPoint_Pad_D2.0mm" H 1700 2550 50  0001 C CNN
 F 3 "~" H 1700 2550 50  0001 C CNN
 	1    1500 2550
@@
 F 0 "TP5" H 4158 5868 50  0000 L CNN
 F 1 "TestPoint" H 4158 5777 50  0000 L CNN
-F 2 "TestPoint:TestPoint_Pad_D1.0mm" H 4300 5750 50  0001 C CNN
+F 2 "TestPoint:TestPoint_Pad_D2.0mm" H 4300 5750 50  0001 C CNN
 F 3 "~" H 4300 5750 50  0001 C CNN
 	1    4100 5750
@@
 Wire Wire Line
 	1900 2250 2300 2250
+NoConn ~ 6400 4850
+NoConn ~ 6400 4950
+NoConn ~ 6400 5050
+NoConn ~ 7700 4950
+$Comp
+L Connector:TestPoint TP3
+U 1 1 5E6FF36A
+P 7700 4650
+F 0 "TP3" V 7654 4838 50  0000 L CNN
+F 1 "TestPoint" V 7745 4838 50  0000 L CNN
+F 2 "TestPoint:TestPoint_Pad_D2.0mm" H 7900 4650 50  0001 C CNN
+F 3 "~" H 7900 4650 50  0001 C CNN
+	1    7700 4650
+	0    1    1    0
+$EndComp
+$Comp
+L Device:R R1
+U 1 1 5E7013A0
+P 8250 4400
+F 0 "R1" H 8320 4446 50  0000 L CNN
+F 1 "100K" H 8320 4355 50  0000 L CNN
+F 2 "Resistor_SMD:R_0402_1005Metric" V 8180 4400 50  0001 C CNN
+F 3 "~" H 8250 4400 50  0001 C CNN
+	1    8250 4400
+	1    0    0    -1
+$EndComp
+$Comp
+L Device:R R2
+U 1 1 5E70217F
+P 8550 4300
+F 0 "R2" H 8620 4346 50  0000 L CNN
+F 1 "100K" H 8620 4255 50  0000 L CNN
+F 2 "Resistor_SMD:R_0402_1005Metric" V 8480 4300 50  0001 C CNN
+F 3 "~" H 8550 4300 50  0001 C CNN
+	1    8550 4300
+	1    0    0    -1
+$EndComp
+Wire Wire Line
+	8550 4450 7700 4450
+Wire Wire Line
+	8250 4550 7700 4550
+$Comp
+L power:+3.3V #PWR01
+U 1 1 5E70AB05
+P 8250 4250
+F 0 "#PWR01" H 8250 4100 50  0001 C CNN
+F 1 "+3.3V" H 8265 4423 50  0000 C CNN
+F 2 "" H 8250 4250 50  0001 C CNN
+F 3 "" H 8250 4250 50  0001 C CNN
+	1    8250 4250
+	1    0    0    -1
+$EndComp
+$Comp
+L power:+3.3V #PWR02
+U 1 1 5E70B726
+P 8550 4150
+F 0 "#PWR02" H 8550 4000 50  0001 C CNN
+F 1 "+3.3V" H 8565 4323 50  0000 C CNN
+F 2 "" H 8550 4150 50  0001 C CNN
+F 3 "" H 8550 4150 50  0001 C CNN
+	1    8550 4150
+	1    0    0    -1
+$EndComp
+$Comp
+L Connector:TestPoint TP4
+U 1 1 5E70E403
+P 8250 4550
+F 0 "TP4" V 8204 4738 50  0000 L CNN
+F 1 "TestPoint" V 8295 4738 50  0000 L CNN
+F 2 "TestPoint:TestPoint_Pad_D2.0mm" H 8450 4550 50  0001 C CNN
+F 3 "~" H 8450 4550 50  0001 C CNN
+	1    8250 4550
+	0    1    1    0
+$EndComp
+$Comp
+L Connector:TestPoint TP6
+U 1 1 5E70FA5A
+P 8550 4450
+F 0 "TP6" V 8504 4638 50  0000 L CNN
+F 1 "TestPoint" V 8595 4638 50  0000 L CNN
+F 2 "TestPoint:TestPoint_Pad_D2.0mm" H 8750 4450 50  0001 C CNN
+F 3 "~" H 8750 4450 50  0001 C CNN
+	1    8550 4450
+	0    1    1    0
+$EndComp
 $EndSCHEMATC

Commit message: Full Send, SMT assembly LOL
Parts:
- removed R1, R2: 100K, Resistor_SMD:R_0402_1005Metric, symbol Device:R
- removed TP6: TestPoint, TestPoint:TestPoint_Pad_D2.0mm, symbol Connector:TestPoint
- added BOOT0UP1: SW_DIP_x01, TestPoint:TestPoint_2Pads_Pitch2.54mm_Drill0.8mm, symbol Switch:SW_DIP_x01
- added C1, C3: 10uF, Capacitor_SMD:C_0402_1005Metric, symbol Device:C
- added C2: 100nF, Capacitor_SMD:C_0402_1005Metric, symbol Device:C
- C17, C20, C23: value 1μF -> 1uF
- C18, C24, C25, C26, C27: value 0.1μF -> 100nF
- C19: value 0.01μF -> 10nF
- TP1, TP2, TP3, TP4, TP5: footprint TestPoint:TestPoint_Pad_D2.0mm -> TestPoint:TestPoint_THTPad_D1.5mm_Drill0.7mm
- U1: value STM32F303CCTx -> STM32F303CCT6
- Y1: value YSX530GA -> X50328MSB2GI
- renumbered SW_debug_1 to RST1
Connections:
- net +3V3: now also BOOT0UP1.1; no longer TP5.1
- net +5V: now also C1.1
- net GND: now also C1.2, C2.2, C3.2
- net at R28.2, U1.44 (BOOT0): now also BOOT0UP1.2
- net at C20.1, D96.1 (K), U4.5 (VOUT): now also C2.1, C3.1
- no-connect marks 12 -> 13
Other:
- moved on the sheet: C17, C18, C19, C20, C24, C25, C26, C27, D96, TP3, TP4, TP5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

Commit message: small changes
Parts:
- Y1: value X50328MSB2GI -> 8Mhz 20PF
Connections:
- net +3V3: now also TP5.1
Other:
- moved on the sheet: TP5
Changed lines of the file:
@@
 $Descr A4 11693 8268
 encoding utf-8
-Sheet 3 3
+Sheet 3 4
 Title ""
 Date ""
@@
 P 4950 3000
 F 0 "Y1" V 4904 3131 50  0000 L CNN
-F 1 "X50328MSB2GI" V 4995 3131 50  0000 L CNN
+F 1 "8Mhz 20PF" V 4995 3131 50  0000 L CNN
 F 2 "Crystal:Crystal_SMD_5032-2Pin_5.0x3.2mm" H 4950 3000 50  0001 C CNN
 F 3 "~" H 4950 3000 50  0001 C CNN
@@
 L Connector:TestPoint TP5
 U 1 1 5E20237D
-P 4400 5600
-F 0 "TP5" H 4458 5718 50  0000 L CNN
-F 1 "TestPoint" H 4458 5627 50  0000 L CNN
-F 2 "TestPoint:TestPoint_THTPad_D1.5mm_Drill0.7mm" H 4600 5600 50  0001 C CNN
-F 3 "~" H 4600 5600 50  0001 C CNN
-	1    4400 5600
-	1    0    0    -1
-$EndComp
+P 4500 5600
+F 0 "TP5" H 4558 5718 50  0000 L CNN
+F 1 "TestPoint" H 4558 5627 50  0000 L CNN
+F 2 "TestPoint:TestPoint_THTPad_D1.5mm_Drill0.7mm" H 4700 5600 50  0001 C CNN
+F 3 "~" H 4700 5600 50  0001 C CNN
+	1    4500 5600
+	1    0    0    -1
+$EndComp

Commit message: Making progress, so many distance warning!!!
Connections:
- net at U1.32 (PA11): now also R26.1; no longer R27.2
- net at U1.33 (PA12): now also R27.2; no longer R26.1
Other:
- moved on the sheet: R26, R27
Changed lines of the file:
@@
 	-1   0    0    1
 $EndComp
-Text Label 8000 5550 3    50   ~ 0
+Text Label 8050 5550 3    50   ~ 0
 USB_D+
 $Comp
@@
 	1    0    0    -1
 $EndComp
-Text Label 7850 5550 3    50   ~ 0
+Text Label 7900 5550 3    50   ~ 0
 USB_D-
 Text Label 2300 2150 0    50   ~ 0
@@
 L Device:R R27
 U 1 1 5E1E3849
-P 8000 5400
-F 0 "R27" V 7793 5400 50  0000 C CNN
-F 1 "22" V 7884 5400 50  0000 C CNN
-F 2 "Resistor_SMD:R_0402_1005Metric" V 7930 5400 50  0001 C CNN
-F 3 "~" H 8000 5400 50  0001 C CNN
-	1    8000 5400
+P 8050 5400
+F 0 "R27" V 7843 5400 50  0000 C CNN
+F 1 "22" V 7934 5400 50  0000 C CNN
+F 2 "Resistor_SMD:R_0402_1005Metric" V 7980 5400 50  0001 C CNN
+F 3 "~" H 8050 5400 50  0001 C CNN
+	1    8050 5400
 	-1   0    0    1
 $EndComp
@@
 L Device:R R26
 U 1 1 5E1E2865
-P 7850 5400
-F 0 "R26" V 7643 5400 50  0000 C CNN
-F 1 "22" V 7734 5400 50  0000 C CNN
-F 2 "Resistor_SMD:R_0402_1005Metric" V 7780 5400 50  0001 C CNN
-F 3 "~" H 7850 5400 50  0001 C CNN
-	1    7850 5400
+P 7900 5400
+F 0 "R26" V 7693 5400 50  0000 C CNN
+F 1 "22" V 7784 5400 50  0000 C CNN
+F 2 "Resistor_SMD:R_0402_1005Metric" V 7830 5400 50  0001 C CNN
+F 3 "~" H 7900 5400 50  0001 C CNN
+	1    7900 5400
 	1    0    0    -1
 $EndComp
@@
 	-1   0    0    1
 $EndComp
-Wire Wire Line
-	7700 4750 8000 4750
-Wire Wire Line
-	8000 4750 8000 5250
-Wire Wire Line
-	7700 4850 7850 4850
-Wire Wire Line
-	7850 4850 7850 5250
 Text HLabel 6400 4750 0    50   Input ~ 0
 COL1
@@
 	3600 6600 4050 6600
 Connection ~ 3600 6600
+Wire Wire Line
+	8050 4850 8050 5250
+Wire Wire Line
+	7900 4750 7700 4750
+Wire Wire Line
+	7900 4750 7900 5250
+Wire Wire Line
+	7700 4850 8050 4850
 $EndSCHEMATC
