File: hardware/testing/testing.kicad_pcb (KiCad board)
At the start: 2 copper layers, 68 x 64.5 mm, 167 parts, among them J1 USB_B_Micro, SW1 SW, SW10 SW, SW11 SW, SW12 SW, SW13 SW, SW14 SW, SW15 SW, SW16 SW, SW17 SW, SW18 SW, SW19 SW, SW2 SW, SW20 SW, SW21 SW, SW22 SW, SW23 SW, SW24 SW, SW25 SW, SW26 SW, SW27 SW, SW28 SW, SW29 SW, SW3 SW, SW30 SW, SW31 SW, SW32 SW, SW33 SW, SW34 SW, SW35 SW, SW36 SW, SW37 SW, SW38 SW, SW39 SW, SW4 SW, SW40 SW, SW41 SW, SW42 SW, SW43 SW, SW44 SW, SW45 SW, SW46 SW, SW47 SW, SW48 SW, SW49 SW, SW5 SW, SW50 SW, SW51 SW, SW52 SW, SW53 SW, SW54 SW, SW55 SW, SW56 SW, SW57 SW, SW58 SW, SW59 SW, SW6 SW, SW60 SW, SW61 SW, SW62 SW, SW63 SW, SW64 SW, SW65 SW, SW66 SW, SW67 SW, SW68 SW, SW7 SW, SW8 SW, SW9 SW, U1 STM32F303CCT6, U4 LD3985M33R, Y1 X50328MSB2GI

Commit message: small changes
Parts:
- added D69: MHT150RGBCT, KiCad:LED_1206_3216Metric, F.Cu at (97.3, 82.9)
- added D70: MHT150RGBCT, KiCad:LED_1206_3216Metric, F.Cu at (100.7, 82.9)
- added D71: MHT150RGBCT, KiCad:LED_1206_3216Metric, F.Cu at (97.3, 77.2)
- added D72: MHT150RGBCT, KiCad:LED_1206_3216Metric, F.Cu at (101.1, 88.1)
- added D73: MHT150RGBCT, KiCad:LED_1206_3216Metric, F.Cu at (100.7, 77.2)
- added D74: MHT150RGBCT, KiCad:LED_1206_3216Metric, F.Cu at (97.3, 71.6)
- added D75: MHT150RGBCT, KiCad:LED_1206_3216Metric, F.Cu at (97.3, 88.2)
- added D76: MHT150RGBCT, KiCad:LED_1206_3216Metric, F.Cu at (100.7, 71.6)
- Y1: value X50328MSB2GI -> 8Mhz 20PF
Connections:
- TP5 pad 1: Net-(TP5-Pad1) -> +3V3
Routing:
- net /SMT32/USB_D+: track 11.0 -> 11.5 mm

Commit message: Making progress, so many distance warning!!!
Parts:
- J1: moved to F.Cu
- moved R26 5.34 mm to (122.0, 55.6)
- moved R27 3.92 mm to (120.3, 56.7)
- turned J1 to 180 degrees
Connections:
- U1 pad 32: Net-(R27-Pad2) -> Net-(R26-Pad1)
- U1 pad 33: Net-(R26-Pad1) -> Net-(R27-Pad2)
Routing:
- net /SMT32/USB_D+: track 11.5 -> 0.00 mm, vias 1 -> 0
- net /SMT32/USB_D-: track 11.3 -> 0.00 mm, vias 1 -> 0
- net Net-(R27-Pad2): track 2.56 -> 0.34 mm
- net Net-(R26-Pad1): track 2.57 -> 0.35 mm
- net +5V: track 17.0 -> 19.1 mm, vias 1 -> 0
