File: hardware/Mounting_PCB/Mounting_PCB.kicad_pcb (KiCad board)
At the start: 2 copper layers, 282.7 x 117.3 mm, 6 parts

Commit message: fix some code, trying to figure out the plate
Parts:
- added REF**: OSHW-Logo_7.5x8mm_Copper, Symbol:OSHW-Logo_7.5x8mm_Copper, F.Cu at (115.9, 114.9)
- added REF**: KiCad-Logo2_5mm_Copper, Symbol:KiCad-Logo2_5mm_Copper, F.Cu at (103.0, 114.9)
- moved H4 11.3 mm to (223.3, 220.4)
- moved H1 11.3 mm to (87.1, 112.3)
- moved H3 11.3 mm to (359.5, 112.3)
- moved H2 11.3 mm to (223.3, 111.2)
- moved H5 11.3 mm to (87.1, 219.2)
- moved H6 11.3 mm to (359.5, 219.2)
Routing:
- added copper zone on F.Cu, net (none)
- removed copper zone on B.Cu, net (none)
Other:
- board text added: "NHW68 V1.0 By Yifei Ding"

Commit message: change footprint
Parts:
- removed REF**: OSHW-Logo_7.5x8mm_Copper, Symbol:OSHW-Logo_7.5x8mm_Copper
- removed REF**: KiCad-Logo2_5mm_Copper, Symbol:KiCad-Logo2_5mm_Copper
- H1, H2, H3, H4, H5, H6: footprint MountingHole:MountingHole_3.2mm_M3_DIN965 -> MountingHole:MountingHole_3.2mm_M3_Pad_Via
- moved H4 45.9 mm to (210.6, 176.3)
- moved H1 45.9 mm to (74.4, 68.3)
- moved H3 45.9 mm to (346.8, 68.3)
- moved H2 45.9 mm to (210.6, 67.1)
- moved H5 45.9 mm to (74.4, 175.2)
- moved H6 45.9 mm to (346.8, 175.2)
Connections:
- H1 pad 1: (no net) -> Net-(H1-Pad1)
- H2 pad 1: (no net) -> Net-(H1-Pad1)
- H3 pad 1: (no net) -> Net-(H1-Pad1)
- H4 pad 1: (no net) -> Net-(H1-Pad1)
- H5 pad 1: (no net) -> Net-(H1-Pad1)
- H6 pad 1: (no net) -> Net-(H1-Pad1)
Routing:
- removed copper zone on F.Cu, net (none)
