File: hardware/Mounting_PCB/Mounting_PCB.kicad_pcb (KiCad board)
At the start: 2 copper layers, 282.7 x 117.3 mm, 6 parts

Commit message: Cleanup, make everything nice, get ready for making it on JLC
Routing:
- net Net-(H1-Pad1): vias 0 -> 345
- added copper zone on B.Cu, net Net-(H1-Pad1)
- added copper zone on F.Cu, net Net-(H1-Pad1)

Commit message: v1.1, too many problems I have to fix
Parts:
- moved H5 0.38 mm to (74.6, 174.8)
- moved H2 0.38 mm to (210.8, 66.7)
- moved H4 0.38 mm to (210.8, 176.0)
- moved H1 0.38 mm to (74.6, 67.9)
- moved H6 0.38 mm to (347.0, 174.8)
- moved H3 0.38 mm to (347.0, 67.9)
Other:
- outline, holes or cut-outs redrawn

Commit message: Non-RGB
Other:
- board text added: "NHW68 V1.0"
- board text removed: "NHW68 V1.0 By Yifei Ding"
Changed lines of the file:
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@@
   (gr_line (start 316.5598 129.1703) (end 316.5598 133.6393) (layer Edge.Cuts) (width 0.05))
   (gr_line (start 93.96 119.87) (end 79.96045 119.87) (layer Edge.Cuts) (width 0.05))
-  (gr_text "NHW68 V1.0 By Yifei Ding" (at 109.511043 72.59) (layer F.SilkS)
+  (gr_text "NHW68 V1.0" (at 109.511043 72.59) (layer F.SilkS)
     (effects (font (size 3 3) (thickness 0.5)))
   )
