File: hardware/Base/base.kicad_pcb (KiCad board)
At the start: 2 copper layers, 282.7 x 117.3 mm, 6 parts

Commit message: change stuff so everything export the right way
Parts:
- H1, H2, H3, H4, H5, H6: footprint MountingHole:MountingHole_3.2mm_M3 -> MountingHole:MountingHole_3.2mm_M3_Pad_Via
Routing:
- net Net-(H1-Pad1): vias 0 -> 536
- net (no net): vias 469 -> 0
- added copper zone on B.Cu, net Net-(H1-Pad1)
- added copper zone on F.Cu, net Net-(H1-Pad1)
- removed copper zone on B.Cu, net (none)
- removed copper zone on F.Cu, net (none)
