File: hardware/Spacer/Spacer.kicad_pcb (KiCad board)
At the start: 2 copper layers, 282.7 x 117.3 mm, 6 parts

Commit message: change stuff so everything export the right way
Parts:
- added NT1: Net-Tie_2, Crystal:Crystal_SMD_0603-2Pin_6.0x3.5mm, F.Cu at (186.8, 66.6)
Connections:
- H1 pad 1: Net-(H1-Pad1) -> (no net)
- H2 pad 1: Net-(H1-Pad1) -> (no net)
- H3 pad 1: Net-(H1-Pad1) -> (no net)
- H4 pad 1: Net-(H1-Pad1) -> (no net)
- H5 pad 1: Net-(H1-Pad1) -> (no net)
- H6 pad 1: Net-(H1-Pad1) -> (no net)
Routing:
- net GND: vias 0 -> 93
- net (no net): vias 93 -> 0
- added copper zone on B.Cu, net GND
- added copper zone on F.Cu, net GND
- removed copper zone on B.Cu, net (none)
- removed copper zone on F.Cu, net (none)

Commit message: v1.1, too many problems I have to fix
Parts:
- moved H6 2.44 mm to (346.4, 177.0)
- moved H4 2.44 mm to (210.2, 68.9)
- moved H3 2.44 mm to (346.4, 70.1)
- moved H2 2.44 mm to (74.1, 177.0)
- moved H1 2.44 mm to (74.1, 70.1)
- moved H5 2.44 mm to (210.2, 178.1)
Routing:
- net GND: vias 93 -> 98
- net (no net): vias 0 -> 1
Other:
- outline, holes or cut-outs redrawn
